File: hardware/kicad/boards/04_flag_reg/04_flag_reg.kicad_sch (KiCad schematic)
At the start: 0 parts

Commit message: feat: designed shift and flag reg kicad boards
Parts:
- added C1, C2, C3: 100nF, symbol Device:C
- added U1, U2: 74HC74, symbol 74xx:74HC74
- added U3: 74LS08, symbol 74xx:74LS08
Connections:
- new net: U3.3, U3.4
- new net GND: C1.2, C2.2, C3.2, U1.7 (GND), U2.7 (GND), U3.10, U3.12, U3.13, U3.7 (GND), U3.9
- new net VCC: C1.1, C2.1, C3.1, U1.1 (~{R}), U1.10 (~{S}), U1.13 (~{R}), U1.14 (VCC), U1.4 (~{S}), U2.1 (~{R}), U2.10 (~{S}), U2.13 (~{R}), U2.14 (VCC), U2.4 (~{S}), U3.14 (VCC)
- new net carry_in: U1.12 (D)
- new net clk: U3.1
- new net clk_gated: U1.11 (C), U1.3 (C), U2.11 (C), U2.3 (C), U3.6
- new net exec: U3.2
- new net flag_c: U1.9 (Q)
- new net flag_cn: U1.8 (~{Q})
- new net flag_en: U3.5
- new net flag_n: U2.5 (Q)
- new net flag_n_n: U2.6 (~{Q})
- new net flag_nz: U1.6 (~{Q})
- new net flag_o: U2.9 (Q)
- new net flag_on: U2.8 (~{Q})
- new net flag_z: U1.5 (Q)
- new net neg_in: U2.2 (D)
- new net overflow_in: U2.12 (D)
- new net zero_in: U1.2 (D)
- no-connect marks 0 -> 2
