File: hardware/kicad/boards/01_alu/alu-1b.kicad_sch (KiCad schematic)
At the start: 4 parts, among them U1 74LS08, U2 74HC86

Commit message: feat: updated kicad 1b alu
Parts:
- renumbered C1 to C13, C2 to C14, U1 to U13, U2 to U14
Connections:
- net G: now also U13.8; no longer U14.8
- net GND: now also U14.10, U14.9
- net P: no longer U13.8
- net aeff: no longer U14.9
- net beff: no longer U14.10
- no-connect marks 2 -> 3
Other:
- sheet mux_8to1 ports: added mux1-out; removed none
