File: hardware/kicad/boards/01_alu/alu-1b.kicad_sch (KiCad schematic)
At the start: 4 parts, among them U13 74LS08, U14 74HC86

Commit message: feat: designed alu0-control unit and wired on top level of 32b alu
Parts:
- renumbered C13 to C1, C14 to C2, U13 to U1, U13 to U2, U13 to U3, U14 to U4, U14 to U5, U14 to U6

Commit message: kicad: checkpoint; designed the alu display logic; clock circuit
Added registers for each display to ensure robustness and less worry about debugging screen, keeping focus on the alu board and other components
Parts:
- renumbered C1 to C31, C2 to C32, U1 to U31, U2 to U32, U3 to U33, U4 to U34, U5 to U35, U6 to U36

Commit message: alu: completed all core schematics; DRC and ERC pending 🎉
Parts:
- renumbered C31 to C33, C32 to C34, U31 to U33, U32 to U34, U33 to U35, U34 to U36, U35 to U37, U36 to U38

Commit message: refactor: changed hpins to global for asel, ainv, precondition, alu-opcode
Parts:
- renumbered U34 to U33, U35 to U33, U36 to U34, U37 to U34, U38 to U34

Commit message: feat: designed ALU board with 0 ERC errors or warnings 🎉
Final review of logical correctness and footprints and then routing begins
Parts:
- renumbered C33 to C301, C34 to C302, U34 to U301, U33 to U302
