File: hardware/kicad/boards/01_alu/display-counter.kicad_sch (KiCad schematic)
At the start: 4 parts, among them U275 74LS154, U276 74LS154, U277 74LS163, U278 74LS163

Commit message: alu: completed all core schematics; DRC and ERC pending 🎉
Parts:
- added C205, C206, C207, C208, C209, C266, C267, C268: 100nF, Capacitor_SMD:C_0805_2012Metric, symbol Device:C
- added U239: 74AHC1G04, Package_TO_SOT_SMD:SOT-23-5, symbol 74xGxx:74AHC1G04
- added U296, U297: 74LS153, Package_SO:SOIC-16_3.9x9.9mm_P1.27mm, symbol 74xx:74LS153
- added U298: KM28C64A, Package_DIP:DIP-28_W15.24mm, symbol Memory_EEPROM:KM28C64A
- U237: renamed from U275; footprint (none) -> Package_SO:SOIC-24W_7.5x15.4mm_P1.27mm
- U238: renamed from U277; footprint (none) -> Package_SO:SOIC-16_3.9x9.9mm_P1.27mm
- U240: renamed from U278; footprint (none) -> Package_SO:SOIC-16_3.9x9.9mm_P1.27mm
- U241: renamed from U276; footprint (none) -> Package_SO:SOIC-24W_7.5x15.4mm_P1.27mm
Connections:
- net q0: now also U237.23 (A0), U241.23 (A0)
- net q1: now also U237.22 (A1), U241.22 (A1)
- net q2: now also U237.21 (A2), U241.21 (A2)
- net q3: now also U237.20 (A3), U241.20 (A3), U296.14 (S0), U297.14 (S0)
- net q4: now also U237.19 (E1), U239.2, U296.2 (S1), U297.2 (S1)
- net regW0: no longer U241.8 (S7)
- net VCC: now reaches U238.1 (~{MR}), U238.10 (CET), U238.7 (CEP), U238.9 (~{PE})
- net VCC: now also U237.24 (VCC), U238.16 (VCC), U240.1 (~{MR}), U240.16 (VCC), U240.9 (~{PE}), U241.24 (VCC), C205.1, C206.1, C207.1, C208.1, C209.1, C266.1, C267.1, C268.1, U239.5 (VCC), U296.16 (VCC), U297.16 (VCC), U298.27 (~{WE}), U298.28 (VCC)
- net tc0: now reaches U238.15 (TC), U240.10 (CET), U240.7 (CEP)
- net clk: now reaches U238.2 (CP)
- net clk: now also U240.2 (CP)
- net GND: now reaches U238.3 (D0)
- net GND: now also U237.12 (GND), U237.18 (E0), U238.4 (D1), U238.5 (D2), U238.6 (D3), U238.8 (GND), U240.3 (D0), U240.4 (D1), U240.5 (D2), U240.6 (D3), U240.8 (GND), U241.12 (GND), U241.18 (E0), C205.2, C206.2, C207.2, C208.2, C209.2, C266.2, C267.2, C268.2, U239.3 (GND), U296.1 (Ea), U296.15 (Eb), U297.1 (Ea), U297.15 (Eb), U297.8 (GND), U298.14 (GND), U298.2 (A12), U298.20 (~{CE}), U298.21 (A10), U298.22 (~{OE}), U298.23 (A11), U298.24 (A9), U298.25 (A8), U298.3 (A7), U298.4 (A6), U298.5 (A5), U298.6 (A4)
- net ~q4: now reaches U241.19 (E1)
- net ~q4: now also U239.4
- net q5: no longer names the net of U240.13 (Q1)
- net q6: no longer names the net of U240.12 (Q2)
- net q7: no longer names the net of U240.11 (Q3)
- new net A0: U296.6 (I0a)
- new net A1: U296.10 (I0b)
- new net A2: U297.6 (I0a)
- new net A3: U297.10 (I0b)
- new net B0: U296.5 (I1a)
- new net B1: U296.11 (I1b)
- new net B2: U297.5 (I1a)
- new net B3: U297.11 (I1b)
- new net C0: U296.4 (I2a)
- new net C1: U296.12 (I2b)
- new net C2: U297.4 (I2a)
- new net C3: U297.12 (I2b)
- new net W0: U296.3 (I3a)
- new net W1: U296.13 (I3b)
- new net W2: U297.3 (I3a)
- new net W3: U297.13 (I3b)
- new net d-text0: U298.11 (I/O0)
- new net d-text1: U298.12 (I/O1)
- new net d-text2: U298.13 (I/O2)
- new net d-text3: U298.15 (I/O3)
- new net d-text4: U298.16 (I/O4)
- new net d-text5: U298.17 (I/O5)
- new net d-text6: U298.18 (I/O6)
- new net d-text7: U298.19 (I/O7)
- new net regC7: U241.8 (S7)
- new net sig0: U296.7 (Za), U298.10 (A0)
- new net sig1: U296.9 (Zb), U298.9 (A1)
- new net sig2: U297.7 (Za), U298.8 (A2)
- new net sig3: U297.9 (Zb), U298.7 (A3)
- no-connect marks 0 -> 4
Other:
- added sheet mux4_8to1-0 (../../modules/mux/mux-74xx/mux4_8to1.kicad_sch)
- added sheet mux4_8to1-1 (../../modules/mux/mux-74xx/mux4_8to1.kicad_sch)
- added sheet mux4_8to1-2 (../../modules/mux/mux-74xx/mux4_8to1.kicad_sch)
- added sheet mux4_8to1-3 (../../modules/mux/mux-74xx/mux4_8to1.kicad_sch)

Commit message: refactor: improved global labeling and reduced ERC from 300+ to 6 power flags and minor connector in errors
Parts:
- renumbered C205 to C169, C206 to C170, C207 to C171, C208 to C172, C209 to C173, C268 to C174, C266 to C175, C267 to C176, U237 to U169, U238 to U170, U239 to U171, U240 to U172, U241 to U173, U298 to U174, U296 to U175, U297 to U176
Connections:
- net GND: now also U175.8 (GND)
- net clk renamed textclk
Other:
- added sheet display-clock (text-clk.kicad_sch)
- added sheet seg-disp0 (1-seg-display.kicad_sch)
- added sheet seg-disp1 (1-seg-display.kicad_sch)
- added sheet seg-disp10 (1-seg-display.kicad_sch)
- added sheet seg-disp11 (1-seg-display.kicad_sch)
- added sheet seg-disp12 (1-seg-display.kicad_sch)
- added sheet seg-disp13 (1-seg-display.kicad_sch)
- added sheet seg-disp14 (1-seg-display.kicad_sch)
- added sheet seg-disp15 (1-seg-display.kicad_sch)
- added sheet seg-disp16 (1-seg-display.kicad_sch)
- added sheet seg-disp17 (1-seg-display.kicad_sch)
- added sheet seg-disp18 (1-seg-display.kicad_sch)
- added sheet seg-disp19 (1-seg-display.kicad_sch)
- added sheet seg-disp20 (1-seg-display.kicad_sch)
- added sheet seg-disp21 (1-seg-display.kicad_sch)
- added sheet seg-disp22 (1-seg-display.kicad_sch)
- added sheet seg-disp23 (1-seg-display.kicad_sch)
- added sheet seg-disp24 (1-seg-display.kicad_sch)
- added sheet seg-disp25 (1-seg-display.kicad_sch)
- added sheet seg-disp26 (1-seg-display.kicad_sch)
- added sheet seg-disp27 (1-seg-display.kicad_sch)
- added sheet seg-disp28 (1-seg-display.kicad_sch)
- added sheet seg-disp29 (1-seg-display.kicad_sch)
- added sheet seg-disp3 (1-seg-display.kicad_sch)
- added sheet seg-disp30 (1-seg-display.kicad_sch)
- added sheet seg-disp31 (1-seg-display.kicad_sch)
- added sheet seg-disp32 (1-seg-display.kicad_sch)
- added sheet seg-disp4 (1-seg-display.kicad_sch)
- added sheet seg-disp5 (1-seg-display.kicad_sch)
- added sheet seg-disp6 (1-seg-display.kicad_sch)
- added sheet seg-disp7 (1-seg-display.kicad_sch)
- added sheet seg-disp8 (1-seg-display.kicad_sch)
- added sheet seg-disp9 (1-seg-display.kicad_sch)
