File: hardware/kicad/boards/01_alu/alu-32b.kicad_sch (KiCad schematic)
At the start: 71 parts, among them J1 Conn_02x06_Odd_Even, J2 Conn_02x05_Odd_Even, J3 Conn_02x04_Odd_Even, J4 Conn_02x16_Odd_Even, J5 Conn_02x16_Odd_Even, J6 Conn_02x16_Odd_Even, J7 Conn_02x16_Odd_Even, U1 74LS540, U10 74LS182, U11 74LS540, U12 74LS540, U13 74LS182, U14 74LS182, U15 74LS153, U16 74AHCT1G08, U17 74LS182, U18 74LS540, U19 74LS182, U2 74LS540, U20 74LS540, U21 74LS182, U22 74LS377, U23 74HC86, U24 74LS30, U25 74LS30, U26 74HCT00, U27 74LS540, U28 74LS377, U29 74LS30, U3 74LS182, U30 74LS30, U31 74AHC541, U32 74AHC541, U4 74LS182, U5 74LS182, U6 74LS540, U7 74LS182, U8 74LS540, U9 74LS182

Commit message: feat: designed ALU board with 0 ERC errors or warnings 🎉
Final review of logical correctness and footprints and then routing begins
Parts:
- removed C1, C11, C12, C14, C18, C19, C2, C20, C5, C6, C7, C8: 100nF, Capacitor_SMD:C_0805_2012Metric, symbol Device:C
- removed C28, C32: C, Capacitor_SMD:C_0805_2012Metric, symbol Device:C
- removed J2: Conn_02x05_Odd_Even, Connector_PinHeader_2.54mm:PinHeader_2x05_P2.54mm_Vertical, symbol Connector_Generic:Conn_02x05_Odd_Even
- removed J3: Conn_02x04_Odd_Even, Connector_PinHeader_2.54mm:PinHeader_2x04_P2.54mm_Vertical, symbol Connector_Generic:Conn_02x04_Odd_Even
- removed J4, J5, J6: Conn_02x16_Odd_Even, Connector_PinHeader_2.54mm:PinHeader_2x16_P2.54mm_Vertical, symbol Connector_Generic:Conn_02x16_Odd_Even
- removed J7: Conn_02x16_Odd_Even, Connector_PinSocket_2.54mm:PinSocket_2x16_P2.54mm_Vertical, symbol Connector_Generic:Conn_02x16_Odd_Even
- removed U1, U11, U12, U18, U2, U20, U6, U8: 74LS540, Package_SO:SOIC-20W_7.5x12.8mm_P1.27mm, symbol 74xx:74LS540
- removed U14, U5: 74LS182, Package_DIP:DIP-16_W7.62mm, symbol 74xx:74LS182
- removed U31, U32: 74AHC541, Package_SO:SOIC-20W_7.5x12.8mm_P1.27mm, symbol 74xx:74AHC541
- added C101, C105, C106, C110: 100nF, Capacitor_SMD:C_0805_2012Metric, symbol Device:C
- added C127, C128, C130: 100nF, Capacitor_SMD:C_0603_1608Metric, symbol Device:C
- added J101, J102, J105: Conn_02x16_Counter_Clockwise, Connector_PinHeader_2.54mm:PinHeader_2x16_P2.54mm_Vertical, symbol Connector_Generic:Conn_02x16_Counter_Clockwise
- added J104: Conn_02x04_Odd_Even, Connector_PinHeader_2.54mm:PinHeader_2x04_P2.54mm_Vertical, symbol Connector_Generic:Conn_02x04_Odd_Even
- added J106: Conn_02x16_Counter_Clockwise, Connector_PinSocket_2.54mm:PinSocket_2x16_P2.54mm_Vertical, symbol Connector_Generic:Conn_02x16_Counter_Clockwise
- added U104, U109: 74LS182, Package_DIP:DIP-16_W7.62mm, symbol 74xx:74LS182
- added U127, U129: 74AHC541, Package_SO:SOIC-20W_7.5x12.8mm_P1.27mm, symbol 74xx:74AHC541
- added U128: 74AHC1G04, Package_TO_SOT_SMD:SOT-23-5, symbol 74xGxx:74AHC1G04
- renumbered C3 to C102, C26 to C103, C9 to C104, C21 to C107, C22 to C108, C13 to C109, C25 to C111, C4 to C112, C17 to C113, C10 to C114, C15 to C115, C16 to C116, C24 to C117, C23 to C118, C27 to C119, C29 to C120, C30 to C121, C31 to C122, J1 to J103, U7 to U101, U3 to U102, U9 to U103, U28 to U105, U19 to U106, U21 to U107, U13 to U108, U22 to U110, U27 to U111, U4 to U112, U17 to U113, U10 to U114, U23 to U115, U24 to U116, U26 to U117, U25 to U118, U15 to U119, U29 to U120, U30 to U121, U16 to U122
Connections:
- net GND: now also C101.1, C105.1, C106.1, C110.1, C127.1, C128.1, C130.1, J104.2 (Pin_2), J104.4 (Pin_4), J104.6 (Pin_6), J104.8 (Pin_8), U104.8 (GND), U109.8 (GND), U127.10 (GND), U128.3 (GND), U129.10 (GND); no longer U119.1 (Ea)
- net VCC: now also C101.2, C105.2, C106.2, C110.2, C127.2, C128.2, C130.2, J104.1 (Pin_1), J104.3 (Pin_3), J104.5 (Pin_5), J104.7 (Pin_7), U104.16 (VCC), U109.16 (VCC), U127.20 (VCC), U128.5 (VCC), U129.20 (VCC)
- net g-out-0: now also U104.10 (G)
- net g-out-2: now also U109.10 (G)
- net gb0: now also U104.3 (G0)
- net gb1: now also U104.1 (G1)
- net gb10: now also U109.14 (G2)
- net gb11: now also U109.5 (G3)
- net gb2: now also U104.14 (G2)
- net gb3: now also U104.5 (G3)
- net gb8: now also U109.3 (G0)
- net gb9: now also U109.1 (G1)
- net p-out-0: now also U104.7 (P)
- net p-out-2: now also U109.7 (P)
- net pb0: now also U104.4 (P0)
- net pb1: now also U104.2 (P1)
- net pb10: now also U109.15 (P2)
- net pb11: now also U109.6 (P3)
- net pb2: now also U104.15 (P2)
- net pb3: now also U104.6 (P3)
- net pb8: now also U109.4 (P0)
- net pb9: now also U109.2 (P1)
- net c0 renamed C0
- net C0: now also J105.1 (Pin_1)
- net ceff0 renamed Ceff0
- net Ceff0: now also U104.13 (Cn)
- net cin-sel renamed CIN-SEL
- net CIN-SEL: now also U127.1 (G1), U127.19 (G2), U128.2
- net cout12 renamed COUT12
- net cout13 renamed COUT13
- net cout14 renamed COUT14
- net cout15 renamed COUT15
- net cout16 renamed COUT16
- net cout17 renamed COUT17
- net cout18 renamed COUT18
- net cout19 renamed COUT19
- net cout20 renamed COUT20
- net cout21 renamed COUT21
- net cout22 renamed COUT22
- net cout23 renamed COUT23
- net cout24 renamed COUT24
- net cout25 renamed COUT25
- net cout26 renamed COUT26
- net cout27 renamed COUT27
- net cout28 renamed COUT28
- net cout29 renamed COUT29
- net cout30 renamed COUT30
- net cout31 renamed COUT31
- net cout32 renamed COUT32
- net cout4 renamed COUT4
- net COUT4: now also U127.5 (A3)
- net cout5 renamed COUT5
- net COUT5: now also U127.6 (A4)
- net cout6 renamed COUT6
- net COUT6: now also U127.7 (A5)
- net cout7 renamed COUT7
- net COUT7: now also U127.8 (A6)
- net cout8 renamed COUT8
- net COUT8: now also U109.13 (Cn)
- net gt-sign renamed GT-SIGN
- net gte-sign renamed GTE-SIGN
- net lt-sign renamed LT-SIGN
- net lte-sign renamed LTE-SIGN
- net nand0: no longer names the net of U116.8, U117.1
- net nand1: no longer names the net of U117.2, U118.8
- net nand2: no longer names the net of U117.4, U120.8
- net nand3: no longer names the net of U117.5, U121.8
- net nout renamed OUT31
- net OUT31: now also J106.32 (Pin_32)
- net out0 renamed OUT0
- net OUT0: now also J106.1 (Pin_1)
- net out1 renamed OUT1
- net OUT1: now also J106.2 (Pin_2)
- net out10 renamed OUT18
- net OUT18: now also J106.19 (Pin_19)
- net out11 renamed OUT19
- net OUT19: now also J106.20 (Pin_20)
- net out12 renamed OUT20
- net OUT20: now also J106.21 (Pin_21)
- net out13 renamed OUT21
- net OUT21: now also J106.22 (Pin_22)
- net out14 renamed OUT22
- net OUT22: now also J106.23 (Pin_23)
- net out15 renamed OUT23
- net OUT23: now also J106.24 (Pin_24)
- net out16 renamed OUT8
- net OUT8: now also J106.9 (Pin_9)
- net out17 renamed OUT9
- net OUT9: now also J106.10 (Pin_10)
- net out18 renamed OUT10
- net OUT10: now also J106.11 (Pin_11)
- net out19 renamed OUT11
- net OUT11: now also J106.12 (Pin_12)
- net out2 renamed OUT2
- net OUT2: now also J106.3 (Pin_3)
- net out20 renamed OUT12
- net OUT12: now also J106.13 (Pin_13)
- net out21 renamed OUT13
- net OUT13: now also J106.14 (Pin_14)
- net out22 renamed OUT14
- net OUT14: now also J106.15 (Pin_15)
- net out23 renamed OUT15
- net OUT15: now also J106.16 (Pin_16)
- net out24 renamed OUT24
- net OUT24: now also J106.25 (Pin_25)
- net out25 renamed OUT25
- net OUT25: now also J106.26 (Pin_26)
- net out26 renamed OUT26
- net OUT26: now also J106.27 (Pin_27)
- net out27 renamed OUT27
- net OUT27: now also J106.28 (Pin_28)
- net out28 renamed OUT28
- net OUT28: now also J106.29 (Pin_29)
- net out29 renamed OUT29
- net OUT29: now also J106.30 (Pin_30)
- net out3 renamed OUT3
- net OUT3: now also J106.4 (Pin_4)
- net out30 renamed OUT30
- net OUT30: now also J106.31 (Pin_31)
- net out4 renamed OUT4
- net OUT4: now also J106.5 (Pin_5)
- net out5 renamed OUT5
- net OUT5: now also J106.6 (Pin_6)
- net out6 renamed OUT6
- net OUT6: now also J106.7 (Pin_7)
- net out7 renamed OUT7
- net OUT7: now also J106.8 (Pin_8)
- net out8 renamed OUT16
- net OUT16: now also J106.17 (Pin_17)
- net out9 renamed OUT17
- net OUT17: now also J106.18 (Pin_18)
- net sys-clk renamed SYS-CLK
- net vout renamed VOUT
- net zout renamed ZOUT
- net ~cout renamed ~COUT
- net ~nout renamed ~NOUT
- net ~vout renamed ~VOUT
- net ~zout renamed ~ZOUT
- new net: U128.4, U129.1 (G1), U129.19 (G2)
- new net A0: J101.1 (Pin_1)
- new net A1: J101.2 (Pin_2)
- new net A10: J101.11 (Pin_11)
- new net A11: J101.12 (Pin_12)
- new net A12: J101.13 (Pin_13)
- new net A13: J101.14 (Pin_14)
- new net A14: J101.15 (Pin_15)
- new net A15: J101.16 (Pin_16)
- new net A16: J101.17 (Pin_17)
- new net A17: J101.18 (Pin_18)
- new net A18: J101.19 (Pin_19)
- new net A19: J101.20 (Pin_20)
- new net A2: J101.3 (Pin_3)
- new net A20: J101.21 (Pin_21)
- new net A21: J101.22 (Pin_22)
- new net A22: J101.23 (Pin_23)
- new net A23: J101.24 (Pin_24)
- new net A24: J101.25 (Pin_25)
- new net A25: J101.26 (Pin_26)
- new net A26: J101.27 (Pin_27)
- new net A27: J101.28 (Pin_28)
- new net A28: J101.29 (Pin_29)
- new net A29: J101.30 (Pin_30)
- new net A3: J101.4 (Pin_4)
- new net A30: J101.31 (Pin_31)
- new net A31: J101.32 (Pin_32)
- new net A4: J101.5 (Pin_5)
- new net A5: J101.6 (Pin_6)
- new net A6: J101.7 (Pin_7)
- new net A7: J101.8 (Pin_8)
- new net A8: J101.9 (Pin_9)
- new net A9: J101.10 (Pin_10)
- new net B0: J102.1 (Pin_1)
- new net B1: J102.2 (Pin_2)
- new net B10: J102.11 (Pin_11)
- new net B11: J102.12 (Pin_12)
- new net B12: J102.13 (Pin_13)
- new net B13: J102.14 (Pin_14)
- new net B14: J102.15 (Pin_15)
- new net B15: J102.16 (Pin_16)
- new net B16: J102.17 (Pin_17)
- new net B17: J102.18 (Pin_18)
- new net B18: J102.19 (Pin_19)
- new net B19: J102.20 (Pin_20)
- new net B2: J102.3 (Pin_3)
- new net B20: J102.21 (Pin_21)
- new net B21: J102.22 (Pin_22)
- new net B22: J102.23 (Pin_23)
- new net B23: J102.24 (Pin_24)
- new net B24: J102.25 (Pin_25)
- new net B25: J102.27 (Pin_27)
- new net B26: J102.26 (Pin_26)
- new net B27: J102.28 (Pin_28)
- new net B28: J102.29 (Pin_29)
- new net B29: J102.30 (Pin_30)
- new net B3: J102.4 (Pin_4)
- new net B30: J102.31 (Pin_31)
- new net B31: J102.32 (Pin_32)
- new net B4: J102.5 (Pin_5)
- new net B5: J102.6 (Pin_6)
- new net B6: J102.7 (Pin_7)
- new net B7: J102.8 (Pin_8)
- new net B8: J102.9 (Pin_9)
- new net B9: J102.10 (Pin_10)
- new net C1: J105.2 (Pin_2), U129.2 (A0)
- new net C10: J105.11 (Pin_11)
- new net C11: J105.12 (Pin_12)
- new net C12: J105.13 (Pin_13)
- new net C13: J105.14 (Pin_14)
- new net C14: J105.15 (Pin_15)
- new net C15: J105.16 (Pin_16)
- new net C16: J105.17 (Pin_17)
- new net C17: J105.18 (Pin_18)
- new net C18: J105.19 (Pin_19)
- new net C19: J105.20 (Pin_20)
- new net C2: J105.3 (Pin_3), U129.3 (A1)
- new net C20: J105.21 (Pin_21)
- new net C21: J105.22 (Pin_22)
- new net C22: J105.23 (Pin_23)
- new net C23: J105.24 (Pin_24)
- new net C24: J105.25 (Pin_25)
- new net C25: J105.26 (Pin_26)
- new net C26: J105.27 (Pin_27)
- new net C27: J105.28 (Pin_28)
- new net C28: J105.29 (Pin_29)
- new net C29: J105.30 (Pin_30)
- new net C3: J105.4 (Pin_4), U129.4 (A2)
- new net C30: J105.31 (Pin_31)
- new net C31: J105.32 (Pin_32)
- new net C4: J105.5 (Pin_5), U129.5 (A3)
- new net C5: J105.6 (Pin_6), U129.6 (A4)
- new net C6: J105.7 (Pin_7), U129.7 (A5)
- new net C7: J105.8 (Pin_8), U129.8 (A6)
- new net C8: J105.9 (Pin_9)
- new net C9: J105.10 (Pin_10)
- new net COUT1: U104.12 (Cn+x), U127.2 (A0)
- new net COUT10: U109.11 (Cn+y)
- new net COUT11: U109.9 (Cn+z)
- new net COUT2: U104.11 (Cn+y), U127.3 (A1)
- new net COUT3: U104.9 (Cn+z), U127.4 (A2)
- new net COUT9: U109.12 (Cn+x)
- new net Ceff1: U127.18 (Y0), U129.18 (Y0)
- new net Ceff2: U127.17 (Y1), U129.17 (Y1)
- new net Ceff3: U127.16 (Y2), U129.16 (Y2)
- new net Ceff4: U127.15 (Y3), U129.15 (Y3)
- new net Ceff5: U127.14 (Y4), U129.14 (Y4)
- new net Ceff6: U127.13 (Y5), U129.13 (Y5)
- new net Ceff7: U127.12 (Y6), U129.12 (Y6)
- no-connect marks 23 -> 25
Other:
- sheet drive_inv32 renamed drive_inv32-0
- removed sheet drive8_2to1-0
- added sheet drive_inv32-1 (../../modules/mux/drivers_inv-74xx/drive_inv32.kicad_sch)
- sheet drive8_2to1-1 ports: added inA[7..0], inB[7..0], outY[7..0]; removed a0, a1, a2, a3, a4, a5, a6, a7, b0, b1, b2, b3, b4, b5, b6, b7, y0, y1, y2, y3, y4, y5, y6, y7
- sheet drive8_2to1-2 ports: added inA[7..0], inB[7..0], outY[7..0]; removed a0, a1, a2, a3, a4, a5, a6, a7, b0, b1, b2, b3, b4, b5, b6, b7, y0, y1, y2, y3, y4, y5, y6, y7
- sheet drive8_2to1-3 ports: added inA[7..0], inB[7..0], outY[7..0]; removed a0, a1, a2, a3, a4, a5, a6, a7, b0, b1, b2, b3, b4, b5, b6, b7, y0, y1, y2, y3, y4, y5, y6, y7
- sheet drive_inv32-0: file drive_inv32.kicad_sch -> ../../modules/mux/drivers_inv-74xx/drive_inv32.kicad_sch
- sheet drive_inv32-0 ports: added y[15..8], y[23..16], y[31..24], y[7..0], ~y[15..8], ~y[23..16], ~y[31..24], ~y[7..0]; removed none
- moved on the sheet: C102, C103, C104, C107, C108, C109, C111, C112, C113, C114, C115, C116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

Commit message: arch: added LEDs, override switches; fixed errors and warnings to 0
ready for routing after logical coherence check
Parts:
- added D1, D10, D11, D12, D13, D14, D2, D3, D4, D5, D6, D7, D8, D9: LED, LED_SMD:LED_0805_2012Metric, symbol Device:LED
- added R1, R10, R11, R12, R13, R14, R2, R3, R4, R5, R6, R8, R9: 330, Resistor_SMD:R_0603_1608Metric, symbol Device:R
- added R7: 500, Resistor_SMD:R_0603_1608Metric, symbol Device:R
- added SW1, SW10, SW11, SW12, SW2, SW3, SW4, SW5, SW6, SW7, SW8, SW9: SW_DIP_x08, Button_Switch_THT:SW_DIP_SPSTx08_Slide_9.78x22.5mm_W7.62mm_P2.54mm, symbol Switch:SW_DIP_x08
- added SW13: SW_SPDT, Button_Switch_THT:SW_Slide_SPDT_Straight_CK_OS102011MS2Q, symbol Switch:SW_SPDT
- renumbered C118 to C1, C121 to C10, C112 to C11, C122 to C12, C105 to C13, C110 to C14, C104 to C15, C107 to C16, C113 to C17, C109 to C18, C102 to C19, C115 to C2, C114 to C20, C106 to C21, C101 to C22, C111 to C23, C108 to C24, C103 to C25, C127 to C3, C117 to C4, C116 to C5, C128 to C6, C119 to C7, C130 to C8, C120 to C9, J103 to J1, J104 to J2, J101 to J3, J105 to J4, J102 to J5, J106 to J6, U115 to U1, U120 to U10, U104 to U11, U109 to U12, U112 to U13, U121 to U14, U103 to U15, U107 to U16, U113 to U17, U108 to U18, U102 to U19, U119 to U2, U114 to U20, U106 to U21, U101 to U22, U111 to U23, U110 to U24, U105 to U25, U127 to U3, U117 to U4, U122 to U5, U128 to U6, U116 to U7, U129 to U8, U118 to U9
Connections:
- net A0: now also SW2.16
- net A1: now also SW2.15
- net A10: now also SW1.14
- net A11: now also SW1.13
- net A12: now also SW1.12
- net A13: now also SW1.11
- net A14: now also SW1.10
- net A15: now also SW1.9
- net A16: now also SW7.16
- net A17: now also SW7.15
- net A18: now also SW7.14
- net A19: now also SW7.13
- net A2: now also SW2.14
- net A20: now also SW7.12
- net A21: now also SW7.11
- net A22: now also SW7.10
- net A23: now also SW7.9
- net A24: now also SW8.16
- net A25: now also SW8.15
- net A26: now also SW8.14
- net A27: now also SW8.13
- net A28: now also SW8.12
- net A29: now also SW8.11
- net A3: now also SW2.13
- net A30: now also SW8.10
- net A31: now also SW8.9
- net A4: now also SW2.12
- net A5: now also SW2.11
- net A6: now also SW2.10
- net A7: now also SW2.9
- net A8: now also SW1.16
- net A9: now also SW1.15
- net B0: now also SW4.16
- net B1: now also SW4.15
- net B10: now also SW3.14
- net B11: now also SW3.13
- net B12: now also SW3.12
- net B13: now also SW3.11
- net B14: now also SW3.10
- net B15: now also SW3.9
- net B16: now also SW9.16
- net B17: now also SW9.15
- net B18: now also SW9.14
- net B19: now also SW9.13
- net B2: now also SW4.14
- net B20: now also SW9.12
- net B21: now also SW9.11
- net B22: now also SW9.10
- net B23: now also SW9.9
- net B24: now also SW10.16
- net B25: now also SW10.14
- net B26: now also SW10.15
- net B27: now also SW10.13
- net B28: now also SW10.12
- net B29: now also SW10.11
- net B3: now also SW4.13
- net B30: now also SW10.10
- net B31: now also SW10.9
- net B4: now also SW4.12
- net B5: now also SW4.11
- net B6: now also SW4.10
- net B7: now also SW4.9
- net B8: now also SW3.16
- net B9: now also SW3.15
- net C0: now also SW6.16
- net C1: now also SW6.15
- net C10: now also SW5.14
- net C11: now also SW5.13
- net C12: now also SW5.12
- net C13: now also SW5.11
- net C14: now also SW5.10
- net C15: now also SW5.9
- net C16: now also SW11.16
- net C17: now also SW11.15
- net C18: now also SW11.14
- net C19: now also SW11.13
- net C2: now also SW6.14
- net C20: now also SW11.12
- net C21: now also SW11.11
- net C22: now also SW11.10
- net C23: now also SW11.9
- net C24: now also SW12.16
- net C25: now also SW12.15
- net C26: now also SW12.14
- net C27: now also SW12.13
- net C28: now also SW12.12
- net C29: now also SW12.11
- net C3: now also SW6.13
- net C30: now also SW12.10
- net C31: now also SW12.9
- net C4: now also SW6.12
- net C5: now also SW6.11
- net C6: now also SW6.10
- net C7: now also SW6.9
- net C8: now also SW5.16
- net C9: now also SW5.15
- net GND: now also D1.1 (K), D10.1 (K), D11.1 (K), D12.1 (K), D13.1 (K), D14.1 (K), D2.1 (K), D3.1 (K), D4.1 (K), D5.1 (K), D6.1 (K), D7.1 (K), D8.1 (K), D9.1 (K)
- net VCC: now also R14.1, SW13.2 (B), SW13.3 (C)
- net flagC: now also R10.1
- net flagGT: now also R13.1
- net flagGTE: now also R6.1; no longer J1.12 (Pin_12)
- net flagLT: now also R12.1
- net flagLTE: now also R5.1; no longer J1.10 (Pin_10)
- net flagN: now also R9.1
- net flagV: now also R11.1
- net flagZ: now also R8.1
- net ~flagC: now also R3.1; no longer J1.6 (Pin_6)
- net ~flagN: now also R2.1; no longer J1.4 (Pin_4)
- net ~flagV: now also R4.1; no longer J1.8 (Pin_8)
- net ~flagZ: now also R1.1; no longer J1.2 (Pin_2)
- new net: D2.2 (A), R2.2
- new net: D11.2 (A), R11.2
- new net: D10.2 (A), R10.2
- new net: D8.2 (A), R8.2
- new net: D7.2 (A), R7.2
- new net: D12.2 (A), R12.2
- new net: D6.2 (A), R6.2
- new net: D13.2 (A), R13.2
- new net: D9.2 (A), R9.2
- new net: D14.2 (A), R14.2
- new net: D5.2 (A), R5.2
- new net: D3.2 (A), R3.2
- new net: D1.2 (A), R1.2
- new net: D4.2 (A), R4.2
- new net iN_Mode: R7.1, SW1.1, SW1.2, SW1.3, SW1.4, SW1.5, SW1.6, SW1.7, SW1.8, SW10.1, SW10.2, SW10.3, SW10.4, SW10.5, SW10.6, SW10.7, SW10.8, SW11.1, SW11.2, SW11.3, SW11.4, SW11.5, SW11.6, SW11.7, SW11.8, SW12.1, SW12.2, SW12.3, SW12.4, SW12.5, SW12.6, SW12.7, SW12.8, SW13.1 (A), SW2.1, SW2.2, SW2.3, SW2.4, SW2.5, SW2.6, SW2.7, SW2.8, SW3.1, SW3.2, SW3.3, SW3.4, SW3.5, SW3.6, SW3.7, SW3.8, SW4.1, SW4.2, SW4.3, SW4.4, SW4.5, SW4.6, SW4.7, SW4.8, SW5.1, SW5.2, SW5.3, SW5.4, SW5.5, SW5.6, SW5.7, SW5.8, SW6.1, SW6.2, SW6.3, SW6.4, SW6.5, SW6.6, SW6.7, SW6.8, SW7.1, SW7.2, SW7.3, SW7.4, SW7.5, SW7.6, SW7.7, SW7.8, SW8.1, SW8.2, SW8.3, SW8.4, SW8.5, SW8.6, SW8.7, SW8.8, SW9.1, SW9.2, SW9.3, SW9.4, SW9.5, SW9.6, SW9.7, SW9.8
