File: hardware/kicad/boards/01_alu/alu-32b.kicad_sch (KiCad schematic)
At the start: 107 parts, among them J1 Conn_02x06_Odd_Even, J2 Conn_02x04_Odd_Even, J3 Conn_02x16_Counter_Clockwise, J4 Conn_02x16_Counter_Clockwise, J5 Conn_02x16_Counter_Clockwise, J6 Conn_02x16_Counter_Clockwise, SW1 SW_DIP_x08, SW10 SW_DIP_x08, SW11 SW_DIP_x08, SW12 SW_DIP_x08, SW13 SW_SPDT, SW2 SW_DIP_x08, SW3 SW_DIP_x08, SW4 SW_DIP_x08, SW5 SW_DIP_x08, SW6 SW_DIP_x08, SW7 SW_DIP_x08, SW8 SW_DIP_x08, SW9 SW_DIP_x08, U1 74HC86, U10 74LS30, U11 74LS182, U12 74LS182, U13 74LS182, U14 74LS30, U15 74LS182, U16 74LS182, U17 74LS182, U18 74LS182, U19 74LS182, U2 74LS153, U20 74LS182, U21 74LS182, U22 74LS182, U23 74LS540, U24 74LS377, U25 74LS377, U299 74AHCT1G08, U3 74AHC541, U300 74LS540, U301 74LS540, U302 74LS540, U303 74LS32, U304 74LS540, U5 74AHCT1G08, U6 74AHC1G04, U7 74LS30, U8 74AHC541, U9 74LS30

Commit message: design: designed and locked in pcb dimension and component placements
Parts:
- removed J3, J4, J5: Conn_02x16_Counter_Clockwise, Connector_PinHeader_2.54mm:PinHeader_2x16_P2.54mm_Vertical, symbol Connector_Generic:Conn_02x16_Counter_Clockwise
- added J3, J4, J5: Conn_02x16_Odd_Even, Connector_PinHeader_2.54mm:PinHeader_2x16_P2.54mm_Vertical, symbol Connector_Generic:Conn_02x16_Odd_Even
- U4: renamed from U303; footprint (none) -> Package_SO:SOIC-14_3.9x8.7mm_P1.27mm
- renumbered C270 to C10, C271 to C11, C10 to C12, C11 to C13, C12 to C14, C13 to C15, C14 to C16, C15 to C17, C16 to C18, C17 to C19, C273 to C20, C272 to C21, C18 to C22, C19 to C23, C20 to C24, C21 to C25, C22 to C26, C23 to C27, C24 to C28, C25 to C29, C269 to C30, U300 to U10, U301 to U11, U10 to U12, U11 to U13, U12 to U14, U13 to U15, U14 to U16, U15 to U17, U16 to U18, U304 to U19, U302 to U20, U17 to U21, U18 to U22, U19 to U23, U20 to U24, U21 to U25, U22 to U26, U23 to U27, U24 to U28, U25 to U29, U299 to U30
Connections:
- net A0: now also J3.1 (Pin_1)
- net A1: now also J3.3 (Pin_3)
- net A10: now also J3.21 (Pin_21)
- net A11: now also J3.23 (Pin_23)
- net A12: now also J3.25 (Pin_25)
- net A13: now also J3.27 (Pin_27)
- net A14: now also J3.29 (Pin_29)
- net A15: now also J3.31 (Pin_31)
- net A16: now also J3.32 (Pin_32)
- net A17: now also J3.30 (Pin_30)
- net A18: now also J3.28 (Pin_28)
- net A19: now also J3.26 (Pin_26)
- net A2: now also J3.5 (Pin_5)
- net A20: now also J3.24 (Pin_24)
- net A21: now also J3.22 (Pin_22)
- net A22: now also J3.20 (Pin_20)
- net A23: now also J3.18 (Pin_18)
- net A24: now also J3.16 (Pin_16)
- net A25: now also J3.14 (Pin_14)
- net A26: now also J3.12 (Pin_12)
- net A27: now also J3.10 (Pin_10)
- net A28: now also J3.8 (Pin_8)
- net A29: now also J3.6 (Pin_6)
- net A3: now also J3.7 (Pin_7)
- net A30: now also J3.4 (Pin_4)
- net A31: now also J3.2 (Pin_2)
- net A4: now also J3.9 (Pin_9)
- net A5: now also J3.11 (Pin_11)
- net A6: now also J3.13 (Pin_13)
- net A7: now also J3.15 (Pin_15)
- net A8: now also J3.17 (Pin_17)
- net A9: now also J3.19 (Pin_19)
- net B0: now also J5.1 (Pin_1)
- net B1: now also J5.3 (Pin_3)
- net B10: now also J5.21 (Pin_21)
- net B11: now also J5.23 (Pin_23)
- net B12: now also J5.25 (Pin_25)
- net B13: now also J5.27 (Pin_27)
- net B14: now also J5.29 (Pin_29)
- net B15: now also J5.31 (Pin_31)
- net B16: now also J5.32 (Pin_32)
- net B17: now also J5.30 (Pin_30)
- net B18: now also J5.28 (Pin_28)
- net B19: now also J5.26 (Pin_26)
- net B2: now also J5.5 (Pin_5)
- net B20: now also J5.24 (Pin_24)
- net B21: now also J5.22 (Pin_22)
- net B22: now also J5.20 (Pin_20)
- net B23: now also J5.18 (Pin_18)
- net B24: now also J5.16 (Pin_16)
- net B25: now also J5.12 (Pin_12)
- net B26: now also J5.14 (Pin_14)
- net B27: now also J5.10 (Pin_10)
- net B28: now also J5.8 (Pin_8)
- net B29: now also J5.6 (Pin_6)
- net B3: now also J5.7 (Pin_7)
- net B30: now also J5.4 (Pin_4)
- net B31: now also J5.2 (Pin_2)
- net B4: now also J5.9 (Pin_9)
- net B5: now also J5.11 (Pin_11)
- net B6: now also J5.13 (Pin_13)
- net B7: now also J5.15 (Pin_15)
- net B8: now also J5.17 (Pin_17)
- net B9: now also J5.19 (Pin_19)
- net C0: now also J4.1 (Pin_1)
- net C1: now also J4.3 (Pin_3)
- net C10: now also J4.21 (Pin_21)
- net C11: now also J4.23 (Pin_23)
- net C12: now also J4.25 (Pin_25)
- net C13: now also J4.27 (Pin_27)
- net C14: now also J4.29 (Pin_29)
- net C15: now also J4.31 (Pin_31)
- net C16: now also J4.32 (Pin_32)
- net C17: now also J4.30 (Pin_30)
- net C18: now also J4.28 (Pin_28)
- net C19: now also J4.26 (Pin_26)
- net C2: now also J4.5 (Pin_5)
- net C20: now also J4.24 (Pin_24)
- net C21: now also J4.22 (Pin_22)
- net C22: now also J4.20 (Pin_20)
- net C23: now also J4.18 (Pin_18)
- net C24: now also J4.16 (Pin_16)
- net C25: now also J4.14 (Pin_14)
- net C26: now also J4.12 (Pin_12)
- net C27: now also J4.10 (Pin_10)
- net C28: now also J4.8 (Pin_8)
- net C29: now also J4.6 (Pin_6)
- net C3: now also J4.7 (Pin_7)
- net C30: now also J4.4 (Pin_4)
- net C31: now also J4.2 (Pin_2)
- net C4: now also J4.9 (Pin_9)
- net C5: now also J4.11 (Pin_11)
- net C6: now also J4.13 (Pin_13)
- net C7: now also J4.15 (Pin_15)
- net C8: now also J4.17 (Pin_17)
- net C9: now also J4.19 (Pin_19)

Commit message: chore: refactored display logic and cleanup alu design
Parts:
- C1: renamed from C26; footprint Capacitor_SMD:C_0805_2012Metric -> Capacitor_SMD:C_0603_1608Metric
- C10: renamed from C16; footprint Capacitor_SMD:C_0805_2012Metric -> Capacitor_SMD:C_0603_1608Metric
- C11: renamed from C27; footprint Capacitor_SMD:C_0805_2012Metric -> Capacitor_SMD:C_0603_1608Metric
- C12: renamed from C13; footprint Capacitor_SMD:C_0805_2012Metric -> Capacitor_SMD:C_0603_1608Metric
- C13: renamed from C19; footprint Capacitor_SMD:C_0805_2012Metric -> Capacitor_SMD:C_0603_1608Metric
- C14: renamed from C24; footprint Capacitor_SMD:C_0805_2012Metric -> Capacitor_SMD:C_0603_1608Metric
- C15: renamed from C10; footprint Capacitor_SMD:C_0805_2012Metric -> Capacitor_SMD:C_0603_1608Metric
- C16: renamed from C21; footprint Capacitor_SMD:C_0805_2012Metric -> Capacitor_SMD:C_0603_1608Metric
- C17: renamed from C30; footprint Capacitor_SMD:C_0805_2012Metric -> Capacitor_SMD:C_0603_1608Metric
- C18: renamed from C2; footprint Capacitor_SMD:C_0805_2012Metric -> Capacitor_SMD:C_0603_1608Metric
- C19: renamed from C11; footprint Capacitor_SMD:C_0805_2012Metric -> Capacitor_SMD:C_0603_1608Metric
- C2: renamed from C23; footprint Capacitor_SMD:C_0805_2012Metric -> Capacitor_SMD:C_0603_1608Metric
- C20: footprint Capacitor_SMD:C_0805_2012Metric -> Capacitor_SMD:C_0603_1608Metric
- C21: renamed from C5; footprint Capacitor_SMD:C_0805_2012Metric -> Capacitor_SMD:C_0603_1608Metric
- C22: renamed from C4; footprint Capacitor_SMD:C_0805_2012Metric -> Capacitor_SMD:C_0603_1608Metric
- C23: renamed from C1; footprint Capacitor_SMD:C_0805_2012Metric -> Capacitor_SMD:C_0603_1608Metric
- C24: renamed from C7; footprint Capacitor_SMD:C_0805_2012Metric -> Capacitor_SMD:C_0603_1608Metric
- C25: renamed from C9; footprint Capacitor_SMD:C_0805_2012Metric -> Capacitor_SMD:C_0603_1608Metric
- C26: renamed from C12; footprint Capacitor_SMD:C_0805_2012Metric -> Capacitor_SMD:C_0603_1608Metric
- C27: renamed from C14; footprint Capacitor_SMD:C_0805_2012Metric -> Capacitor_SMD:C_0603_1608Metric
- C3: renamed from C29; footprint Capacitor_SMD:C_0805_2012Metric -> Capacitor_SMD:C_0603_1608Metric
- C4: renamed from C17; footprint Capacitor_SMD:C_0805_2012Metric -> Capacitor_SMD:C_0603_1608Metric
- C5: renamed from C15; footprint Capacitor_SMD:C_0805_2012Metric -> Capacitor_SMD:C_0603_1608Metric
- C6: renamed from C25; footprint Capacitor_SMD:C_0805_2012Metric -> Capacitor_SMD:C_0603_1608Metric
- C7: renamed from C18; footprint Capacitor_SMD:C_0805_2012Metric -> Capacitor_SMD:C_0603_1608Metric
- C8: renamed from C28; footprint Capacitor_SMD:C_0805_2012Metric -> Capacitor_SMD:C_0603_1608Metric
- C9: renamed from C22; footprint Capacitor_SMD:C_0805_2012Metric -> Capacitor_SMD:C_0603_1608Metric
- renumbered C3 to C28, C8 to C29, C6 to C30, D12 to D10, D6 to D11, D13 to D12, D14 to D13, D7 to D14, D8 to D2, D2 to D3, D9 to D4, D3 to D5, D10 to D6, D4 to D7, D11 to D8, D5 to D9, J3 to J1, J5 to J2, J1 to J3, J2 to J4, J4 to J5, R12 to R10, R6 to R11, R13 to R12, R14 to R13, R7 to R14, R8 to R2, R2 to R3, R9 to R4, R3 to R5, R10 to R6, R4 to R7, R11 to R8, R5 to R9, SW2 to SW1, SW5 to SW10, SW8 to SW11, SW10 to SW12, SW12 to SW13, SW4 to SW2, SW6 to SW3, SW7 to SW4, SW9 to SW5, SW11 to SW6, SW13 to SW7, SW1 to SW8, SW3 to SW9, U26 to U1, U28 to U10, U27 to U11, U15 to U12, U21 to U13, U24 to U14, U1 to U15, U4 to U16, U7 to U17, U12 to U18, U9 to U18, U10 to U19, U23 to U2, U30 to U21, U2 to U22, U9 to U23, U12 to U23, U16 to U24, U11 to U25, U19 to U26, U5 to U27, U3 to U28, U8 to U29, U17 to U3, U6 to U30, U13 to U4, U29 to U5, U25 to U6, U18 to U7, U22 to U8, U14 to U9
Other:
- removed sheet alu_control
- added sheet alu-control (alu-control.kicad_sch)

Commit message: schematics: designed alu into 4b slices saving several chips and "de-bloating" board of several glue and drivers
Parts:
- removed C1, C10, C12, C13, C14, C17, C18, C2, C21, C28, C29, C30, C4, C5, C6, C7, C9: 100nF, Capacitor_SMD:C_0603_1608Metric, symbol Device:C
- removed J3: Conn_02x06_Odd_Even, Connector_PinSocket_2.54mm:PinSocket_2x06_P2.54mm_Vertical, symbol Connector_Generic:Conn_02x06_Odd_Even
- removed U1, U12, U13, U14, U2, U3, U4, U6, U7, U8, U9: 74LS182, Package_DIP:DIP-16_W7.62mm, symbol 74xx:74LS182
- removed U15: 74HC86, Package_SO:SOIC-14_3.9x8.7mm_P1.27mm, symbol 74xx:74HC86
- removed U16: 74LS32, Package_SO:SOIC-14_3.9x8.7mm_P1.27mm, symbol 74xx:74LS32
- removed U17, U18, U23, U24: 74LS30, Package_SO:SOIC-14_3.9x8.7mm_P1.27mm, symbol 74xx:74LS30
- removed U21, U27: 74AHCT1G08, Package_TO_SOT_SMD:SOT-23-5, symbol 74xGxx:74AHCT1G08
- removed U22: 74LS153, Package_SO:SOIC-16_3.9x9.9mm_P1.27mm, symbol 74xx:74LS153
- removed U28, U29: 74AHC541, Package_SO:SOIC-20W_7.5x12.8mm_P1.27mm, symbol 74xx:74AHC541
- removed U30: 74AHC1G04, Package_TO_SOT_SMD:SOT-23-5, symbol 74xGxx:74AHC1G04
- added C11: 100nF, Capacitor_SMD:C_0603_1608Metric, symbol Device:C
- added J6: Conn_02x07_Odd_Even, Connector_PinHeader_2.54mm:PinHeader_2x07_P2.54mm_Vertical, symbol Connector_Generic:Conn_02x07_Odd_Even
- added U10: 74LS32, Package_SO:SOIC-14_3.9x8.7mm_P1.27mm, symbol 74xx:74LS32
- added U11, U12, U6, U7: 74LS30, Package_SO:SOIC-14_3.9x8.7mm_P1.27mm, symbol 74xx:74LS30
- added U4: 74HC86, Package_SO:SOIC-14_3.9x8.7mm_P1.27mm, symbol 74xx:74HC86
- added U5: 74LS08, Package_SO:SOIC-14_3.9x8.7mm_P1.27mm, symbol 74xx:74LS08
- renumbered C3 to C1, C24 to C10, C25 to C12, C26 to C13, C27 to C14, C8 to C2, C11 to C3, C15 to C4, C16 to C5, C19 to C6, C20 to C7, C22 to C8, C23 to C9, J4 to J3, J5 to J4, J6 to J5, U5 to U1, U25 to U13, U26 to U14, U10 to U2, U11 to U3, U19 to U8, U20 to U9
Connections:
- net COUT32: now also U5.5
- net GND: now also C11.1, U10.7 (GND), U11.7 (GND), U12.7 (GND), U4.7 (GND), U5.7 (GND), U6.7 (GND), U7.7 (GND); no longer U2.13 (D4), U2.14 (D5)
- net GT-SIGN: now also U5.11
- net GTE-SIGN: now also U5.12
- net LT-SIGN: now also U4.8
- net OUT31: now also U4.9
- net VCC: now also C11.2, U10.14 (VCC), U11.14 (VCC), U12.14 (VCC), U4.14 (VCC), U5.14 (VCC), U6.14 (VCC), U7.14 (VCC)
- net VOUT: now also U4.10, U5.3
- net flagC: now also J6.5 (Pin_5)
- net flagGT: now also J6.11 (Pin_11)
- net flagGTE: now also J6.12 (Pin_12)
- net flagLT: now also J6.9 (Pin_9)
- net flagLTE: now also J6.10 (Pin_10)
- net flagN: now also J6.3 (Pin_3)
- net flagV: now also J6.7 (Pin_7)
- net flagZ: now also J6.1 (Pin_1)
- net ~ZOUT: now also U10.6, U5.13, U5.4
- net ~flagC: now also J6.6 (Pin_6)
- net ~flagN: now also J6.4 (Pin_4)
- net ~flagV: now also J6.8 (Pin_8)
- net ~flagZ: now also J6.2 (Pin_2)
- net at U13.11 (Y7): now also U11.12
- net at U13.12 (Y6): now also U11.11
- net at U13.13 (Y5): now also U11.6
- net at U13.14 (Y4): now also U11.5
- net at U13.15 (Y3): now also U11.4
- net at U13.16 (Y2): now also U11.3
- net at U13.17 (Y1): now also U11.2
- net at U13.18 (Y0): now also U11.1
- net flagGT-unsign: now reaches U2.12 (Q4)
- net flagGT-unsign: now also J6.13 (Pin_13)
- net flagLTE-unsign: now reaches U2.15 (Q5)
- net flagLTE-unsign: now also J6.14 (Pin_14)
- net at U9.18 (Y0): now also U7.1
- net at U9.12 (Y6): now also U7.11
- net at U9.11 (Y7): now also U7.12
- net at U9.17 (Y1): now also U7.2
- net at U9.16 (Y2): now also U7.3
- net at U9.15 (Y3): now also U7.4
- net at U9.14 (Y4): now also U7.5
- net at U9.13 (Y5): now also U7.6
- net at U14.11 (Y7): now also U12.12
- net at U14.12 (Y6): now also U12.11
- net at U14.13 (Y5): now also U12.6
- net at U14.14 (Y4): now also U12.5
- net at U14.15 (Y3): now also U12.4
- net at U14.16 (Y2): now also U12.3
- net at U14.17 (Y1): now also U12.2
- net at U14.18 (Y0): now also U12.1
- net LTE-UNSIGN: now reaches U3.11 (Y7)
- net LTE-UNSIGN: now also U2.14 (D5)
- net GT-UNSIGN: now reaches U3.9 (A7)
- net GT-UNSIGN: now also U2.13 (D4), U5.6
- net at U8.11 (Y7): now also U6.12
- net at U8.12 (Y6): now also U6.11
- net at U8.13 (Y5): now also U6.6
- net at U8.14 (Y4): now also U6.5
- net at U8.15 (Y3): now also U6.4
- net at U8.16 (Y2): now also U6.3
- net at U8.17 (Y1): now also U6.2
- net at U8.18 (Y0): now also U6.1
- new net: U10.10, U12.8
- new net: U10.5, U10.8
- new net: U10.9, U11.8
- new net: U10.1, U7.8
- new net: U10.2, U6.8
- new net: U10.3, U10.4
- new net: U4.3, U5.1
- new net: U4.6, U5.2
- new net AEFF31: U4.1
- new net BEFF31: U4.5
- new net SUM31: U4.2, U4.4
- no-connect marks 29 -> 33
Other:
- removed sheet alu-8b-0
- removed sheet alu-8b-1
- removed sheet alu-8b-2
- removed sheet alu-8b-3
- removed sheet display
- removed sheet drive8_2to1-1
- removed sheet drive8_2to1-2
- removed sheet drive8_2to1-3
- removed sheet drive_inv32-0
- removed sheet drive_inv32-1
- added sheet alu-4b-0 (alu-4b.kicad_sch)
- added sheet alu-4b-1 (alu-4b.kicad_sch)
- added sheet alu-4b-2 (alu-4b.kicad_sch)
- added sheet alu-4b-3 (alu-4b.kicad_sch)
- added sheet alu-4b-4 (alu-4b.kicad_sch)
- added sheet alu-4b-5 (alu-4b.kicad_sch)
- added sheet alu-4b-6 (alu-4b.kicad_sch)
- added sheet alu-4b-7 (alu-4b.kicad_sch)

Commit message: checkpoint: placed components for optimized routing on alu-32b board pcb
Parts:
- removed C1, C10, C11, C12, C13, C14, C2, C3, C4, C5, C6, C7, C8, C9: 100nF, Capacitor_SMD:C_0603_1608Metric, symbol Device:C
- removed D1, D10, D11, D12, D2, D3, D4, D5, D6, D7, D8, D9: LED, LED_SMD:LED_0805_2012Metric, symbol Device:LED
- removed J6: Conn_02x07_Odd_Even, Connector_PinHeader_2.54mm:PinHeader_2x07_P2.54mm_Vertical, symbol Connector_Generic:Conn_02x07_Odd_Even
- removed R1, R10, R11, R12, R2, R3, R4, R5, R6, R7, R8, R9: 330, Resistor_SMD:R_0603_1608Metric, symbol Device:R
- removed U1, U2: 74LS377, Package_SO:SOIC-20W_7.5x12.8mm_P1.27mm, symbol 74xx:74LS377
- removed U10: 74LS32, Package_SO:SOIC-14_3.9x8.7mm_P1.27mm, symbol 74xx:74LS32
- removed U11, U12, U6, U7: 74LS30, Package_SO:SOIC-14_3.9x8.7mm_P1.27mm, symbol 74xx:74LS30
- removed U13, U14, U3, U8, U9: 74LS540, Package_SO:SOIC-20W_7.5x12.8mm_P1.27mm, symbol 74xx:74LS540
- removed U4: 74HC86, Package_SO:SOIC-14_3.9x8.7mm_P1.27mm, symbol 74xx:74HC86
- removed U5: 74LS08, Package_SO:SOIC-14_3.9x8.7mm_P1.27mm, symbol 74xx:74LS08
- added RN1, RN10, RN11, RN12, RN2, RN3, RN4, RN5, RN6, RN7, RN8, RN9: R_Network08, Resistor_THT:R_Array_SIP9, symbol Device:R_Network08
Connections:
- net A0: now also RN4.2 (R1)
- net A1: now also RN4.3 (R2)
- net A10: now also RN3.7 (R6)
- net A11: now also RN3.6 (R5)
- net A12: now also RN3.5 (R4)
- net A13: now also RN3.4 (R3)
- net A14: now also RN3.3 (R2)
- net A15: now also RN3.2 (R1)
- net A16: now also RN2.2 (R1)
- net A17: now also RN2.3 (R2)
- net A18: now also RN2.4 (R3)
- net A19: now also RN2.5 (R4)
- net A2: now also RN4.4 (R3)
- net A20: now also RN2.6 (R5)
- net A21: now also RN2.7 (R6)
- net A22: now also RN2.8 (R7)
- net A23: now also RN2.9 (R8)
- net A24: now also RN1.9 (R8)
- net A25: now also RN1.8 (R7)
- net A26: now also RN1.7 (R6)
- net A27: now also RN1.6 (R5)
- net A28: now also RN1.5 (R4)
- net A29: now also RN1.4 (R3)
- net A3: now also RN4.5 (R4)
- net A30: now also RN1.3 (R2)
- net A31: now also RN1.2 (R1)
- net A4: now also RN4.6 (R5)
- net A5: now also RN4.7 (R6)
- net A6: now also RN4.8 (R7)
- net A7: now also RN4.9 (R8)
- net A8: now also RN3.9 (R8)
- net A9: now also RN3.8 (R7)
- net B0: now also RN5.2 (R1)
- net B1: now also RN5.3 (R2)
- net B10: now also RN6.7 (R6)
- net B11: now also RN6.6 (R5)
- net B12: now also RN6.5 (R4)
- net B13: now also RN6.4 (R3)
- net B14: now also RN6.3 (R2)
- net B15: now also RN6.2 (R1)
- net B16: now also RN7.2 (R1)
- net B17: now also RN7.3 (R2)
- net B18: now also RN7.4 (R3)
- net B19: now also RN7.5 (R4)
- net B2: now also RN5.4 (R3)
- net B20: now also RN7.6 (R5)
- net B21: now also RN7.7 (R6)
- net B22: now also RN7.8 (R7)
- net B23: now also RN7.9 (R8)
- net B24: now also RN8.9 (R8)
- net B25: now also RN8.8 (R7)
- net B26: now also RN8.7 (R6)
- net B27: now also RN8.6 (R5)
- net B28: now also RN8.5 (R4)
- net B29: now also RN8.4 (R3)
- net B3: now also RN5.5 (R4)
- net B30: now also RN8.3 (R2)
- net B31: now also RN8.2 (R1)
- net B4: now also RN5.6 (R5)
- net B5: now also RN5.7 (R6)
- net B6: now also RN5.8 (R7)
- net B7: now also RN5.9 (R8)
- net B8: now also RN6.9 (R8)
- net B9: now also RN6.8 (R7)
- net C0: now also RN9.2 (R1)
- net C1: now also RN9.3 (R2)
- net C10: now also RN10.7 (R6)
- net C11: now also RN10.6 (R5)
- net C12: now also RN10.5 (R4)
- net C13: now also RN10.4 (R3)
- net C14: now also RN10.3 (R2)
- net C15: now also RN10.2 (R1)
- net C16: now also RN11.2 (R1)
- net C17: now also RN11.3 (R2)
- net C18: now also RN11.4 (R3)
- net C19: now also RN11.5 (R4)
- net C2: now also RN9.4 (R3)
- net C20: now also RN11.6 (R5)
- net C21: now also RN11.7 (R6)
- net C22: now also RN11.8 (R7)
- net C23: now also RN11.9 (R8)
- net C24: now also RN12.9 (R8)
- net C25: now also RN12.8 (R7)
- net C26: now also RN12.7 (R6)
- net C27: now also RN12.6 (R5)
- net C28: now also RN12.5 (R4)
- net C29: now also RN12.4 (R3)
- net C3: now also RN9.5 (R4)
- net C30: now also RN12.3 (R2)
- net C31: now also RN12.2 (R1)
- net C4: now also RN9.6 (R5)
- net C5: now also RN9.7 (R6)
- net C6: now also RN9.8 (R7)
- net C7: now also RN9.9 (R8)
- net C8: now also RN10.9 (R8)
- net C9: now also RN10.8 (R7)
- net GND: now also RN1.1 (common), RN10.1 (common), RN11.1 (common), RN12.1 (common), RN2.1 (common), RN3.1 (common), RN4.1 (common), RN5.1 (common), RN6.1 (common), RN7.1 (common), RN8.1 (common), RN9.1 (common)
- no-connect marks 33 -> 22
Other:
- removed sheet alu-control
