File: hardware/kicad/boards/01_alu/alu-32b.kicad_sch (KiCad schematic)
At the start: 36 parts, among them J1 Conn_02x16_Odd_Even, J2 Conn_02x16_Odd_Even, J3 Conn_02x04_Odd_Even, J4 Conn_02x16_Odd_Even, J5 Conn_02x16_Counter_Clockwise, SW1 SW_DIP_x08, SW10 SW_DIP_x08, SW11 SW_DIP_x08, SW12 SW_DIP_x08, SW13 SW_DIP_x08, SW2 SW_DIP_x08, SW3 SW_DIP_x08, SW4 SW_DIP_x08, SW5 SW_DIP_x08, SW6 SW_DIP_x08, SW7 SW_SPDT, SW8 SW_DIP_x08, SW9 SW_DIP_x08, U42 74ACT151

Commit message: feat(web): story gallery and live datapath; wire 01_alu display sheet (#27)
* chore(web): add the in-place media optimizer

* media(web): recompress plates, pcb, and gallery WebPs

* media(web): add story gallery stills and responsive WebPs

* test(web): cover story gallery LCP preload

* feat(web): retell the gallery from notebook to 07_alu

* feat(web): embed the Dual-LUT strip on the front page

* feat(web): expand playground with overview, pipe, map, and sliders

* feat(web): let mast burger attach to scroll-rail

* media: compress microcode control log still

* feat(hardware): wire display sheet into 01_alu 32-bit project

* feat(hardware): add display sheet stub for 01_alu
Parts:
- added C1, C10, C11, C12, C13, C14, C15, C17, C19, C2, C21, C23, C27, C6, C7, C8, C9: 100nF, Capacitor_SMD:C_0603_1608Metric, symbol Device:C
- added C3, C4, C5: C, Capacitor_SMD:C_0603_1608Metric, symbol Device:C
- added D1, D10, D11, D12, D2, D3, D4, D5, D6, D7, D8, D9: LED, LED_SMD:LED_0805_2012Metric, symbol Device:LED
- added J6: Conn_02x05_Odd_Even, Connector_PinHeader_2.54mm:PinHeader_2x05_P2.54mm_Vertical, symbol Connector_Generic:Conn_02x05_Odd_Even
- added J7: Conn_02x01, Connector_PinHeader_2.54mm:PinHeader_2x01_P2.54mm_Horizontal, symbol Connector_Generic:Conn_02x01
- added J8: Conn_02x07_Odd_Even, Connector_PinHeader_2.54mm:PinHeader_2x07_P2.54mm_Vertical, symbol Connector_Generic:Conn_02x07_Odd_Even
- added R1, R10, R11, R12, R2, R3, R4, R5, R6, R7, R8, R9: 330, Resistor_SMD:R_0603_1608Metric, symbol Device:R
- added RN13: R_Network04, Resistor_THT:R_Array_SIP5, symbol Device:R_Network04
- added SW14: SW_Slide_DPDT, Button_Switch_SMD:SW_DPDT_CK_JS202011JCQN, symbol Switch:SW_Slide_DPDT
- added SW15: SW_DIP_x08, Button_Switch_THT:SW_DIP_SPSTx08_Slide_9.78x22.5mm_W7.62mm_P2.54mm, symbol Switch:SW_DIP_x08
- added SW16: SW_DIP_x04, symbol Switch:SW_DIP_x04
- added U43, U45, U46, U48: 74AHC541, Package_SO:SOIC-20W_7.5x12.8mm_P1.27mm, symbol 74xx:74AHC541
- added U44, U51: KM28C64A, Package_DIP:DIP-28_W15.24mm, symbol Memory_EEPROM:KM28C64A
- added U52, U53, U54, U55: 74LS30, Package_SO:SOIC-14_3.9x8.7mm_P1.27mm, symbol 74xx:74LS30
- added U56, U58, U64, U65, U66: 74LS540, Package_SO:SOIC-20W_7.5x12.8mm_P1.27mm, symbol 74xx:74LS540
- added U61: 74LS32, Package_SO:SOIC-14_3.9x8.7mm_P1.27mm, symbol 74xx:74LS32
- added U62: 74HC86, Package_SO:SOIC-14_3.9x8.7mm_P1.27mm, symbol 74xx:74HC86
- added U63: 74LS08, Package_SO:SOIC-14_3.9x8.7mm_P1.27mm, symbol 74xx:74LS08
- added U68, U71: 74LS377, Package_SO:SOIC-20W_7.5x12.8mm_P1.27mm, symbol 74xx:74LS377
Connections:
- net AEFF31: now also U62.1
- net BEFF31: now also U62.5
- net COUT32: now also U63.5, U66.3 (A1), U71.13 (D4)
- net CSEL0: now also U48.16 (Y2)
- net CSEL1: now also U48.15 (Y3)
- net CSEL2: now also U48.14 (Y4)
- net GND: now also C1.2, C10.1, C11.1, C12.1, C13.1, C14.1, C15.1, C17.1, C19.1, C2.1, C21.1, C23.1, C27.1, C3.2, C4.1, C5.1, C6.1, C7.1, C8.1, C9.1, D1.1 (K), D10.1 (K), D11.1 (K), D12.1 (K), D2.1 (K), D3.1 (K), D4.1 (K), D5.1 (K), D6.1 (K), D7.1 (K), D8.1 (K), D9.1 (K), RN13.1 (common), SW14.3 (C), U43.10 (GND), U44.14 (GND), U44.2 (A12), U44.20 (~{CE}), U44.21 (A10), U44.22 (~{OE}), U44.23 (A11), U45.1 (G1), U45.10 (GND), U45.19 (G2), U46.1 (G1), U46.10 (GND), U46.19 (G2), U48.10 (GND), U51.14 (GND), U51.2 (A12), U51.20 (~{CE}), U51.21 (A10), U51.22 (~{OE}), U51.23 (A11), U52.7 (GND), U53.7 (GND), U54.7 (GND), U55.7 (GND), U56.1 (G1), U56.10 (GND), U56.19 (G2), U58.1 (G1), U58.10 (GND), U58.19 (G2), U61.7 (GND), U62.7 (GND), U63.7 (GND), U64.1 (G1), U64.10 (GND), U64.19 (G2), U65.1 (G1), U65.10 (GND), U65.19 (G2), U66.1 (G1), U66.10 (GND), U66.19 (G2), U68.10 (GND), U68.17 (D6), U68.18 (D7), U71.10 (GND)
- net OUT0: now also U56.2 (A0)
- net OUT1: now also U56.3 (A1)
- net OUT10: now also U58.4 (A2)
- net OUT11: now also U58.5 (A3)
- net OUT12: now also U58.6 (A4)
- net OUT13: now also U58.7 (A5)
- net OUT14: now also U58.8 (A6)
- net OUT15: now also U58.9 (A7)
- net OUT16: now also U65.2 (A0)
- net OUT17: now also U65.3 (A1)
- net OUT18: now also U65.4 (A2)
- net OUT19: now also U65.5 (A3)
- net OUT2: now also U56.4 (A2)
- net OUT20: now also U65.6 (A4)
- net OUT21: now also U65.7 (A5)
- net OUT22: now also U65.8 (A6)
- net OUT23: now also U65.9 (A7)
- net OUT24: now also U64.2 (A0)
- net OUT25: now also U64.3 (A1)
- net OUT26: now also U64.4 (A2)
- net OUT27: now also U64.5 (A3)
- net OUT28: now also U64.6 (A4)
- net OUT29: now also U64.7 (A5)
- net OUT3: now also U56.5 (A3)
- net OUT30: now also U64.8 (A6)
- net OUT31: now also U62.9, U64.9 (A7), U66.6 (A4), U71.7 (D2)
- net OUT4: now also U56.6 (A4)
- net OUT5: now also U56.7 (A5)
- net OUT6: now also U56.8 (A6)
- net OUT7: now also U56.9 (A7)
- net OUT8: now also U58.2 (A0)
- net OUT9: now also U58.3 (A1)
- net SUM31: now also U62.2, U62.4
- net VCC: now also C1.1, C10.2, C11.2, C12.2, C13.2, C14.2, C15.2, C17.2, C19.2, C2.2, C21.2, C23.2, C27.2, C3.1, C4.2, C5.2, C6.2, C7.2, C8.2, C9.2, SW14.1 (A), SW14.6 (C), U43.20 (VCC), U44.27 (~{WE}), U44.28 (VCC), U45.20 (VCC), U46.20 (VCC), U48.20 (VCC), U51.27 (~{WE}), U51.28 (VCC), U52.14 (VCC), U53.14 (VCC), U54.14 (VCC), U55.14 (VCC), U56.20 (VCC), U58.20 (VCC), U61.14 (VCC), U62.14 (VCC), U63.14 (VCC), U64.20 (VCC), U65.20 (VCC), U66.20 (VCC), U68.20 (VCC), U71.20 (VCC)
- net cin-main: now also RN13.3 (R2), SW16.6
- net flagC: now also J8.5 (Pin_5), R6.1, U71.12 (Q4)
- net flagLT: now also J8.9 (Pin_9), R10.1, U68.2 (Q0)
- net flagN: now also J8.3 (Pin_3), R4.1, U71.6 (Q2)
- net flagV: now also J8.7 (Pin_7), R8.1, U71.16 (Q6)
- net flagZ: now also J8.1 (Pin_1), R2.1, U71.2 (Q0)
- net ~flagC: now also J8.6 (Pin_6), R5.1, U71.15 (Q5)
- new net: D7.2 (A), R7.2
- new net: U48.2 (A0), U51.11 (I/O0)
- new net: U48.3 (A1), U51.12 (I/O1)
- new net: U48.4 (A2), U51.13 (I/O2)
- new net: U48.5 (A3), U51.15 (I/O3)
- new net: U48.6 (A4), U51.16 (I/O4)
- new net: U48.7 (A5), U51.17 (I/O5)
- new net: U48.8 (A6), U51.18 (I/O6)
- new net: U48.9 (A7), U51.19 (I/O7)
- new net: U62.3, U63.1
- new net: U62.6, U63.2
- new net: U52.12, U56.11 (Y7)
- new net: U52.11, U56.12 (Y6)
- new net: U52.6, U56.13 (Y5)
- new net: U52.5, U56.14 (Y4)
- new net: U52.4, U56.15 (Y3)
- new net: U52.3, U56.16 (Y2)
- new net: U52.2, U56.17 (Y1)
- new net: U52.1, U56.18 (Y0)
- new net: D10.2 (A), R10.2
- new net: D1.2 (A), R1.2
- new net: U55.8, U61.10
- new net: U61.5, U61.8
- new net: U53.8, U61.9
- new net: D3.2 (A), R3.2
- new net: U54.12, U65.11 (Y7)
- new net: U54.11, U65.12 (Y6)
- new net: U54.6, U65.13 (Y5)
- new net: U54.5, U65.14 (Y4)
- new net: U54.4, U65.15 (Y3)
- new net: U54.3, U65.16 (Y2)
- new net: U54.2, U65.17 (Y1)
- new net: U54.1, U65.18 (Y0)
- new net: J7.1 (Pin_1), J7.2 (Pin_2), U45.4 (A2), U45.5 (A3), U45.6 (A4), U45.7 (A5), U45.8 (A6), U45.9 (A7)
- new net: U43.2 (A0), U44.11 (I/O0)
- new net: U43.3 (A1), U44.12 (I/O1)
- new net: U43.4 (A2), U44.13 (I/O2)
- new net: U43.5 (A3), U44.15 (I/O3)
- new net: U43.6 (A4), U44.16 (I/O4)
- new net: U43.7 (A5), U44.17 (I/O5)
- new net: U43.8 (A6), U44.18 (I/O6)
- new net: U43.9 (A7), U44.19 (I/O7)
- new net: U53.1, U58.18 (Y0)
- new net: U53.11, U58.12 (Y6)
- new net: U53.12, U58.11 (Y7)
- new net: U53.2, U58.17 (Y1)
- new net: U53.3, U58.16 (Y2)
- new net: U53.4, U58.15 (Y3)
- new net: U53.5, U58.14 (Y4)
- new net: U53.6, U58.13 (Y5)
- new net: U55.1, U64.18 (Y0)
- new net: U55.11, U64.12 (Y6)
- new net: U55.12, U64.11 (Y7)
- new net: U55.2, U64.17 (Y1)
- new net: U55.3, U64.16 (Y2)
- new net: U55.4, U64.15 (Y3)
- new net: U55.5, U64.14 (Y4)
- new net: U55.6, U64.13 (Y5)
- new net: D11.2 (A), R11.2
- new net: D5.2 (A), R5.2
- new net: D9.2 (A), R9.2
- new net: D4.2 (A), R4.2
- new net: D8.2 (A), R8.2
- new net: J6.2 (Pin_2), U46.2 (A0)
- new net: J6.4 (Pin_4), U46.3 (A1)
- new net: J6.6 (Pin_6), U46.4 (A2)
- new net: J6.8 (Pin_8), U46.5 (A3)
- new net: J6.10 (Pin_10), U46.6 (A4)
- new net: J6.9 (Pin_9), U46.7 (A5)
- new net: J6.7 (Pin_7), U46.8 (A6)
- new net: J6.5 (Pin_5), U46.9 (A7)
- new net: J6.1 (Pin_1), U45.2 (A0)
- new net: J6.3 (Pin_3), U45.3 (A1)
- new net: D12.2 (A), R12.2
- new net: U54.8, U61.1
- new net: U52.8, U61.2
- new net: D2.2 (A), R2.2
- new net: U61.3, U61.4
- new net: D6.2 (A), R6.2
- new net ALU-OPCODE0: SW15.16, U43.18 (Y0)
- new net ALU-OPCODE1: SW15.15, U43.17 (Y1)
- new net ALU-OPCODE2: SW15.14, U43.16 (Y2)
- new net ALU-OPCODE3: SW15.13, U43.15 (Y3)
- new net ALU-OPCODE4: SW15.12, U43.14 (Y4)
- new net ALU-OPCODE5: SW15.11, U43.13 (Y5)
- new net ALU-OPCODE6: SW15.10, U43.12 (Y6)
- new net ALU-OPCODE7: SW15.9, U43.11 (Y7)
- new net Ctrl_EN: SW14.2 (B), U48.1 (G1), U48.19 (G2)
- new net GT-SIGN: U63.11, U66.8 (A6), U68.7 (D2)
- new net GT-UNSIGN: U63.6, U66.9 (A7), U68.13 (D4)
- new net GTE-SIGN: U63.12, U66.15 (Y3), U68.8 (D3)
- new net IR-OPCODE0: U44.10 (A0), U45.18 (Y0), U51.10 (A0)
- new net IR-OPCODE1: U44.9 (A1), U46.18 (Y0), U51.9 (A1)
- new net IR-OPCODE2: U44.8 (A2), U45.17 (Y1), U51.8 (A2)
- new net IR-OPCODE3: U44.7 (A3), U46.17 (Y1), U51.7 (A3)
- new net IR-OPCODE4: U44.6 (A4), U46.11 (Y7), U51.6 (A4)
- new net IR-OPCODE5: U44.5 (A5), U46.16 (Y2), U51.5 (A5)
- new net IR-OPCODE6: U44.4 (A6), U46.12 (Y6), U51.4 (A6)
- new net IR-OPCODE7: U44.3 (A7), U46.15 (Y3), U51.3 (A7)
- new net IR-OPCODE8: U44.25 (A8), U46.13 (Y5), U51.25 (A8)
- new net IR-OPCODE9: U44.24 (A9), U46.14 (Y4), U51.24 (A9)
- new net LT-SIGN: U62.8, U66.5 (A3), U68.3 (D0)
- new net LTE-SIGN: U66.12 (Y6), U68.4 (D1)
- new net LTE-UNSIGN: U66.11 (Y7), U68.14 (D5)
- new net Override: U43.1 (G1), U43.19 (G2)
- new net SW_EN: SW14.5 (B), SW15.1, SW15.2, SW15.3, SW15.4, SW15.5, SW15.6, SW15.7, SW15.8
- new net SYS-CLK: U45.11 (Y7), U45.12 (Y6), U45.13 (Y5), U45.14 (Y4), U45.15 (Y3), U45.16 (Y2), U68.11 (CP), U71.11 (CP)
- new net VOUT: U62.10, U63.3, U66.4 (A2), U71.17 (D6)
- new net ZOUT: U66.18 (Y0), U71.3 (D0)
- new net binv: RN13.4 (R3), SW16.7, U48.17 (Y1)
- new net bsel: RN13.5 (R4), SW16.8, U48.18 (Y0)
- new net flagGT: J8.11 (Pin_11), R12.1, U68.6 (Q2)
- new net flagGT-unsign: J8.13 (Pin_13), U68.12 (Q4)
- new net flagGTE: J8.12 (Pin_12), R11.1, U68.9 (Q3)
- new net flagLTE: J8.10 (Pin_10), R9.1, U68.5 (Q1)
- new net flagLTE-unsign: J8.14 (Pin_14), U68.15 (Q5)
- new net flagWE: RN13.2 (R1), SW16.5, U48.13 (Y5), U66.7 (A5)
- new net ~COUT: U66.17 (Y1), U71.14 (D5)
- new net ~NOUT: U66.14 (Y4), U71.8 (D3)
- new net ~VOUT: U66.16 (Y2), U71.18 (D7)
- new net ~ZOUT: U61.6, U63.13, U63.4, U66.2 (A0), U71.4 (D1)
- new net ~flagN: J8.4 (Pin_4), R3.1, U71.9 (Q3)
- new net ~flagV: J8.8 (Pin_8), R7.1, U71.19 (Q7)
- new net ~flagWE: U66.13 (Y5), U68.1 (~{E}), U71.1 (~{E})
- new net ~flagZ: J8.2 (Pin_2), R1.1, U71.5 (Q1)
- no-connect marks 23 -> 37
Other:
- added sheet display (untitled.kicad_sch)
- title: Tomato32 ALU -> Tomato ALU
- moved on the sheet: RN4, RN5, RN9, SW7
