File: hardware/kicad/boards/01_alu/alu-32b.kicad_pcb (KiCad board)
At the start: 2 copper layers, 895 parts, among them J1 Conn_02x06_Odd_Even, J2 Conn_02x05_Odd_Even, J3 Conn_02x16_Odd_Even, J4 Conn_02x16_Odd_Even, J5 Conn_02x16_Odd_Even, J6 Conn_02x16_Odd_Even, J7 Conn_02x04_Odd_Even, U1 74LS540, U10 74LS182, U100 74AHCT125, U101 74AHCT125, U102 74AHCT138, U103 74LS08, U104 74HC86, U105 74AHCT125, U106 74AHCT125, U107 74AHCT138, U108 74LS08, U109 74HC86, U11 74LS540, U110 74AHCT125, U111 74AHCT125, U112 74AHCT138, U113 74LS08, U114 74HC86, U115 74AHCT125, U116 74AHCT125, U117 74AHCT138, U118 74LS08, U119 74HC86, U12 74LS540, U120 74AHCT125, U121 74AHCT125, U122 74AHCT138, U123 74LS08, U124 74HC86, U125 74AHCT125, U126 74AHCT125, U127 74AHCT138, U128 74LS08, U129 74HC86, U13 74LS182, U130 74AHCT125, U131 74AHCT125, U132 74AHCT138, U133 74LS08, U134 74HC86, U135 74AHCT125, U136 74AHCT125, U137 74AHCT138, U138 74LS08, U139 74HC86, U14 74LS182, U140 74AHCT125, U141 74AHCT125, U142 74AHCT138, U143 74LS08, U144 74HC86, U145 74AHCT125, U146 74AHCT125, U147 74AHCT138, U148 74LS08, U149 74HC86, U15 74LS153, U150 74AHCT125, U151 74AHCT125, U152 74AHCT138, U153 KM28C64A, U154 KM28C64A, U155 74AHC541, U156 74AHC541, U157 74AHC541, U158 74AHC1G04, U159 74AHC541, U16 74AHCT1G08, U160 74AHC541, U161 74AHC1G04, U162 74AHC541, U163 74AHC541, U164 74AHC1G04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

Commit message: feat: designed ALU board with 0 ERC errors or warnings 🎉
Final review of logical correctness and footprints and then routing begins
Parts:
- removed C269: 100nF, Capacitor_SMD:C_0805_2012Metric
- removed R291, R292, R293, R294, R295, R296: 120, Resistor_SMD:R_0805_2012Metric
- removed R297: 1k, Resistor_SMD:R_0805_2012Metric
- removed R298: 10k, Resistor_SMD:R_0805_2012Metric
- removed U299: 74AHCT125, Package_SO:SOIC-14_3.9x8.7mm_P1.27mm
- removed U300: 74AHCT138, Package_SO:SOIC-16_3.9x9.9mm_P1.27mm
- added C187: 100nF, Capacitor_SMD:C_0805_2012Metric, F.Cu at (264.1, 96.6)
- added J8: Conn_02x05_Odd_Even, Connector_PinHeader_2.54mm:PinHeader_2x05_P2.54mm_Vertical, F.Cu at (172.5, -19.3)
- added R100: 120, Resistor_SMD:R_0805_2012Metric, F.Cu at (132.8, 66.4)
- added R101: 120, Resistor_SMD:R_0805_2012Metric, F.Cu at (132.8, 69.4)
- added R102: 120, Resistor_SMD:R_0805_2012Metric, F.Cu at (132.8, 72.3)
- added R103: 120, Resistor_SMD:R_0805_2012Metric, F.Cu at (132.8, 75.3)
- added R104: 120, Resistor_SMD:R_0805_2012Metric, F.Cu at (132.8, 78.2)
- added R97: 120, Resistor_SMD:R_0805_2012Metric, F.Cu at (132.8, 57.6)
- added R98: 120, Resistor_SMD:R_0805_2012Metric, F.Cu at (132.8, 60.5)
- added R99: 120, Resistor_SMD:R_0805_2012Metric, F.Cu at (132.8, 63.5)
- added U195: 74HC86, Package_SO:SOIC-14_3.9x8.7mm_P1.27mm, F.Cu at (190.5, 86.9)
- added U196: 74AHCT125, Package_SO:SOIC-14_3.9x8.7mm_P1.27mm, F.Cu at (210.4, 219.7)
- C149, C150, C151, C152: value 100nF -> C
- C153, C154, C214, C215, C216: footprint Capacitor_SMD:C_0805_2012Metric -> Capacitor_SMD:C_0603_1608Metric
- C155, C156: value C -> 100nF; footprint Capacitor_SMD:C_0805_2012Metric -> Capacitor_SMD:C_0603_1608Metric
- C162, C163, C164, C165, C166, C167, C168: footprint Capacitor_SMD:C_0603_1608Metric -> Capacitor_SMD:C_0805_2012Metric
- C246: value 100nF -> 10nF
- C251: value 10nF -> 100nF
- C28, C31: value C -> 100nF
- J1: value Conn_02x06_Odd_Even -> Conn_02x04_Odd_Even; footprint Connector_PinSocket_2.54mm:PinSocket_2x06_P2.54mm_Vertical -> Connector_PinHeader_2.54mm:PinHeader_2x04_P2.54mm_Vertical
- J2: value Conn_02x05_Odd_Even -> Conn_02x16_Counter_Clockwise; footprint Connector_PinHeader_2.54mm:PinHeader_2x05_P2.54mm_Vertical -> Connector_PinHeader_2.54mm:PinHeader_2x16_P2.54mm_Vertical
- J3, J4: value Conn_02x16_Odd_Even -> Conn_02x16_Counter_Clockwise
- J5: value Conn_02x16_Odd_Even -> Conn_02x16_Counter_Clockwise; footprint Connector_PinHeader_2.54mm:PinHeader_2x16_P2.54mm_Vertical -> Connector_PinSocket_2.54mm:PinSocket_2x16_P2.54mm_Vertical
- J6: value Conn_02x16_Odd_Even -> Conn_02x06_Odd_Even; footprint Connector_PinSocket_2.54mm:PinSocket_2x16_P2.54mm_Vertical -> Connector_PinSocket_2.54mm:PinSocket_2x06_P2.54mm_Vertical
- J7: value Conn_02x04_Odd_Even -> Conn_02x01; footprint Connector_PinHeader_2.54mm:PinHeader_2x04_P2.54mm_Vertical -> Connector_PinHeader_2.54mm:PinHeader_2x01_P2.54mm_Horizontal
- R257: value 120 -> 1k
- R258: value 120 -> 10k
- U1: value 74LS540 -> 74LS153; footprint Package_SO:SOIC-20W_7.5x12.8mm_P1.27mm -> Package_SO:SOIC-16_3.9x9.9mm_P1.27mm
- U11, U12, U6, U8: value 74LS540 -> 74LS182; footprint Package_SO:SOIC-20W_7.5x12.8mm_P1.27mm -> Package_DIP:DIP-16_W7.62mm
- U14, U17: value 74LS182 -> 74LS30; footprint Package_DIP:DIP-16_W7.62mm -> Package_SO:SOIC-14_3.9x8.7mm_P1.27mm
- U143: value 74LS08 -> 74LS540; footprint Package_SO:SOIC-14_3.9x8.7mm_P1.27mm -> Package_SO:SOIC-20W_7.5x12.8mm_P1.27mm
- U144: value 74HC86 -> 74LS540; footprint Package_SO:SOIC-14_3.9x8.7mm_P1.27mm -> Package_SO:SOIC-20W_7.5x12.8mm_P1.27mm
- U145, U146: value 74AHCT125 -> 74LS540; footprint Package_SO:SOIC-14_3.9x8.7mm_P1.27mm -> Package_SO:SOIC-20W_7.5x12.8mm_P1.27mm
- U147: value 74AHCT138 -> KM28C64A; footprint Package_SO:SOIC-16_3.9x9.9mm_P1.27mm -> Package_DIP:DIP-28_W15.24mm
- U148: value 74LS08 -> KM28C64A; footprint Package_SO:SOIC-14_3.9x8.7mm_P1.27mm -> Package_DIP:DIP-28_W15.24mm
- U149: value 74HC86 -> 74AHC541; footprint Package_SO:SOIC-14_3.9x8.7mm_P1.27mm -> Package_SO:SOIC-20W_7.5x12.8mm_P1.27mm
- U15: value 74LS153 -> 74LS30; footprint Package_SO:SOIC-16_3.9x9.9mm_P1.27mm -> Package_SO:SOIC-14_3.9x8.7mm_P1.27mm
- U150, U151: value 74AHCT125 -> 74AHC541; footprint Package_SO:SOIC-14_3.9x8.7mm_P1.27mm -> Package_SO:SOIC-20W_7.5x12.8mm_P1.27mm
- U152: value 74AHCT138 -> 74AHC541; footprint Package_SO:SOIC-16_3.9x9.9mm_P1.27mm -> Package_SO:SOIC-20W_7.5x12.8mm_P1.27mm
- U153: value KM28C64A -> 74AHC541; footprint Package_DIP:DIP-28_W15.24mm -> Package_SO:SOIC-20W_7.5x12.8mm_P1.27mm
- U154: value KM28C64A -> 74AHC1G04; footprint Package_DIP:DIP-28_W15.24mm -> Package_TO_SOT_SMD:SOT-23-5
- U157, U160: value 74AHC541 -> 74AHC1G04; footprint Package_SO:SOIC-20W_7.5x12.8mm_P1.27mm -> Package_TO_SOT_SMD:SOT-23-5
- U158, U161: value 74AHC1G04 -> 74AHC541; footprint Package_TO_SOT_SMD:SOT-23-5 -> Package_SO:SOIC-20W_7.5x12.8mm_P1.27mm
- U16: value 74AHCT1G08 -> 74LS30; footprint Package_TO_SOT_SMD:SOT-23-5 -> Package_SO:SOIC-14_3.9x8.7mm_P1.27mm
- U162, U166: value 74AHC541 -> 74LS154; footprint Package_SO:SOIC-20W_7.5x12.8mm_P1.27mm -> Package_SO:SOIC-24W_7.5x15.4mm_P1.27mm
- U163, U165: value 74AHC541 -> 74LS163; footprint Package_SO:SOIC-20W_7.5x12.8mm_P1.27mm -> Package_SO:SOIC-16_3.9x9.9mm_P1.27mm
- U167: value 74AHC1G04 -> KM28C64A; footprint Package_TO_SOT_SMD:SOT-23-5 -> Package_DIP:DIP-28_W15.24mm
- U168: value 74AHC541 -> 74LS153; footprint Package_SO:SOIC-20W_7.5x12.8mm_P1.27mm -> Package_SO:SOIC-16_3.9x9.9mm_P1.27mm
- U169: value 74LS154 -> 74LS153; footprint Package_SO:SOIC-24W_7.5x15.4mm_P1.27mm -> Package_SO:SOIC-16_3.9x9.9mm_P1.27mm
- U170, U172: value 74LS163 -> 74LS540; footprint Package_SO:SOIC-16_3.9x9.9mm_P1.27mm -> Package_SO:SOIC-20W_7.5x12.8mm_P1.27mm
- U171: value 74AHC1G04 -> 74LS540; footprint Package_TO_SOT_SMD:SOT-23-5 -> Package_SO:SOIC-20W_7.5x12.8mm_P1.27mm
- U173: value 74LS154 -> 74LS540; footprint Package_SO:SOIC-24W_7.5x15.4mm_P1.27mm -> Package_SO:SOIC-20W_7.5x12.8mm_P1.27mm
- U174: value KM28C64A -> 74LS08; footprint Package_DIP:DIP-28_W15.24mm -> Package_SO:SOIC-14_3.9x8.7mm_P1.27mm
- U175: value 74LS153 -> 74HC86; footprint Package_SO:SOIC-16_3.9x9.9mm_P1.27mm -> Package_SO:SOIC-14_3.9x8.7mm_P1.27mm
- U176: value 74LS153 -> 74AHCT125; footprint Package_SO:SOIC-16_3.9x9.9mm_P1.27mm -> Package_SO:SOIC-14_3.9x8.7mm_P1.27mm
- U177: value 74LS08 -> 74AHCT125
- U178: value 74HC86 -> 74AHCT138; footprint Package_SO:SOIC-14_3.9x8.7mm_P1.27mm -> Package_SO:SOIC-16_3.9x9.9mm_P1.27mm
- U179, U189, U199, U209, U28: value 74LS377 -> 74LS08; footprint Package_SO:SOIC-20W_7.5x12.8mm_P1.27mm -> Package_SO:SOIC-14_3.9x8.7mm_P1.27mm
- U18: value 74LS540 -> 74HCT00; footprint Package_SO:SOIC-20W_7.5x12.8mm_P1.27mm -> Package_SO:SOIC-14_3.9x8.7mm_P1.27mm
- U180, U190, U200, U210: value HDSP-A153 -> 74HC86; footprint Display_7Segment:HDSP-A151 -> Package_SO:SOIC-14_3.9x8.7mm_P1.27mm
- U181, U187, U191, U197, U201, U207, U211: value 74LS377 -> 74AHCT125; footprint Package_SO:SOIC-20W_7.5x12.8mm_P1.27mm -> Package_SO:SOIC-14_3.9x8.7mm_P1.27mm
- U182, U186, U192, U202, U206, U212: value HDSP-A153 -> 74AHCT125; footprint Display_7Segment:HDSP-A151 -> Package_SO:SOIC-14_3.9x8.7mm_P1.27mm
- U183, U193, U203, U213: value 74LS377 -> 74AHCT138; footprint Package_SO:SOIC-20W_7.5x12.8mm_P1.27mm -> Package_SO:SOIC-16_3.9x9.9mm_P1.27mm
- U184, U194, U204: value HDSP-A153 -> 74LS08; footprint Display_7Segment:HDSP-A151 -> Package_SO:SOIC-14_3.9x8.7mm_P1.27mm
- U185, U205: value 74LS377 -> 74HC86; footprint Package_SO:SOIC-20W_7.5x12.8mm_P1.27mm -> Package_SO:SOIC-14_3.9x8.7mm_P1.27mm
- U188, U198, U208: value HDSP-A153 -> 74AHCT138; footprint Display_7Segment:HDSP-A151 -> Package_SO:SOIC-16_3.9x9.9mm_P1.27mm
- U19: value 74LS182 -> 74LS377; footprint Package_DIP:DIP-16_W7.62mm -> Package_SO:SOIC-20W_7.5x12.8mm_P1.27mm
- U2: value 74LS540 -> 74AHCT1G08; footprint Package_SO:SOIC-20W_7.5x12.8mm_P1.27mm -> Package_TO_SOT_SMD:SOT-23-5
- U20: value 74LS540 -> 74LS377
- U21: value 74LS182 -> 74HC86; footprint Package_DIP:DIP-16_W7.62mm -> Package_SO:SOIC-14_3.9x8.7mm_P1.27mm
- U214, U216: value HDSP-A153 -> 74AHC541; footprint Display_7Segment:HDSP-A151 -> Package_SO:SOIC-20W_7.5x12.8mm_P1.27mm
- U215: value 74LS377 -> 74AHC1G04; footprint Package_SO:SOIC-20W_7.5x12.8mm_P1.27mm -> Package_TO_SOT_SMD:SOT-23-5
- U22: value 74LS377 -> 74LS540
- U23: value 74HC86 -> 74LS08
- U24, U29: value 74LS30 -> 74HC86
- U245, U247, U249, U251, U253, U255, U257, U259: value 74LS151 -> 74LS377; footprint Package_SO:SOIC-16_3.9x9.9mm_P1.27mm -> Package_SO:SOIC-20W_7.5x12.8mm_P1.27mm
- U246, U248, U250, U252, U254, U256, U258, U260: value 74LS151 -> HDSP-A153; footprint Package_SO:SOIC-16_3.9x9.9mm_P1.27mm -> Display_7Segment:HDSP-A151
- U25, U30: value 74LS30 -> 74AHCT125
- U26: value 74HCT00 -> 74AHCT125
- U261, U267, U271, U277, U281: value 74AHCT125 -> 74LS377; footprint Package_SO:SOIC-14_3.9x8.7mm_P1.27mm -> Package_SO:SOIC-20W_7.5x12.8mm_P1.27mm
- U262, U266, U272, U282: value 74AHCT125 -> HDSP-A153; footprint Package_SO:SOIC-14_3.9x8.7mm_P1.27mm -> Display_7Segment:HDSP-A151
- U263, U273: value 74AHCT138 -> 74LS377; footprint Package_SO:SOIC-16_3.9x9.9mm_P1.27mm -> Package_SO:SOIC-20W_7.5x12.8mm_P1.27mm
- U264: value 74LS08 -> HDSP-A153; footprint Package_SO:SOIC-14_3.9x8.7mm_P1.27mm -> Display_7Segment:HDSP-A151
- U265: value 74HC86 -> 74LS377; footprint Package_SO:SOIC-14_3.9x8.7mm_P1.27mm -> Package_SO:SOIC-20W_7.5x12.8mm_P1.27mm
- U268, U278: value 74AHCT138 -> HDSP-A153; footprint Package_SO:SOIC-16_3.9x9.9mm_P1.27mm -> Display_7Segment:HDSP-A151
- U269, U279: value 74LS08 -> 74LS377; footprint Package_SO:SOIC-14_3.9x8.7mm_P1.27mm -> Package_SO:SOIC-20W_7.5x12.8mm_P1.27mm
- U27: value 74LS540 -> 74AHCT138; footprint Package_SO:SOIC-20W_7.5x12.8mm_P1.27mm -> Package_SO:SOIC-16_3.9x9.9mm_P1.27mm
- U270, U275, U280: value 74HC86 -> HDSP-A153; footprint Package_SO:SOIC-14_3.9x8.7mm_P1.27mm -> Display_7Segment:HDSP-A151
- U274: value 74LS08 -> ICM7555xB; footprint Package_SO:SOIC-14_3.9x8.7mm_P1.27mm -> Package_SO:SOIC-8_3.9x4.9mm_P1.27mm
- U276: value 74AHCT125 -> 74HCT541; footprint Package_SO:SOIC-14_3.9x8.7mm_P1.27mm -> Package_SO:SOIC-20W_7.5x12.8mm_P1.27mm
- U283, U290, U295: value 74AHCT138 -> 74LS151
- U284: value ICM7555xB -> 74LS151; footprint Package_SO:SOIC-8_3.9x4.9mm_P1.27mm -> Package_SO:SOIC-16_3.9x9.9mm_P1.27mm
- U285: value 74HCT541 -> 74LS151; footprint Package_SO:SOIC-20W_7.5x12.8mm_P1.27mm -> Package_SO:SOIC-16_3.9x9.9mm_P1.27mm
- U286, U291, U296: value 74LS08 -> 74LS151; footprint Package_SO:SOIC-14_3.9x8.7mm_P1.27mm -> Package_SO:SOIC-16_3.9x9.9mm_P1.27mm
- U287, U292, U297: value 74HC86 -> 74LS151; footprint Package_SO:SOIC-14_3.9x8.7mm_P1.27mm -> Package_SO:SOIC-16_3.9x9.9mm_P1.27mm
- U288, U289, U293, U294, U298: value 74AHCT125 -> 74LS151; footprint Package_SO:SOIC-14_3.9x8.7mm_P1.27mm -> Package_SO:SOIC-16_3.9x9.9mm_P1.27mm
- U31: value 74AHC541 -> 74AHCT125; footprint Package_SO:SOIC-20W_7.5x12.8mm_P1.27mm -> Package_SO:SOIC-14_3.9x8.7mm_P1.27mm
- U32: value 74AHC541 -> 74AHCT138; footprint Package_SO:SOIC-20W_7.5x12.8mm_P1.27mm -> Package_SO:SOIC-16_3.9x9.9mm_P1.27mm
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Connections:
- C143 pad 1: VCC -> GND
- C143 pad 2: GND -> VCC
- C144 pad 1: VCC -> GND
- C144 pad 2: GND -> VCC
- C148 pad 1: VCC -> GND
- C148 pad 2: GND -> VCC
- C149 pad 1: VCC -> GND
- C149 pad 2: GND -> VCC
- C151 pad 1: GND -> VCC
- C151 pad 2: VCC -> GND
- C162 pad 1: GND -> VCC
- C162 pad 2: VCC -> GND
- C163 pad 1: GND -> VCC
- C163 pad 2: VCC -> GND
- C164 pad 1: GND -> VCC
- C164 pad 2: VCC -> GND
- C165 pad 1: GND -> VCC
- C165 pad 2: VCC -> GND
- C166 pad 1: GND -> VCC
- C166 pad 2: VCC -> GND
- C167 pad 1: GND -> VCC
- C167 pad 2: VCC -> GND
- C168 pad 1: GND -> VCC
- C168 pad 2: VCC -> GND
- C170 pad 1: VCC -> GND
- C170 pad 2: GND -> VCC
- C171 pad 1: VCC -> GND
- C171 pad 2: GND -> VCC
- C172 pad 1: VCC -> GND
- C172 pad 2: GND -> VCC
- C173 pad 1: VCC -> GND
- C173 pad 2: GND -> VCC
- C176 pad 1: VCC -> GND
- C176 pad 2: GND -> VCC
- C177 pad 1: VCC -> GND
- C177 pad 2: GND -> VCC
- C178 pad 1: VCC -> GND
- C178 pad 2: GND -> VCC
- C181 pad 1: VCC -> GND
- C181 pad 2: GND -> VCC
- C182 pad 1: VCC -> GND
- C182 pad 2: GND -> VCC
- C183 pad 1: VCC -> GND
- C183 pad 2: GND -> VCC
- C186 pad 1: VCC -> GND
- C186 pad 2: GND -> VCC
- C188 pad 1: VCC -> GND
- C188 pad 2: GND -> VCC
- C191 pad 1: VCC -> GND
- C191 pad 2: GND -> VCC
- C192 pad 1: VCC -> GND
- C192 pad 2: GND -> VCC
- C193 pad 1: VCC -> GND
- C193 pad 2: GND -> VCC
- C196 pad 1: VCC -> GND
- C196 pad 2: GND -> VCC
- C197 pad 1: VCC -> GND
- C197 pad 2: GND -> VCC
- C198 pad 1: VCC -> GND
- C198 pad 2: GND -> VCC
- C201 pad 1: VCC -> GND
- C201 pad 2: GND -> VCC
- C202 pad 1: VCC -> GND
- C202 pad 2: GND -> VCC
- C203 pad 1: VCC -> GND
- C203 pad 2: GND -> VCC
- C206 pad 1: VCC -> GND
- C206 pad 2: GND -> VCC
- C207 pad 1: VCC -> GND
- C207 pad 2: GND -> VCC
- C208 pad 1: VCC -> GND
- C208 pad 2: GND -> VCC
- C211 pad 1: VCC -> GND
- C211 pad 2: GND -> VCC
- C217 pad 1: GND -> VCC
- C217 pad 2: VCC -> GND
- C218 pad 1: GND -> VCC
- C218 pad 2: VCC -> GND
- C219 pad 1: GND -> VCC
- C219 pad 2: VCC -> GND
- C220 pad 1: GND -> VCC
- C220 pad 2: VCC -> GND
- C221 pad 1: GND -> VCC
- C221 pad 2: VCC -> GND
- C222 pad 1: GND -> VCC
- C222 pad 2: VCC -> GND
- C223 pad 1: GND -> VCC
- C223 pad 2: VCC -> GND
- C224 pad 1: GND -> VCC
- C224 pad 2: VCC -> GND
- C225 pad 1: GND -> VCC
- C225 pad 2: VCC -> GND
- C226 pad 1: GND -> VCC
- C226 pad 2: VCC -> GND
- C227 pad 1: GND -> VCC
- C227 pad 2: VCC -> GND
- C228 pad 1: GND -> VCC
- C228 pad 2: VCC -> GND
- C229 pad 1: GND -> VCC
- C229 pad 2: VCC -> GND
- C23 pad 1: GND -> VCC
- C23 pad 2: VCC -> GND
- C230 pad 1: GND -> VCC
- C230 pad 2: VCC -> GND
- C233 pad 1: GND -> VCC
- C233 pad 2: VCC -> GND
- C234 pad 1: GND -> VCC
- C234 pad 2: VCC -> GND
- C235 pad 1: GND -> VCC
- C235 pad 2: VCC -> GND
- C238 pad 1: GND -> VCC
- C238 pad 2: VCC -> GND
- C239 pad 1: GND -> VCC
- C239 pad 2: VCC -> GND
- C24 pad 1: GND -> VCC
- C24 pad 2: VCC -> GND
- C240 pad 1: GND -> VCC
- C240 pad 2: VCC -> GND
- C243 pad 1: GND -> VCC
- C243 pad 2: VCC -> GND
- C244 pad 1: GND -> VCC
- C244 pad 2: VCC -> GND
- C245 pad 1: GND -> VCC
- C245 pad 2: VCC -> GND
- C246 pad 1: VCC -> Net-(U274-THRES)
- C247 pad 1: VCC -> Net-(U274-CONT)
- C248 pad 1: GND -> VCC
- C248 pad 2: VCC -> GND
- C249 pad 1: GND -> VCC
- C249 pad 2: VCC -> GND
- C250 pad 1: GND -> VCC
- C250 pad 2: VCC -> GND
- C251 pad 1: Net-(U284-THRES) -> VCC
- C252 pad 1: Net-(U284-CONT) -> VCC
- C253 pad 1: VCC -> GND
- C253 pad 2: GND -> VCC
- C254 pad 1: VCC -> GND
- C254 pad 2: GND -> VCC
- C255 pad 1: VCC -> GND
- C255 pad 2: GND -> VCC
- C256 pad 1: VCC -> GND
- C256 pad 2: GND -> VCC
- C260 pad 1: VCC -> GND
- C260 pad 2: GND -> VCC
- C261 pad 1: VCC -> GND
- C261 pad 2: GND -> VCC
- C265 pad 1: VCC -> GND
- C265 pad 2: GND -> VCC
- C266 pad 1: VCC -> GND
- C266 pad 2: GND -> VCC
- C28 pad 1: GND -> VCC
- C28 pad 2: VCC -> GND
- C29 pad 1: GND -> VCC
- C29 pad 2: VCC -> GND
- J1 pad 1: /flagZ -> VCC
- J1 pad 2: /~flagZ -> GND
- J1 pad 3: /flagN -> VCC
- J1 pad 4: /~flagN -> GND
- J1 pad 5: /flagC -> VCC
- J1 pad 6: /~flagC -> GND
- J1 pad 7: /flagV -> VCC
- J1 pad 8: /~flagV -> GND
- J2 pad 1: Net-(J2-Pin_1) -> A0
- J2 pad 10: Net-(J2-Pin_10) -> A9
- J2 pad 2: Net-(J2-Pin_2) -> A1
- J2 pad 3: Net-(J2-Pin_3) -> A2
- J2 pad 4: Net-(J2-Pin_4) -> A3
- J2 pad 5: Net-(J2-Pin_5) -> A4
- J2 pad 6: Net-(J2-Pin_6) -> A5
- J2 pad 7: Net-(J2-Pin_7) -> A6
- J2 pad 8: Net-(J2-Pin_8) -> A7
- J2 pad 9: Net-(J2-Pin_9) -> A8
- J3 pad 1: a0 -> C0
- J3 pad 10: a9 -> C9
- J3 pad 11: a10 -> C10
- J3 pad 12: a11 -> C11
- J3 pad 13: a12 -> C12
- J3 pad 14: a13 -> C13
- J3 pad 15: a14 -> C14
- J3 pad 16: a15 -> C15
- J3 pad 17: a16 -> C16
- J3 pad 18: a17 -> C17
- J3 pad 19: a18 -> C18
- J3 pad 2: a1 -> C1
- J3 pad 20: a19 -> C19
- J3 pad 21: a20 -> C20
- J3 pad 22: a21 -> C21
- J3 pad 23: a22 -> C22
- J3 pad 24: a23 -> C23
- J3 pad 25: a24 -> C24
- J3 pad 26: a25 -> C25
- J3 pad 27: a26 -> C26
- J3 pad 28: a27 -> C27
- J3 pad 29: a28 -> C28
- J3 pad 3: a2 -> C2
- J3 pad 30: a29 -> C29
- J3 pad 31: a30 -> C30
- J3 pad 32: a31 -> C31
- J3 pad 4: a3 -> C3
- J3 pad 5: a4 -> C4
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
Commit message: arch: added LEDs, override switches; fixed errors and warnings to 0
ready for routing after logical coherence check
Parts:
- removed C1, C10, C100, C101, C102, C103, C104, C105, C106, C107, C108, C109, C11, C110, C111, C112, C113, C114, C115, C116, C117, C118, C119, C12, C120, C121, C122, C123, C124, C125, C126, C127, C128, C129, C13, C130, C131, C132, C133, C134, C135, C136, C137, C138, C139, C14, C140, C141, C142, C143, C144, C145, C146, C147, C148, C15, C16, C162, C163, C164, C165, C166, C167, C168, C169, C17, C170, C171, C172, C173, C174, C175, C176, C177, C178, C179, C18, C180, C181, C182, C183, C184, C185, C186, C187, C188, C189, C19, C190, C191, C192, C193, C194, C195, C196, C197, C198, C199, C2, C20, C200, C201, C202, C203, C204, C205, C206, C207, C208, C209, C21, C210, C211, C212, C213, C217, C218, C219, C22, C220, C221, C222, C223, C224, C225, C226, C227, C228, C229, C23, C230, C231, C232, C233, C234, C235, C236, C237, C238, C239, C24, C240, C241, C242, C243, C244, C245, C247, C248, C249, C25, C250, C251, C252, C253, C254, C255, C256, C257, C258, C259, C26, C260, C261, C262, C263, C264, C265, C266, C267, C268, C27, C28, C29, C3, C30, C31, C32, C33, C34, C35, C36, C37, C38, C39, C4, C40, C41, C42, C43, C44, C45, C46, C47, C48, C49, C5, C50, C51, C52, C53, C54, C55, C56, C57, C58, C59, C6, C60, C61, C62, C63, C64, C65, C66, C67, C68, C69, C7, C70, C71, C72, C73, C74, C75, C76, C77, C78, C79, C8, C80, C81, C82, C83, C84, C85, C86, C87, C88, C89, C9, C90, C91, C92, C93, C94, C95, C96, C97, C98, C99: 100nF, Capacitor_SMD:C_0805_2012Metric
- removed C149, C150, C151, C152: C, Capacitor_SMD:C_0805_2012Metric
- removed C153, C154, C155, C156, C157, C158, C159, C160, C161, C214, C215, C216: 100nF, Capacitor_SMD:C_0603_1608Metric
- removed C246: 10nF, Capacitor_SMD:C_0805_2012Metric
- removed D1, D10, D11, D12, D13, D14, D15, D16, D17, D18, D19, D2, D20, D21, D22, D23, D24, D25, D26, D27, D28, D29, D3, D30, D31, D32, D4, D5, D6, D7, D8, D9: LED, LED_THT:LED_D5.0mm
- removed J1: Conn_02x04_Odd_Even, Connector_PinHeader_2.54mm:PinHeader_2x04_P2.54mm_Vertical
- removed J2, J3, J4: Conn_02x16_Counter_Clockwise, Connector_PinHeader_2.54mm:PinHeader_2x16_P2.54mm_Vertical
- removed J5: Conn_02x16_Counter_Clockwise, Connector_PinSocket_2.54mm:PinSocket_2x16_P2.54mm_Vertical
- removed J6: Conn_02x06_Odd_Even, Connector_PinSocket_2.54mm:PinSocket_2x06_P2.54mm_Vertical
- removed J7: Conn_02x01, Connector_PinHeader_2.54mm:PinHeader_2x01_P2.54mm_Horizontal
- removed J8: Conn_02x05_Odd_Even, Connector_PinHeader_2.54mm:PinHeader_2x05_P2.54mm_Vertical
- removed R1, R10, R11, R12, R13, R14, R15, R16, R17, R18, R19, R2, R20, R21, R22, R23, R24, R25, R26, R27, R28, R29, R3, R30, R31, R32, R4, R5, R6, R7, R8, R9: 3.3k, Resistor_SMD:R_0805_2012Metric
- removed R100, R101, R102, R103, R104, R105, R106, R107, R108, R109, R110, R111, R112, R113, R114, R115, R116, R117, R118, R119, R120, R121, R122, R123, R124, R125, R126, R127, R128, R129, R130, R131, R132, R133, R134, R135, R136, R137, R138, R139, R140, R141, R142, R143, R144, R145, R146, R147, R148, R149, R150, R151, R152, R153, R154, R155, R156, R157, R158, R159, R160, R161, R162, R163, R164, R165, R166, R167, R168, R169, R170, R171, R172, R173, R174, R175, R176, R177, R178, R179, R180, R181, R182, R183, R184, R185, R186, R187, R188, R189, R190, R191, R192, R193, R194, R195, R196, R197, R198, R199, R200, R201, R202, R203, R204, R205, R206, R207, R208, R209, R210, R211, R212, R213, R214, R215, R216, R217, R218, R219, R220, R221, R222, R223, R224, R225, R226, R227, R228, R229, R230, R231, R232, R233, R234, R235, R236, R237, R238, R239, R240, R241, R242, R243, R244, R245, R246, R247, R248, R249, R250, R251, R252, R253, R254, R255, R256, R259, R260, R261, R262, R263, R264, R265, R266, R267, R268, R269, R270, R271, R272, R273, R274, R275, R276, R277, R278, R279, R280, R281, R282, R283, R284, R285, R286, R287, R288, R289, R290, R33, R34, R35, R36, R37, R38, R39, R40, R41, R42, R43, R44, R45, R46, R47, R48, R49, R50, R51, R52, R53, R54, R55, R56, R57, R58, R59, R60, R61, R62, R63, R64, R65, R66, R67, R68, R69, R70, R71, R72, R73, R74, R75, R76, R77, R78, R79, R80, R81, R82, R83, R84, R85, R86, R87, R88, R89, R90, R91, R92, R93, R94, R95, R96, R97, R98, R99: 120, Resistor_SMD:R_0805_2012Metric
- removed R257: 1k, Resistor_SMD:R_0805_2012Metric
- removed R258: 10k, Resistor_SMD:R_0805_2012Metric
- removed U1, U168, U169: 74LS153, Package_SO:SOIC-16_3.9x9.9mm_P1.27mm
- removed U10, U11, U12, U13, U3, U4, U5, U6, U7, U8, U9: 74LS182, Package_DIP:DIP-16_W7.62mm
- removed U100, U101, U105, U106, U110, U111, U115, U116, U120, U121, U125, U126, U130, U131, U135, U136, U140, U141, U176, U177, U181, U182, U186, U187, U191, U192, U196, U197, U201, U202, U206, U207, U211, U212, U25, U26, U30, U31, U35, U36, U40, U41, U45, U46, U50, U51, U55, U56, U60, U61, U65, U66, U70, U71, U75, U76, U80, U81, U85, U86, U90, U91, U95, U96: 74AHCT125, Package_SO:SOIC-14_3.9x8.7mm_P1.27mm
- removed U102, U107, U112, U117, U122, U127, U132, U137, U142, U178, U183, U188, U193, U198, U203, U208, U213, U27, U32, U37, U42, U47, U52, U57, U62, U67, U72, U77, U82, U87, U92, U97: 74AHCT138, Package_SO:SOIC-16_3.9x9.9mm_P1.27mm
- removed U103, U108, U113, U118, U123, U128, U133, U138, U174, U179, U184, U189, U194, U199, U204, U209, U23, U28, U33, U38, U43, U48, U53, U58, U63, U68, U73, U78, U83, U88, U93, U98: 74LS08, Package_SO:SOIC-14_3.9x8.7mm_P1.27mm
- removed U104, U109, U114, U119, U124, U129, U134, U139, U175, U180, U185, U190, U195, U200, U205, U21, U210, U24, U29, U34, U39, U44, U49, U54, U59, U64, U69, U74, U79, U84, U89, U94, U99: 74HC86, Package_SO:SOIC-14_3.9x8.7mm_P1.27mm
- removed U14, U15, U16, U17: 74LS30, Package_SO:SOIC-14_3.9x8.7mm_P1.27mm
- removed U143, U144, U145, U146, U170, U171, U172, U173, U22: 74LS540, Package_SO:SOIC-20W_7.5x12.8mm_P1.27mm
- removed U147, U148, U167: KM28C64A, Package_DIP:DIP-28_W15.24mm
- removed U149, U150, U151, U152, U153, U155, U156, U158, U159, U161, U214, U216: 74AHC541, Package_SO:SOIC-20W_7.5x12.8mm_P1.27mm
- removed U154, U157, U160, U164, U215: 74AHC1G04, Package_TO_SOT_SMD:SOT-23-5
- removed U162, U166: 74LS154, Package_SO:SOIC-24W_7.5x15.4mm_P1.27mm
- removed U163, U165: 74LS163, Package_SO:SOIC-16_3.9x9.9mm_P1.27mm
- removed U18: 74HCT00, Package_SO:SOIC-14_3.9x8.7mm_P1.27mm
- removed U19, U20, U217, U219, U221, U223, U225, U227, U229, U231, U233, U235, U237, U239, U241, U243, U245, U247, U249, U251, U253, U255, U257, U259, U261, U263, U265, U267, U269, U271, U273, U277, U279, U281: 74LS377, Package_SO:SOIC-20W_7.5x12.8mm_P1.27mm
- removed U2: 74AHCT1G08, Package_TO_SOT_SMD:SOT-23-5
- removed U218, U220, U222, U224, U226, U228, U230, U232, U234, U236, U238, U240, U242, U244, U246, U248, U250, U252, U254, U256, U258, U260, U262, U264, U266, U268, U270, U272, U275, U278, U280, U282: HDSP-A153, Display_7Segment:HDSP-A151
- removed U274: ICM7555xB, Package_SO:SOIC-8_3.9x4.9mm_P1.27mm
- removed U276: 74HCT541, Package_SO:SOIC-20W_7.5x12.8mm_P1.27mm
- removed U283, U284, U285, U286, U287, U288, U289, U290, U291, U292, U293, U294, U295, U296, U297, U298: 74LS151, Package_SO:SOIC-16_3.9x9.9mm_P1.27mm
Other:
- copper layers 2 -> 4

Commit message: fix: fixed the zero flag detection logic
Parts:
- added C1: 100nF, Capacitor_SMD:C_0805_2012Metric, F.Cu at (-454.9, 161.3)
- added C10: 100nF, Capacitor_SMD:C_0805_2012Metric, F.Cu at (-450.5, 161.3)
- added C100: 100nF, Capacitor_SMD:C_0805_2012Metric, F.Cu at (-283.1, 235.2)
- added C101: 100nF, Capacitor_SMD:C_0805_2012Metric, F.Cu at (-275.1, 387.5)
- added C102: 100nF, Capacitor_SMD:C_0805_2012Metric, F.Cu at (-275.1, 390.5)
- added C103: 100nF, Capacitor_SMD:C_0805_2012Metric, F.Cu at (-207.3, 83.6)
- added C104: 100nF, Capacitor_SMD:C_0805_2012Metric, F.Cu at (-207.2, 93.2)
- added C105: 100nF, Capacitor_SMD:C_0805_2012Metric, F.Cu at (-218.4, 85.0)
- added C106: 100nF, Capacitor_SMD:C_0805_2012Metric, F.Cu at (-350.7, 369.1)
- added C107: 100nF, Capacitor_SMD:C_0805_2012Metric, F.Cu at (-350.7, 372.1)
- added C108: 100nF, Capacitor_SMD:C_0805_2012Metric, F.Cu at (-317.7, 257.7)
- added C109: 100nF, Capacitor_SMD:C_0805_2012Metric, F.Cu at (-317.6, 267.4)
- added C11: 100nF, Capacitor_SMD:C_0805_2012Metric, F.Cu at (-450.5, 164.3)
- added C110: 100nF, Capacitor_SMD:C_0805_2012Metric, F.Cu at (-328.8, 259.2)
- added C111: 100nF, Capacitor_SMD:C_0805_2012Metric, F.Cu at (-331.8, 387.5)
- added C112: 100nF, Capacitor_SMD:C_0805_2012Metric, F.Cu at (-331.8, 390.5)
- added C113: 100nF, Capacitor_SMD:C_0805_2012Metric, F.Cu at (-393.3, 281.7)
- added C114: 100nF, Capacitor_SMD:C_0805_2012Metric, F.Cu at (-393.2, 291.3)
- added C115: 100nF, Capacitor_SMD:C_0805_2012Metric, F.Cu at (-404.4, 283.1)
- added C116: 100nF, Capacitor_SMD:C_0805_2012Metric, F.Cu at (-294.0, 369.1)
- added C117: 100nF, Capacitor_SMD:C_0805_2012Metric, F.Cu at (-294.0, 372.1)
- added C118: 100nF, Capacitor_SMD:C_0805_2012Metric, F.Cu at (-206.5, 64.0)
- added C119: 100nF, Capacitor_SMD:C_0805_2012Metric, F.Cu at (-206.4, 73.7)
- added C12: 100nF, Capacitor_SMD:C_0805_2012Metric, F.Cu at (-450.5, 167.3)
- added C120: 100nF, Capacitor_SMD:C_0805_2012Metric, F.Cu at (-217.6, 65.5)
- added C121: 100nF, Capacitor_SMD:C_0805_2012Metric, F.Cu at (-294.0, 332.3)
- added C122: 100nF, Capacitor_SMD:C_0805_2012Metric, F.Cu at (-294.0, 335.4)
- added C123: 100nF, Capacitor_SMD:C_0805_2012Metric, F.Cu at (-374.4, 257.7)
- added C124: 100nF, Capacitor_SMD:C_0805_2012Metric, F.Cu at (-374.3, 267.4)
- added C125: 100nF, Capacitor_SMD:C_0805_2012Metric, F.Cu at (-385.5, 259.2)
- added C126: 100nF, Capacitor_SMD:C_0805_2012Metric, F.Cu at (-331.8, 350.7)
- added C127: 100nF, Capacitor_SMD:C_0805_2012Metric, F.Cu at (-331.8, 353.7)
- added C128: 100nF, Capacitor_SMD:C_0805_2012Metric, F.Cu at (-393.3, 353.6)
- added C129: 100nF, Capacitor_SMD:C_0805_2012Metric, F.Cu at (-393.2, 363.3)
- added C13: 100nF, Capacitor_SMD:C_0805_2012Metric, F.Cu at (-450.5, 170.4)
- added C130: 100nF, Capacitor_SMD:C_0805_2012Metric, F.Cu at (-404.4, 355.1)
- added C131: 100nF, Capacitor_SMD:C_0805_2012Metric, F.Cu at (-312.9, 369.1)
- added C132: 100nF, Capacitor_SMD:C_0805_2012Metric, F.Cu at (-312.9, 372.1)
- added C133: 100nF, Capacitor_SMD:C_0805_2012Metric, F.Cu at (-412.2, 353.6)
- added C134: 100nF, Capacitor_SMD:C_0805_2012Metric, F.Cu at (-412.1, 363.3)
- added C135: 100nF, Capacitor_SMD:C_0805_2012Metric, F.Cu at (-423.3, 355.1)
- added C136: 100nF, Capacitor_SMD:C_0805_2012Metric, F.Cu at (-293.6, 290.0)
- added C137: 100nF, Capacitor_SMD:C_0805_2012Metric, F.Cu at (-293.6, 293.0)
- added C138: 100nF, Capacitor_SMD:C_0805_2012Metric, F.Cu at (-290.9, 233.7)
- added C139: 100nF, Capacitor_SMD:C_0805_2012Metric, F.Cu at (-290.8, 243.3)
- added C14: 100nF, Capacitor_SMD:C_0805_2012Metric, F.Cu at (-450.5, 173.4)
- added C140: 100nF, Capacitor_SMD:C_0805_2012Metric, F.Cu at (-302.0, 235.2)
- added C141: 100nF, Capacitor_SMD:C_0805_2012Metric, F.Cu at (-294.0, 387.5)
- added C142: 100nF, Capacitor_SMD:C_0805_2012Metric, F.Cu at (-294.0, 390.5)
- added C143: 100nF, Capacitor_SMD:C_0805_2012Metric, F.Cu at (-412.2, 257.7)
- added C144: 100nF, Capacitor_SMD:C_0805_2012Metric, F.Cu at (-412.1, 267.4)
- added C145: 100nF, Capacitor_SMD:C_0805_2012Metric, F.Cu at (-423.3, 259.2)
- added C146: 100nF, Capacitor_SMD:C_0805_2012Metric, F.Cu at (-409.0, 189.8)
- added C147: 100nF, Capacitor_SMD:C_0805_2012Metric, F.Cu at (-409.0, 192.8)
- added C148: 100nF, Capacitor_SMD:C_0805_2012Metric, F.Cu at (-409.0, 195.8)
- added C149: 100nF, Capacitor_SMD:C_0805_2012Metric, F.Cu at (-409.0, 198.8)
- added C15: 100nF, Capacitor_SMD:C_0805_2012Metric, F.Cu at (-450.5, 176.4)
- added C150: 100nF, Capacitor_SMD:C_0805_2012Metric, F.Cu at (-372.3, 153.9)
- added C151: 100nF, Capacitor_SMD:C_0805_2012Metric, F.Cu at (-372.3, 156.9)
- added C152: C, Capacitor_SMD:C_0805_2012Metric, F.Cu at (-372.3, 160.0)
- added C153: 100nF, Capacitor_SMD:C_0805_2012Metric, F.Cu at (-372.3, 163.0)
- added C154: C, Capacitor_SMD:C_0805_2012Metric, F.Cu at (-372.3, 166.0)
- added C155: C, Capacitor_SMD:C_0805_2012Metric, F.Cu at (-372.3, 169.0)
- added C156: 100nF, Capacitor_SMD:C_0603_1608Metric, F.Cu at (-398.7, 245.9)
- added C157: 100nF, Capacitor_SMD:C_0603_1608Metric, F.Cu at (-398.7, 248.4)
- added C158: 100nF, Capacitor_SMD:C_0603_1608Metric, F.Cu at (-398.7, 250.9)
- added C159: 100nF, Capacitor_SMD:C_0603_1608Metric, F.Cu at (-370.9, 245.9)
- added C16: 100nF, Capacitor_SMD:C_0805_2012Metric, F.Cu at (-446.0, 161.3)
- added C160: 100nF, Capacitor_SMD:C_0603_1608Metric, F.Cu at (-370.9, 248.4)
- added C161: 100nF, Capacitor_SMD:C_0603_1608Metric, F.Cu at (-370.9, 250.9)
- added C162: 100nF, Capacitor_SMD:C_0603_1608Metric, F.Cu at (-426.6, 245.9)
- added C163: 100nF, Capacitor_SMD:C_0603_1608Metric, F.Cu at (-426.6, 248.4)
- added C164: 100nF, Capacitor_SMD:C_0603_1608Metric, F.Cu at (-426.6, 250.9)
- added C165: 100nF, Capacitor_SMD:C_0805_2012Metric, F.Cu at (-206.1, 44.4)
- added C166: 100nF, Capacitor_SMD:C_0805_2012Metric, F.Cu at (-206.0, 54.1)
- added C167: 100nF, Capacitor_SMD:C_0805_2012Metric, F.Cu at (-217.2, 45.9)
- added C168: 100nF, Capacitor_SMD:C_0805_2012Metric, F.Cu at (-303.2, 155.4)
- added C169: 100nF, Capacitor_SMD:C_0805_2012Metric, F.Cu at (-303.2, 158.4)
- added C17: 100nF, Capacitor_SMD:C_0805_2012Metric, F.Cu at (-446.0, 164.3)
- added C170: 100nF, Capacitor_SMD:C_0805_2012Metric, F.Cu at (-303.2, 161.4)
- added C171: 100nF, Capacitor_SMD:C_0805_2012Metric, F.Cu at (-303.2, 164.4)
- added C172: 100nF, Capacitor_SMD:C_0805_2012Metric, F.Cu at (-303.2, 167.4)
- added C173: 100nF, Capacitor_SMD:C_0805_2012Metric, F.Cu at (-303.2, 170.4)
- added C174: 100nF, Capacitor_SMD:C_0805_2012Metric, F.Cu at (-303.2, 173.5)
- added C175: 100nF, Capacitor_SMD:C_0805_2012Metric, F.Cu at (-303.2, 176.5)
- added C176: 100nF, Capacitor_SMD:C_0805_2012Metric, F.Cu at (-347.4, 129.7)
- added C177: 100nF, Capacitor_SMD:C_0805_2012Metric, F.Cu at (-347.4, 132.7)
- added C178: 100nF, Capacitor_SMD:C_0805_2012Metric, F.Cu at (-347.4, 135.8)
- added C179: 100nF, Capacitor_SMD:C_0805_2012Metric, F.Cu at (-347.4, 138.8)
- added C18: 100nF, Capacitor_SMD:C_0805_2012Metric, F.Cu at (-446.0, 167.3)
- added C180: 100nF, Capacitor_SMD:C_0805_2012Metric, F.Cu at (-350.7, 387.5)
- added C181: 100nF, Capacitor_SMD:C_0805_2012Metric, F.Cu at (-350.7, 390.5)
- added C182: 100nF, Capacitor_SMD:C_0805_2012Metric, F.Cu at (-298.8, 257.7)
- added C183: 100nF, Capacitor_SMD:C_0805_2012Metric, F.Cu at (-298.7, 267.4)
- added C184: 100nF, Capacitor_SMD:C_0805_2012Metric, F.Cu at (-309.9, 259.2)
- added C185: 100nF, Capacitor_SMD:C_0805_2012Metric, F.Cu at (-331.8, 332.3)
- added C186: 100nF, Capacitor_SMD:C_0805_2012Metric, F.Cu at (-331.8, 335.4)
- added C187: 100nF, Capacitor_SMD:C_0805_2012Metric, F.Cu at (-412.2, 305.7)
- added C188: 100nF, Capacitor_SMD:C_0805_2012Metric, F.Cu at (-412.1, 315.3)
- added C189: 100nF, Capacitor_SMD:C_0805_2012Metric, F.Cu at (-423.3, 307.1)
- added C19: 100nF, Capacitor_SMD:C_0805_2012Metric, F.Cu at (-446.0, 170.4)
- added C190: 100nF, Capacitor_SMD:C_0805_2012Metric, F.Cu at (-294.0, 350.7)
- added C191: 100nF, Capacitor_SMD:C_0805_2012Metric, F.Cu at (-294.0, 353.7)
- added C192: 100nF, Capacitor_SMD:C_0805_2012Metric, F.Cu at (-374.4, 329.7)
- added C193: 100nF, Capacitor_SMD:C_0805_2012Metric, F.Cu at (-374.3, 339.3)
- added C194: 100nF, Capacitor_SMD:C_0805_2012Metric, F.Cu at (-385.5, 331.1)
- added C195: 100nF, Capacitor_SMD:C_0805_2012Metric, F.Cu at (-294.0, 314.0)
- added C196: 100nF, Capacitor_SMD:C_0805_2012Metric, F.Cu at (-294.0, 317.0)
- added C197: 100nF, Capacitor_SMD:C_0805_2012Metric, F.Cu at (-374.4, 281.7)
- added C198: 100nF, Capacitor_SMD:C_0805_2012Metric, F.Cu at (-374.3, 291.3)
- added C199: 100nF, Capacitor_SMD:C_0805_2012Metric, F.Cu at (-385.5, 283.1)
- added C2: 100nF, Capacitor_SMD:C_0805_2012Metric, F.Cu at (-454.9, 164.3)
- added C20: 100nF, Capacitor_SMD:C_0805_2012Metric, F.Cu at (-446.0, 173.4)
- added C200: 100nF, Capacitor_SMD:C_0805_2012Metric, F.Cu at (-350.7, 332.3)
- added C201: 100nF, Capacitor_SMD:C_0805_2012Metric, F.Cu at (-350.7, 335.4)
- added C202: 100nF, Capacitor_SMD:C_0805_2012Metric, F.Cu at (-279.9, 257.7)
- added C203: 100nF, Capacitor_SMD:C_0805_2012Metric, F.Cu at (-279.8, 267.4)
- added C204: 100nF, Capacitor_SMD:C_0805_2012Metric, F.Cu at (-291.0, 259.2)
- added C205: 100nF, Capacitor_SMD:C_0805_2012Metric, F.Cu at (-369.6, 369.1)
- added C206: 100nF, Capacitor_SMD:C_0805_2012Metric, F.Cu at (-369.6, 372.1)
- added C207: 100nF, Capacitor_SMD:C_0805_2012Metric, F.Cu at (-374.4, 377.6)
- added C208: 100nF, Capacitor_SMD:C_0805_2012Metric, F.Cu at (-374.3, 387.3)
- added C209: 100nF, Capacitor_SMD:C_0805_2012Metric, F.Cu at (-385.5, 379.1)
- added C21: 100nF, Capacitor_SMD:C_0805_2012Metric, F.Cu at (-446.0, 176.4)
- added C210: 100nF, Capacitor_SMD:C_0805_2012Metric, F.Cu at (-350.7, 350.7)
- added C211: 100nF, Capacitor_SMD:C_0805_2012Metric, F.Cu at (-350.7, 353.7)
- added C212: 100nF, Capacitor_SMD:C_0805_2012Metric, F.Cu at (-336.6, 257.7)
- added C213: 100nF, Capacitor_SMD:C_0805_2012Metric, F.Cu at (-336.5, 267.4)
- added C214: 100nF, Capacitor_SMD:C_0805_2012Metric, F.Cu at (-347.7, 259.2)
- added C215: 100nF, Capacitor_SMD:C_0805_2012Metric, F.Cu at (-369.6, 314.0)
- added C216: 100nF, Capacitor_SMD:C_0805_2012Metric, F.Cu at (-369.6, 317.0)
- added C217: 100nF, Capacitor_SMD:C_0805_2012Metric, F.Cu at (-293.8, 126.9)
- added C218: 100nF, Capacitor_SMD:C_0805_2012Metric, F.Cu at (-293.8, 129.9)
- added C219: 100nF, Capacitor_SMD:C_0805_2012Metric, F.Cu at (-293.8, 132.9)
- added C22: 100nF, Capacitor_SMD:C_0805_2012Metric, F.Cu at (-441.6, 161.3)
- added C220: 100nF, Capacitor_SMD:C_0805_2012Metric, F.Cu at (-293.8, 135.9)
- added C221: 100nF, Capacitor_SMD:C_0805_2012Metric, F.Cu at (-548.0, 217.7)
- added C222: 100nF, Capacitor_SMD:C_0805_2012Metric, F.Cu at (-548.0, 220.7)
- added C223: 100nF, Capacitor_SMD:C_0805_2012Metric, F.Cu at (-548.0, 223.7)
- added C224: 100nF, Capacitor_SMD:C_0805_2012Metric, F.Cu at (-548.0, 226.7)
- added C225: 100nF, Capacitor_SMD:C_0805_2012Metric, F.Cu at (-296.8, 155.4)
- added C226: 100nF, Capacitor_SMD:C_0805_2012Metric, F.Cu at (-296.8, 158.4)
- added C227: 100nF, Capacitor_SMD:C_0805_2012Metric, F.Cu at (-296.8, 161.4)
- added C228: 100nF, Capacitor_SMD:C_0805_2012Metric, F.Cu at (-296.8, 164.4)
- added C229: 100nF, Capacitor_SMD:C_0805_2012Metric, F.Cu at (-296.8, 181.1)
- added C23: 100nF, Capacitor_SMD:C_0805_2012Metric, F.Cu at (-441.6, 164.3)
- added C230: 100nF, Capacitor_SMD:C_0805_2012Metric, F.Cu at (-296.8, 184.1)
- added C231: 100nF, Capacitor_SMD:C_0805_2012Metric, F.Cu at (-296.8, 187.1)
- added C232: 100nF, Capacitor_SMD:C_0805_2012Metric, F.Cu at (-296.8, 190.1)
- added C233: 100nF, Capacitor_SMD:C_0805_2012Metric, F.Cu at (-437.6, 374.0)
- added C234: 100nF, Capacitor_SMD:C_0805_2012Metric, F.Cu at (-437.6, 297.2)
- added C235: 100nF, Capacitor_SMD:C_0805_2012Metric, F.Cu at (-466.3, 322.8)
- added C236: 100nF, Capacitor_SMD:C_0805_2012Metric, F.Cu at (-494.9, 374.0)
- added C237: 100nF, Capacitor_SMD:C_0805_2012Metric, F.Cu at (-494.9, 348.4)
- added C238: 100nF, Capacitor_SMD:C_0805_2012Metric, F.Cu at (-437.6, 246.0)
- added C239: 100nF, Capacitor_SMD:C_0805_2012Metric, F.Cu at (-494.9, 271.6)
- added C24: 100nF, Capacitor_SMD:C_0805_2012Metric, F.Cu at (-441.6, 167.3)
- added C240: 100nF, Capacitor_SMD:C_0805_2012Metric, F.Cu at (-437.6, 220.4)
- added C241: 100nF, Capacitor_SMD:C_0805_2012Metric, F.Cu at (-380.4, 220.4)
- added C242: 100nF, Capacitor_SMD:C_0805_2012Metric, F.Cu at (-294.5, 220.4)
- added C243: 100nF, Capacitor_SMD:C_0805_2012Metric, F.Cu at (-494.9, 297.2)
- added C244: 100nF, Capacitor_SMD:C_0805_2012Metric, F.Cu at (-530.7, 297.3)
- added C245: 100nF, Capacitor_SMD:C_0805_2012Metric, F.Cu at (-530.7, 374.1)
- added C246: 100nF, Capacitor_SMD:C_0805_2012Metric, F.Cu at (-494.9, 322.8)
- added C247: 100nF, Capacitor_SMD:C_0805_2012Metric, F.Cu at (-323.1, 220.4)
- added C248: 100nF, Capacitor_SMD:C_0805_2012Metric, F.Cu at (-466.3, 271.6)
- added C249: 100nF, Capacitor_SMD:C_0805_2012Metric, F.Cu at (-466.3, 220.4)
- added C25: 100nF, Capacitor_SMD:C_0805_2012Metric, F.Cu at (-441.6, 170.4)
- added C250: 100nF, Capacitor_SMD:C_0805_2012Metric, F.Cu at (-466.3, 374.0)
- added C251: 100nF, Capacitor_SMD:C_0805_2012Metric, F.Cu at (-494.9, 220.4)
- added C252: 100nF, Capacitor_SMD:C_0805_2012Metric, F.Cu at (-494.9, 246.0)
- added C253: 100nF, Capacitor_SMD:C_0805_2012Metric, F.Cu at (-437.6, 322.8)
- added C254: 100nF, Capacitor_SMD:C_0805_2012Metric, F.Cu at (-437.6, 271.6)
- added C255: 100nF, Capacitor_SMD:C_0805_2012Metric, F.Cu at (-437.6, 348.4)
- added C256: 100nF, Capacitor_SMD:C_0805_2012Metric, F.Cu at (-530.7, 322.9)
- added C257: 100nF, Capacitor_SMD:C_0805_2012Metric, F.Cu at (-466.3, 246.0)
- added C258: 100nF, Capacitor_SMD:C_0805_2012Metric, F.Cu at (-530.7, 246.1)
- added C259: 10nF, Capacitor_SMD:C_0805_2012Metric, F.Cu at (-300.0, 279.6)
- added C26: 100nF, Capacitor_SMD:C_0805_2012Metric, F.Cu at (-350.7, 314.0)
- added C260: 100nF, Capacitor_SMD:C_0805_2012Metric, F.Cu at (-300.0, 282.6)
- added C261: 100nF, Capacitor_SMD:C_0805_2012Metric, F.Cu at (-300.0, 285.6)
- added C262: 100nF, Capacitor_SMD:C_0805_2012Metric, F.Cu at (-300.0, 288.7)
- added C263: 100nF, Capacitor_SMD:C_0805_2012Metric, F.Cu at (-530.7, 348.5)
- added C264: 100nF, Capacitor_SMD:C_0805_2012Metric, F.Cu at (-409.0, 220.4)
- added C265: 100nF, Capacitor_SMD:C_0805_2012Metric, F.Cu at (-530.7, 271.7)
- added C266: 100nF, Capacitor_SMD:C_0805_2012Metric, F.Cu at (-466.3, 348.4)
- added C267: 100nF, Capacitor_SMD:C_0805_2012Metric, F.Cu at (-351.8, 220.4)
- added C268: 100nF, Capacitor_SMD:C_0805_2012Metric, F.Cu at (-466.3, 297.2)
- added C27: 100nF, Capacitor_SMD:C_0805_2012Metric, F.Cu at (-350.7, 317.0)
- added C28: 100nF, Capacitor_SMD:C_0805_2012Metric, F.Cu at (-336.6, 281.7)
- added C29: 100nF, Capacitor_SMD:C_0805_2012Metric, F.Cu at (-336.5, 291.3)
- added C3: 100nF, Capacitor_SMD:C_0603_1608Metric, F.Cu at (-424.0, 161.1)
- added C30: 100nF, Capacitor_SMD:C_0805_2012Metric, F.Cu at (-347.7, 283.1)
- added C31: 100nF, Capacitor_SMD:C_0805_2012Metric, F.Cu at (-369.6, 332.3)
- added C32: 100nF, Capacitor_SMD:C_0805_2012Metric, F.Cu at (-369.6, 335.4)
- added C33: 100nF, Capacitor_SMD:C_0805_2012Metric, F.Cu at (-309.8, 233.7)
- added C34: 100nF, Capacitor_SMD:C_0805_2012Metric, F.Cu at (-309.7, 243.3)
- added C35: 100nF, Capacitor_SMD:C_0805_2012Metric, F.Cu at (-320.9, 235.2)
- added C36: 100nF, Capacitor_SMD:C_0805_2012Metric, F.Cu at (-331.8, 314.0)
- added C37: 100nF, Capacitor_SMD:C_0805_2012Metric, F.Cu at (-331.8, 317.0)
- added C38: 100nF, Capacitor_SMD:C_0805_2012Metric, F.Cu at (-374.4, 353.6)
- added C39: 100nF, Capacitor_SMD:C_0805_2012Metric, F.Cu at (-374.3, 363.3)
- added C4: 100nF, Capacitor_SMD:C_0805_2012Metric, F.Cu at (-454.9, 167.3)
- added C40: 100nF, Capacitor_SMD:C_0805_2012Metric, F.Cu at (-385.5, 355.1)
- added C41: 100nF, Capacitor_SMD:C_0805_2012Metric, F.Cu at (-369.6, 350.7)
- added C42: 100nF, Capacitor_SMD:C_0805_2012Metric, F.Cu at (-369.6, 353.7)
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Routing:
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- added copper zone on In1.Cu, net GND
- added copper zone on In2.Cu, net VCC
Other:
- board outline added: 263 x 208.6 mm
