File: hardware/kicad/boards/01_alu/alu-32b.kicad_pcb (KiCad board)
At the start: 4 copper layers, 220 x 220 mm, 760 parts, among them J1 Conn_02x06_Odd_Even, J2 Conn_02x04_Odd_Even, J3 Conn_02x16_Odd_Even, J4 Conn_02x16_Odd_Even, J5 Conn_02x16_Odd_Even, J6 Conn_02x16_Counter_Clockwise, J7 Conn_02x01, J8 Conn_02x05_Odd_Even, SW1 SW_DIP_x08, SW10 SW_DIP_x08, SW11 SW_DIP_x08, SW12 SW_DIP_x08, SW13 SW_SPDT, SW14 SW_DIP_x08, SW15 SW_DIP_x08, SW16 SW_Slide_DPDT, SW2 SW_DIP_x08, SW3 SW_DIP_x08, SW4 SW_DIP_x08, SW5 SW_DIP_x08, SW6 SW_DIP_x08, SW7 SW_DIP_x08, SW8 SW_DIP_x08, SW9 SW_DIP_x08, U1 74HC86, U10 74LS540, U100 74AHCT138, U101 74LS08, U102 74HC86, U103 74AHCT125, U104 74AHCT125, U105 74AHCT138, U106 74LS08, U107 74HC86, U108 74AHCT125, U109 74AHCT125, U11 74LS540, U110 74AHCT138, U111 74LS08, U112 74HC86, U113 74AHCT125, U114 74AHCT125, U115 74AHCT138, U116 74LS08, U117 74HC86, U118 74AHCT125, U119 74AHCT125, U12 74LS30, U120 74AHCT138, U121 74LS08, U122 74HC86, U123 74AHCT125, U124 74AHCT125, U125 74AHCT138, U126 74LS08, U127 74HC86, U128 74AHCT125, U129 74AHCT125, U13 74LS182, U130 74AHCT138, U131 74LS08, U132 74HC86, U133 74AHCT125, U134 74AHCT125, U135 74AHCT138, U136 74LS08, U137 74HC86, U138 74AHCT125, U139 74AHCT125, U14 74LS182, U140 74AHCT138, U141 74LS08, U142 74HC86, U143 74AHCT125, U144 74AHCT125, U145 74AHCT138, U146 74LS08, U147 74HC86, U148 74AHCT125, U149 74AHCT125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

Commit message: schematics: designed alu into 4b slices saving several chips and "de-bloating" board of several glue and drivers
Parts:
- removed C112, C116, C118, C122, C124, C128, C130, C134, C135, C136, C137, C138, C139, C142, C149, C153, C161, C162, C163, C164, C165, C166, C168, C172, C174, C178, C180, C184, C186, C190, C192, C196, C198, C202, C204, C208, C210, C214, C215, C216, C217, C218, C219, C220, C221, C222, C223, C224, C225, C226, C227, C228, C229, C230, C231, C232, C233, C234, C235, C236, C237, C238, C239, C240, C241, C242, C243, C244, C245, C246, C247, C248, C249, C250, C251, C252, C253, C254, C255, C256, C257, C259, C260, C262, C263, C264, C265: 100nF, Capacitor_SMD:C_0603_1608Metric
- removed C157, C159, C160: C, Capacitor_SMD:C_0603_1608Metric
- removed C258: 10nF, Capacitor_SMD:C_0603_1608Metric
- removed R100, R101, R102, R103, R104, R105, R106, R107, R108, R109, R110, R111, R112, R113, R114, R115, R116, R117, R118, R119, R120, R121, R122, R123, R124, R125, R126, R127, R128, R129, R130, R131, R132, R133, R134, R135, R136, R137, R138, R139, R140, R141, R142, R143, R144, R145, R146, R147, R148, R149, R15, R150, R151, R152, R153, R154, R155, R156, R157, R158, R159, R16, R160, R161, R162, R163, R164, R165, R166, R167, R168, R169, R17, R170, R171, R172, R173, R174, R18, R19, R20, R21, R22, R23, R24, R25, R26, R27, R28, R29, R30, R31, R32, R33, R34, R35, R36, R37, R38, R39, R40, R41, R42, R43, R44, R45, R46, R47, R48, R49, R50, R51, R52, R53, R54, R55, R56, R57, R58, R59, R60, R61, R62, R63, R64, R65, R66, R67, R68, R69, R70, R71, R72, R73, R74, R75, R76, R77, R78, R79, R80, R81, R82, R83, R84, R85, R86, R87, R88, R89, R90, R91, R92, R93, R94, R95, R96, R97, R98, R99: 120, Resistor_SMD:R_0805_2012Metric
- removed R175: 1k, Resistor_SMD:R_0805_2012Metric
- removed R176: 10k, Resistor_SMD:R_0805_2012Metric
- removed U102, U186, U196, U201, U206, U216, U221, U42, U57, U72, U87: 74HC86, Package_SO:SOIC-14_3.9x8.7mm_P1.27mm
- removed U109, U119, U123, U124, U171, U187, U188, U192, U193, U202, U203, U207, U208, U213, U217, U218, U33, U39, U48, U54, U63, U69, U78, U84: 74AHCT125, Package_SO:SOIC-14_3.9x8.7mm_P1.27mm
- removed U116, U185, U195, U200, U210, U215, U220, U36, U51, U66, U81: 74LS08, Package_SO:SOIC-14_3.9x8.7mm_P1.27mm
- removed U120, U172, U189, U194, U199, U209, U214, U219, U45, U60, U75, U90, U95: 74AHCT138, Package_SO:SOIC-16_3.9x9.9mm_P1.27mm
- removed U152, U153, U181, U182: 74LS540, Package_SO:SOIC-20W_7.5x12.8mm_P1.27mm
- removed U156, U178: KM28C64A, Package_DIP:DIP-28_W15.24mm
- removed U157, U158, U159, U160, U161, U164, U166, U167: 74AHC541, Package_SO:SOIC-20W_7.5x12.8mm_P1.27mm
- removed U165, U168, U175: 74AHC1G04, Package_TO_SOT_SMD:SOT-23-5
- removed U173: 74LS154, Package_SO:SOIC-24W_7.5x15.4mm_P1.27mm
- removed U174: 74LS163, Package_SO:SOIC-16_3.9x9.9mm_P1.27mm
- removed U179, U180: 74LS153, Package_SO:SOIC-16_3.9x9.9mm_P1.27mm
- removed U222, U223, U224, U225, U226, U227, U228, U229, U230, U231, U232, U233, U234, U235, U236, U237, U280, U281, U282, U283: 74LS151, Package_SO:SOIC-16_3.9x9.9mm_P1.27mm
- removed U238, U240, U242, U244, U246, U248, U250, U252, U254, U256, U258, U260, U262, U264, U266, U268, U270, U272, U274, U276: 74LS377, Package_SO:SOIC-20W_7.5x12.8mm_P1.27mm
- removed U239, U241, U243, U245, U247, U249, U251, U253, U255, U257, U259, U261, U263, U265, U267, U269, U271, U273, U275, U277: HDSP-A153, Display_7Segment:HDSP-A151
- removed U278: ICM7555xB, Package_SO:SOIC-8_3.9x4.9mm_P1.27mm
- C10, C101, C104, C106, C109, C11, C114, C119, C121, C126, C131, C141, C146, C169, C171, C188, C193, C195, C20, C200, C205, C21, C213, C27, C28, C29, C30, C34, C36, C4, C41, C44, C46, C49, C54, C56, C61, C64, C66, C69, C74, C76, C81, C84, C86, C89, C94, C96, U11, U19, U20: moved to F.Cu
- C103, C107, C117, C123, C173, C179, C191, C197, C209, C35, C43, C47, C55, C63, C67, C75, C83, C87, C95: value 100nF -> 10nF
- C111, C129, C167, C185, C203, C31, C39, C51, C59, C71, C79, C91, C99: value 100nF -> 10nF; moved to F.Cu
- C143, C145: value 100nF -> C
- C144: value 100nF -> C; moved to F.Cu
- J1: value Conn_02x06_Odd_Even -> Conn_02x16_Odd_Even; footprint Connector_PinSocket_2.54mm:PinSocket_2x06_P2.54mm_Vertical -> Connector_PinHeader_2.54mm:PinHeader_2x16_P2.54mm_Vertical
- J2: value Conn_02x04_Odd_Even -> Conn_02x16_Odd_Even; footprint Connector_PinHeader_2.54mm:PinHeader_2x04_P2.54mm_Vertical -> Connector_PinHeader_2.54mm:PinHeader_2x16_P2.54mm_Vertical
- J3: value Conn_02x16_Odd_Even -> Conn_02x06_Odd_Even; footprint Connector_PinHeader_2.54mm:PinHeader_2x16_P2.54mm_Vertical -> Connector_PinSocket_2.54mm:PinSocket_2x06_P2.54mm_Vertical
- J4: value Conn_02x16_Odd_Even -> Conn_02x04_Odd_Even; footprint Connector_PinHeader_2.54mm:PinHeader_2x16_P2.54mm_Vertical -> Connector_PinHeader_2.54mm:PinHeader_2x04_P2.54mm_Vertical
- J7: value Conn_02x01 -> Conn_02x05_Odd_Even; footprint Connector_PinHeader_2.54mm:PinHeader_2x01_P2.54mm_Horizontal -> Connector_PinHeader_2.54mm:PinHeader_2x05_P2.54mm_Vertical
- J8: value Conn_02x05_Odd_Even -> Conn_02x01; footprint Connector_PinHeader_2.54mm:PinHeader_2x05_P2.54mm_Vertical -> Connector_PinHeader_2.54mm:PinHeader_2x01_P2.54mm_Horizontal
- R14: value 330 -> 500
- R7: value 500 -> 330
- SW13: value SW_SPDT -> SW_DIP_x08; footprint Button_Switch_THT:SW_Slide_SPDT_Straight_CK_OS102011MS2Q -> Button_Switch_THT:SW_DIP_SPSTx08_Slide_9.78x22.5mm_W7.62mm_P2.54mm
- SW14: value SW_DIP_x08 -> SW_Slide_DPDT; footprint Button_Switch_THT:SW_DIP_SPSTx08_Slide_9.78x22.5mm_W7.62mm_P2.54mm -> Button_Switch_SMD:SW_DPDT_CK_JS202011JCQN
- SW16: value SW_Slide_DPDT -> SW_DIP_x08; footprint Button_Switch_SMD:SW_DPDT_CK_JS202011JCQN -> Button_Switch_THT:SW_DIP_SPSTx08_Slide_9.78x22.5mm_W7.62mm_P2.54mm
- SW7: value SW_DIP_x08 -> SW_SPDT; footprint Button_Switch_THT:SW_DIP_SPSTx08_Slide_9.78x22.5mm_W7.62mm_P2.54mm -> Button_Switch_THT:SW_Slide_SPDT_Straight_CK_OS102011MS2Q
- U1: value 74HC86 -> 74LS182; footprint Package_SO:SOIC-14_3.9x8.7mm_P1.27mm -> Package_DIP:DIP-16_W7.62mm; moved to F.Cu
- U10: value 74LS540 -> 74LS377; moved to F.Cu
- U100, U204, U40, U55, U70, U85: value 74AHCT138 -> 74AC251
- U101, U205, U41, U56, U71, U86: value 74LS08 -> 74HC86
- U103, U104, U113, U118, U128, U148, U149, U98, U99: value 74AHCT125 -> 74HC00
- U105, U110, U135, U140, U145, U150: value 74AHCT138 -> 74HC00; footprint Package_SO:SOIC-16_3.9x9.9mm_P1.27mm -> Package_SO:SOIC-14_3.9x8.7mm_P1.27mm
- U106, U111, U121, U136, U141, U146, U91, U96: value 74LS08 -> 74HC00
- U107, U211, U37, U52, U67, U82: value 74HC86 -> 74AC251; footprint Package_SO:SOIC-14_3.9x8.7mm_P1.27mm -> Package_SO:SOIC-16_3.9x9.9mm_P1.27mm
- U108, U170, U198, U212, U38, U44, U53, U59, U68, U74, U83, U89, U94: value 74AHCT125 -> 74HC86
- U112, U117, U122, U127, U92, U97: value 74HC86 -> 74HC00
- U114, U197, U34, U43, U49, U58, U64, U73, U79, U88, U93: value 74AHCT125 -> 74AC251; footprint Package_SO:SOIC-14_3.9x8.7mm_P1.27mm -> Package_SO:SOIC-16_3.9x9.9mm_P1.27mm
- U115, U35, U50, U65, U80: value 74AHCT138 -> 74HC86; footprint Package_SO:SOIC-16_3.9x9.9mm_P1.27mm -> Package_SO:SOIC-14_3.9x8.7mm_P1.27mm
- U12, U7, U9: value 74LS30 -> 74LS182; footprint Package_SO:SOIC-14_3.9x8.7mm_P1.27mm -> Package_DIP:DIP-16_W7.62mm; moved to F.Cu
- U125, U130: value 74AHCT138 -> 74AHC541; footprint Package_SO:SOIC-16_3.9x9.9mm_P1.27mm -> Package_SO:SOIC-20W_7.5x12.8mm_P1.27mm
- U126: value 74LS08 -> KM28C64A; footprint Package_SO:SOIC-14_3.9x8.7mm_P1.27mm -> Package_DIP:DIP-28_W15.24mm
- U129, U133, U134, U138, U139, U143, U144: value 74AHCT125 -> 74AHC541; footprint Package_SO:SOIC-14_3.9x8.7mm_P1.27mm -> Package_SO:SOIC-20W_7.5x12.8mm_P1.27mm
- U131: value 74LS08 -> 74AHC541; footprint Package_SO:SOIC-14_3.9x8.7mm_P1.27mm -> Package_SO:SOIC-20W_7.5x12.8mm_P1.27mm
- U132: value 74HC86 -> KM28C64A; footprint Package_SO:SOIC-14_3.9x8.7mm_P1.27mm -> Package_DIP:DIP-28_W15.24mm
- U137, U142, U147: value 74HC86 -> 74AHC1G04; footprint Package_SO:SOIC-14_3.9x8.7mm_P1.27mm -> Package_TO_SOT_SMD:SOT-23-5
- U15: value 74LS182 -> 74HC86; footprint Package_DIP:DIP-16_W7.62mm -> Package_SO:SOIC-14_3.9x8.7mm_P1.27mm
- U151: value 74LS540 -> 74HC00; footprint Package_SO:SOIC-20W_7.5x12.8mm_P1.27mm -> Package_SO:SOIC-14_3.9x8.7mm_P1.27mm
- U154: value 74LS540 -> 74HC00; footprint Package_SO:SOIC-20W_7.5x12.8mm_P1.27mm -> Package_SO:SOIC-14_3.9x8.7mm_P1.27mm; moved to F.Cu
- U155: value KM28C64A -> 74HC00; footprint Package_DIP:DIP-28_W15.24mm -> Package_SO:SOIC-14_3.9x8.7mm_P1.27mm
- U16: value 74LS30 -> 74LS32; moved to F.Cu
- U162: value 74AHC1G04 -> 74AC251; footprint Package_TO_SOT_SMD:SOT-23-5 -> Package_SO:SOIC-16_3.9x9.9mm_P1.27mm
- U163: value 74AHC541 -> 74HC86; footprint Package_SO:SOIC-20W_7.5x12.8mm_P1.27mm -> Package_SO:SOIC-14_3.9x8.7mm_P1.27mm
- U169: value 74AHC541 -> 74AC251; footprint Package_SO:SOIC-20W_7.5x12.8mm_P1.27mm -> Package_SO:SOIC-16_3.9x9.9mm_P1.27mm; moved to F.Cu
- U17, U18, U23, U24: value 74LS182 -> 74LS30; footprint Package_DIP:DIP-16_W7.62mm -> Package_SO:SOIC-14_3.9x8.7mm_P1.27mm
- U176: value 74LS163 -> 74AC251
- U177: value 74LS154 -> 74HC86; footprint Package_SO:SOIC-24W_7.5x15.4mm_P1.27mm -> Package_SO:SOIC-14_3.9x8.7mm_P1.27mm
- U183: value 74LS540 -> 74AC251; footprint Package_SO:SOIC-20W_7.5x12.8mm_P1.27mm -> Package_SO:SOIC-16_3.9x9.9mm_P1.27mm
- U184: value 74LS540 -> 74HC86; footprint Package_SO:SOIC-20W_7.5x12.8mm_P1.27mm -> Package_SO:SOIC-14_3.9x8.7mm_P1.27mm
- U190, U31, U46, U61, U76: value 74LS08 -> 74AC251; footprint Package_SO:SOIC-14_3.9x8.7mm_P1.27mm -> Package_SO:SOIC-16_3.9x9.9mm_P1.27mm
- U2: value 74LS153 -> 74LS182; footprint Package_SO:SOIC-16_3.9x9.9mm_P1.27mm -> Package_DIP:DIP-16_W7.62mm; moved to F.Cu
- U21: value 74LS182 -> 74AHCT1G08; footprint Package_DIP:DIP-16_W7.62mm -> Package_TO_SOT_SMD:SOT-23-5
- U22: value 74LS182 -> 74LS153; footprint Package_DIP:DIP-16_W7.62mm -> Package_SO:SOIC-16_3.9x9.9mm_P1.27mm
- U25, U26: value 74LS182 -> 74LS540; footprint Package_DIP:DIP-16_W7.62mm -> Package_SO:SOIC-20W_7.5x12.8mm_P1.27mm
- U27: value 74LS540 -> 74AHCT1G08; footprint Package_SO:SOIC-20W_7.5x12.8mm_P1.27mm -> Package_TO_SOT_SMD:SOT-23-5
- U28: value 74LS377 -> 74AHC541
- U29: value 74LS377 -> 74AHC541; moved to F.Cu
- U3: value 74AHC541 -> 74LS182; footprint Package_SO:SOIC-20W_7.5x12.8mm_P1.27mm -> Package_DIP:DIP-16_W7.62mm
- U30: value 74AHCT1G08 -> 74AHC1G04; moved to F.Cu
- U4: value 74LS32 -> 74LS182; footprint Package_SO:SOIC-14_3.9x8.7mm_P1.27mm -> Package_DIP:DIP-16_W7.62mm; moved to F.Cu
- U5: value 74AHCT1G08 -> 74LS377; footprint Package_TO_SOT_SMD:SOT-23-5 -> Package_SO:SOIC-20W_7.5x12.8mm_P1.27mm
- U6: value 74AHC1G04 -> 74LS182; footprint Package_TO_SOT_SMD:SOT-23-5 -> Package_DIP:DIP-16_W7.62mm
- U8: value 74AHC541 -> 74LS182; footprint Package_SO:SOIC-20W_7.5x12.8mm_P1.27mm -> Package_DIP:DIP-16_W7.62mm; moved to F.Cu
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Connections:
- C105 pad 1: GND -> VCC
- C105 pad 2: VCC -> GND
- C107 pad 1: VCC -> GND
- C107 pad 2: GND -> VCC
- C109 pad 1: GND -> VCC
- C109 pad 2: VCC -> GND
- C110 pad 1: GND -> VCC
- C110 pad 2: VCC -> GND
- C111 pad 1: VCC -> GND
- C111 pad 2: GND -> VCC
- C114 pad 1: GND -> VCC
- C114 pad 2: VCC -> GND
- C115 pad 1: GND -> VCC
- C115 pad 2: VCC -> GND
- C117 pad 1: VCC -> GND
- C117 pad 2: GND -> VCC
- C120 pad 1: GND -> VCC
- C120 pad 2: VCC -> GND
- C131 pad 1: VCC -> GND
- C131 pad 2: GND -> VCC
- C133 pad 1: GND -> VCC
- C133 pad 2: VCC -> GND
- C140 pad 1: GND -> VCC
- C140 pad 2: VCC -> GND
- C141 pad 1: VCC -> GND
- C141 pad 2: GND -> VCC
- C143 pad 1: GND -> VCC
- C143 pad 2: VCC -> GND
- C146 pad 1: VCC -> GND
- C146 pad 2: GND -> VCC
- C147 pad 1: VCC -> GND
- C147 pad 2: GND -> VCC
- C158 pad 1: VCC -> GND
- C158 pad 2: GND -> VCC
- C170 pad 1: GND -> VCC
- C170 pad 2: VCC -> GND
- C171 pad 1: GND -> VCC
- C171 pad 2: VCC -> GND
- C173 pad 1: VCC -> GND
- C173 pad 2: GND -> VCC
- C175 pad 1: VCC -> GND
- C175 pad 2: GND -> VCC
- C179 pad 1: VCC -> GND
- C179 pad 2: GND -> VCC
- C182 pad 1: GND -> VCC
- C182 pad 2: VCC -> GND
- C183 pad 1: GND -> VCC
- C183 pad 2: VCC -> GND
- C185 pad 1: VCC -> GND
- C185 pad 2: GND -> VCC
- C188 pad 1: GND -> VCC
- C188 pad 2: VCC -> GND
- C189 pad 1: GND -> VCC
- C189 pad 2: VCC -> GND
- C191 pad 1: VCC -> GND
- C191 pad 2: GND -> VCC
- C194 pad 1: GND -> VCC
- C194 pad 2: VCC -> GND
- C205 pad 1: VCC -> GND
- C205 pad 2: GND -> VCC
- C207 pad 1: GND -> VCC
- C207 pad 2: VCC -> GND
- C211 pad 1: VCC -> GND
- C211 pad 2: GND -> VCC
- C212 pad 1: GND -> VCC
- C212 pad 2: VCC -> GND
- C213 pad 1: GND -> VCC
- C213 pad 2: VCC -> GND
- C31 pad 1: VCC -> GND
- C31 pad 2: GND -> VCC
- C32 pad 1: VCC -> GND
- C32 pad 2: GND -> VCC
- C33 pad 1: GND -> VCC
- C33 pad 2: VCC -> GND
- C34 pad 1: GND -> VCC
- C34 pad 2: VCC -> GND
- C36 pad 1: VCC -> GND
- C36 pad 2: GND -> VCC
- C38 pad 1: GND -> VCC
- C38 pad 2: VCC -> GND
- C45 pad 1: GND -> VCC
- C45 pad 2: VCC -> GND
- C47 pad 1: VCC -> GND
- C47 pad 2: GND -> VCC
- C49 pad 1: GND -> VCC
- C49 pad 2: VCC -> GND
- C50 pad 1: GND -> VCC
- C50 pad 2: VCC -> GND
- C51 pad 1: VCC -> GND
- C51 pad 2: GND -> VCC
- C52 pad 1: VCC -> GND
- C52 pad 2: GND -> VCC
- C53 pad 1: GND -> VCC
- C53 pad 2: VCC -> GND
- C54 pad 1: GND -> VCC
- C54 pad 2: VCC -> GND
- C56 pad 1: VCC -> GND
- C56 pad 2: GND -> VCC
- C58 pad 1: GND -> VCC
- C58 pad 2: VCC -> GND
- C65 pad 1: GND -> VCC
- C65 pad 2: VCC -> GND
- C67 pad 1: VCC -> GND
- C67 pad 2: GND -> VCC
- C69 pad 1: GND -> VCC
- C69 pad 2: VCC -> GND
- C70 pad 1: GND -> VCC
- C70 pad 2: VCC -> GND
- C71 pad 1: VCC -> GND
- C71 pad 2: GND -> VCC
- C72 pad 1: VCC -> GND
- C72 pad 2: GND -> VCC
- C73 pad 1: GND -> VCC
- C73 pad 2: VCC -> GND
- C74 pad 1: GND -> VCC
- C74 pad 2: VCC -> GND
- C76 pad 1: VCC -> GND
- C76 pad 2: GND -> VCC
- C78 pad 1: GND -> VCC
- C78 pad 2: VCC -> GND
- C85 pad 1: GND -> VCC
- C85 pad 2: VCC -> GND
- C87 pad 1: VCC -> GND
- C87 pad 2: GND -> VCC
- C89 pad 1: GND -> VCC
- C89 pad 2: VCC -> GND
- C90 pad 1: GND -> VCC
- C90 pad 2: VCC -> GND
- C91 pad 1: VCC -> GND
- C91 pad 2: GND -> VCC
- C92 pad 1: VCC -> GND
- C92 pad 2: GND -> VCC
- C93 pad 1: GND -> VCC
- C93 pad 2: VCC -> GND
- C94 pad 1: GND -> VCC
- C94 pad 2: VCC -> GND
- C96 pad 1: VCC -> GND
- C96 pad 2: GND -> VCC
- C98 pad 1: GND -> VCC
- C98 pad 2: VCC -> GND
- J1 pad 1: flagZ -> A0
- J1 pad 10: flagLTE -> A27
- J1 pad 11: flagGT -> A5
- J1 pad 12: flagGTE -> A26
- J1 pad 2: ~flagZ -> A31
- J1 pad 3: flagN -> A1
- J1 pad 4: ~flagN -> A30
- J1 pad 5: flagC -> A2
- J1 pad 6: ~flagC -> A29
- J1 pad 7: flagV -> A3
- J1 pad 8: ~flagV -> A28
- J1 pad 9: flagLT -> A4
- J2 pad 1: VCC -> B0
- J2 pad 2: GND -> B31
- J2 pad 3: VCC -> B1
- J2 pad 4: GND -> B30
- J2 pad 5: VCC -> B2
- J2 pad 6: GND -> B29
- J2 pad 7: VCC -> B3
- J2 pad 8: GND -> B28
- J3 pad 1: A0 -> flagZ
- J3 pad 10: A27 -> flagLTE
- J3 pad 11: A5 -> flagGT
- J3 pad 12: A26 -> flagGTE
- J3 pad 2: A31 -> ~flagZ
- J3 pad 3: A1 -> flagN
- J3 pad 4: A30 -> ~flagN
- J3 pad 5: A2 -> flagC
- J3 pad 6: A29 -> ~flagC
- J3 pad 7: A3 -> flagV
- J3 pad 8: A28 -> ~flagV
- J3 pad 9: A4 -> flagLT
- J4 pad 1: C0 -> VCC
- J4 pad 2: C31 -> GND
- J4 pad 3: C1 -> VCC
- J4 pad 4: C30 -> GND
- J4 pad 5: C2 -> VCC
- J4 pad 6: C29 -> GND
- J4 pad 7: C3 -> VCC
- J4 pad 8: C28 -> GND
- J5 pad 1: B0 -> C0
- J5 pad 10: B27 -> C27
- J5 pad 11: B5 -> C5
- J5 pad 12: B25 -> C26
- J5 pad 13: B6 -> C6
- J5 pad 14: B26 -> C25
- J5 pad 15: B7 -> C7
- J5 pad 16: B24 -> C24
- J5 pad 17: B8 -> C8
- J5 pad 18: B23 -> C23
- J5 pad 19: B9 -> C9
- J5 pad 2: B31 -> C31
- J5 pad 20: B22 -> C22
- J5 pad 21: B10 -> C10
- J5 pad 22: B21 -> C21
- J5 pad 23: B11 -> C11
- J5 pad 24: B20 -> C20
- J5 pad 25: B12 -> C12
- J5 pad 26: B19 -> C19
- J5 pad 27: B13 -> C13
- J5 pad 28: B18 -> C18
- J5 pad 29: B14 -> C14
- J5 pad 3: B1 -> C1
- J5 pad 30: B17 -> C17
- J5 pad 31: B15 -> C15
- J5 pad 32: B16 -> C16
- J5 pad 4: B30 -> C30
- J5 pad 5: B2 -> C2
- J5 pad 6: B29 -> C29
- J5 pad 7: B3 -> C3
- J5 pad 8: B28 -> C28
- J5 pad 9: B4 -> C4
- J7 pad 2: Net-(J7-Pin_1) -> Net-(J7-Pin_2)
- J8 pad 2: Net-(J8-Pin_2) -> Net-(J8-Pin_1)
- R10 pad 1: flagC -> flagLT
- R11 pad 1: flagV -> flagGTE
- R12 pad 1: flagLT -> flagGT
- R13 pad 1: flagGT -> VCC
- R14 pad 1: VCC -> /iN_Mode
- R2 pad 1: ~flagN -> flagZ
- R3 pad 1: ~flagC -> ~flagN
- R4 pad 1: ~flagV -> flagN
- R5 pad 1: flagLTE -> ~flagC
- R6 pad 1: flagGTE -> flagC
- R7 pad 1: /iN_Mode -> ~flagV
- R8 pad 1: flagZ -> flagV
- R9 pad 1: flagN -> flagLTE
- SW1 pad 10: A14 -> A6
- SW1 pad 11: A13 -> A5
- SW1 pad 12: A12 -> A4
- SW1 pad 13: A11 -> A3
- SW1 pad 14: A10 -> A2
- SW1 pad 15: A9 -> A1
- SW1 pad 16: A8 -> A0
- SW1 pad 9: A15 -> A7
- SW10 pad 10: B30 -> C14
- SW10 pad 11: B29 -> C13
- SW10 pad 12: B28 -> C12
- SW10 pad 13: B27 -> C11
- SW10 pad 14: B25 -> C10
- SW10 pad 15: B26 -> C9
- SW10 pad 16: B24 -> C8
- SW10 pad 9: B31 -> C15
- SW11 pad 10: C22 -> A30
- SW11 pad 11: C21 -> A29
- SW11 pad 12: C20 -> A28
- SW11 pad 13: C19 -> A27
- SW11 pad 14: C18 -> A26
- SW11 pad 15: C17 -> A25
- SW11 pad 16: C16 -> A24
- SW11 pad 9: C23 -> A31
- SW12 pad 10: C30 -> B30
- SW12 pad 11: C29 -> B29
- SW12 pad 12: C28 -> B28
- SW12 pad 13: C27 -> B27
- SW12 pad 14: C26 -> B25
- SW12 pad 15: C25 -> B26
- SW12 pad 16: C24 -> B24
- SW12 pad 9: C31 -> B31
- SW13 pad 2: VCC -> /iN_Mode
- SW13 pad 3: unconnected-(SW13-C-Pad3) -> /iN_Mode
- SW14 pad 1: /alu_control/SW_EN -> VCC
- SW14 pad 2: /alu_control/SW_EN -> /alu-control/Ctrl_EN
- SW14 pad 3: /alu_control/SW_EN -> GND
- SW14 pad 4: /alu_control/SW_EN -> unconnected-(SW14-A-Pad4)
- SW14 pad 5: /alu_control/SW_EN -> /alu-control/SW_EN
- SW14 pad 6: /alu_control/SW_EN -> VCC
- SW15 pad 1: /alu_control/Override -> /alu-control/SW_EN
- SW15 pad 10: flagWE -> ALU-OPCODE6
- SW15 pad 11: csel1 -> ALU-OPCODE5
- SW15 pad 12: csel0 -> ALU-OPCODE4
- SW15 pad 13: binv -> ALU-OPCODE3
- SW15 pad 14: bsel -> ALU-OPCODE2
- SW15 pad 15: ainv -> ALU-OPCODE1
- SW15 pad 16: asel -> ALU-OPCODE0
- SW15 pad 2: /alu_control/Override -> /alu-control/SW_EN
- SW15 pad 3: /alu_control/Override -> /alu-control/SW_EN
- SW15 pad 4: /alu_control/Override -> /alu-control/SW_EN
- SW15 pad 5: /alu_control/Override -> /alu-control/SW_EN
- SW15 pad 6: /alu_control/Override -> /alu-control/SW_EN
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Routing:
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- removed copper zone on In1.Cu, net GND
- removed copper zone on In2.Cu, net VCC
Other:
- board text removed: "Tomato32 ALU"
- board text removed: "Tyrone Marhguy, 2026 Computer Engineering, BSE University of Pennsylvania"

Commit message: checkpoint: placed components for optimized routing on alu-32b board pcb
Parts:
- removed C1, C10, C101, C105, C109, C11, C113, C115, C119, C12, C121, C125, C127, C13, C131, C132, C133, C14, C140, C141, C146, C147, C148, C15, C150, C151, C152, C154, C155, C156, C158, C169, C17, C170, C171, C175, C176, C177, C181, C182, C183, C187, C188, C189, C19, C193, C194, C195, C199, C2, C200, C201, C205, C206, C207, C21, C211, C212, C213, C23, C25, C27, C29, C3, C33, C37, C4, C41, C45, C49, C5, C53, C57, C6, C61, C65, C69, C7, C73, C77, C8, C81, C85, C89, C9, C93, C97: 100nF, Capacitor_SMD:C_0603_1608Metric
- removed C103, C107, C111, C117, C123, C129, C167, C173, C179, C185, C191, C197, C203, C209, C31, C35, C39, C43, C47, C51, C55, C59, C63, C67, C71, C75, C79, C83, C87, C91, C95, C99: 10nF, Capacitor_SMD:C_0603_1608Metric
- removed C143, C144, C145: C, Capacitor_SMD:C_0603_1608Metric
- removed D1, D10, D11, D12, D2, D3, D4, D5, D6, D7, D8, D9: LED, LED_SMD:LED_0805_2012Metric
- removed J6: Conn_02x16_Counter_Clockwise, Connector_PinSocket_2.54mm:PinSocket_2x16_P2.54mm_Vertical
- removed J7: Conn_02x05_Odd_Even, Connector_PinHeader_2.54mm:PinHeader_2x05_P2.54mm_Vertical
- removed J8: Conn_02x01, Connector_PinHeader_2.54mm:PinHeader_2x01_P2.54mm_Horizontal
- removed R1, R10, R11, R12, R2, R3, R4, R5, R6, R7, R8, R9: 330, Resistor_SMD:R_0603_1608Metric
- removed SW14: SW_Slide_DPDT, Button_Switch_SMD:SW_DPDT_CK_JS202011JCQN
- removed SW15, SW16: SW_DIP_x08, Button_Switch_THT:SW_DIP_SPSTx08_Slide_9.78x22.5mm_W7.62mm_P2.54mm
- removed U1, U12, U13, U14, U2, U3, U4, U6, U7, U8, U9: 74LS182, Package_DIP:DIP-16_W7.62mm
- removed U10, U5: 74LS377, Package_SO:SOIC-20W_7.5x12.8mm_P1.27mm
- removed U100, U107, U114, U162, U169, U176, U183, U190, U197, U204, U211, U46, U55, U58, U76, U85, U88: 74AC251, Package_SO:SOIC-16_3.9x9.9mm_P1.27mm
- removed U101, U108, U115, U15, U163, U170, U177, U184, U191, U198, U205, U212, U35, U38, U56, U65, U68, U86: 74HC86, Package_SO:SOIC-14_3.9x8.7mm_P1.27mm
- removed U103, U104, U105, U106, U110, U111, U112, U113, U117, U118, U121, U122, U127, U128, U135, U136, U140, U141, U145, U146, U148, U149, U150, U151, U154, U155, U96, U97, U98, U99: 74HC00, Package_SO:SOIC-14_3.9x8.7mm_P1.27mm
- removed U11, U25, U26: 74LS540, Package_SO:SOIC-20W_7.5x12.8mm_P1.27mm
- removed U125, U129, U130, U131, U133, U134, U138, U139, U143, U144, U28: 74AHC541, Package_SO:SOIC-20W_7.5x12.8mm_P1.27mm
- removed U126, U132: KM28C64A, Package_DIP:DIP-28_W15.24mm
- removed U137, U142, U147: 74AHC1G04, Package_TO_SOT_SMD:SOT-23-5
- removed U16: 74LS32, Package_SO:SOIC-14_3.9x8.7mm_P1.27mm
- removed U18: 74LS30, Package_SO:SOIC-14_3.9x8.7mm_P1.27mm
- added C112: 100nF, Capacitor_SMD:C_0603_1608Metric, F.Cu at (192.7, 126.6)
- added C116: 100nF, Capacitor_SMD:C_0603_1608Metric, F.Cu at (130.7, 153.1)
- added C118: 100nF, Capacitor_SMD:C_0603_1608Metric, F.Cu at (130.7, 163.8)
- added C122: 100nF, Capacitor_SMD:C_0603_1608Metric, F.Cu at (150.4, 148.1)
- added C124: 100nF, Capacitor_SMD:C_0603_1608Metric, F.Cu at (150.4, 136.6)
- added RN1: R_Network08, Resistor_THT:R_Array_SIP9, F.Cu at (125.2, 81.8)
- added RN10: R_Network08, Resistor_THT:R_Array_SIP9, F.Cu at (282.8, 93.2)
- added RN11: R_Network08, Resistor_THT:R_Array_SIP9, F.Cu at (282.8, 81.8)
- added RN12: R_Network08, Resistor_THT:R_Array_SIP9, F.Cu at (237.7, 81.8)
- added RN2: R_Network08, Resistor_THT:R_Array_SIP9, F.Cu at (170.3, 81.8)
- added RN3: R_Network08, Resistor_THT:R_Array_SIP9, F.Cu at (170.3, 93.2)
- added RN4: R_Network08, Resistor_THT:R_Array_SIP9, F.Cu at (125.2, 93.2)
- added RN5: R_Network08, Resistor_THT:R_Array_SIP9, F.Cu at (182.1, 93.2)
- added RN6: R_Network08, Resistor_THT:R_Array_SIP9, F.Cu at (227.3, 93.2)
- added RN7: R_Network08, Resistor_THT:R_Array_SIP9, F.Cu at (227.3, 81.9)
- added RN8: R_Network08, Resistor_THT:R_Array_SIP9, F.Cu at (182.1, 81.8)
- added RN9: R_Network08, Resistor_THT:R_Array_SIP9, F.Cu at (237.7, 93.2)
- added U33: 74AC251, Package_SO:SOIC-16_3.9x9.9mm_P1.27mm, F.Cu at (178.5, 210.2)
- added U39: 74HC00, Package_SO:SOIC-14_3.9x8.7mm_P1.27mm, F.Cu at (229.6, 205.4)
- added U42: 74AC251, Package_SO:SOIC-16_3.9x9.9mm_P1.27mm, F.Cu at (220.8, 222.4)
- added U51: 74AC251, Package_SO:SOIC-16_3.9x9.9mm_P1.27mm, F.Cu at (263.1, 199.2)
- added U54: 74AC251, Package_SO:SOIC-16_3.9x9.9mm_P1.27mm, F.Cu at (263.1, 234.0)
- added U57: 74HC86, Package_SO:SOIC-14_3.9x8.7mm_P1.27mm, F.Cu at (263.0, 138.1)
- added U60: 74LS283, Package_SO:SOIC-16_3.9x9.9mm_P1.27mm, F.Cu at (263.0, 149.1)
- added U63: 74AC251, Package_SO:SOIC-16_3.9x9.9mm_P1.27mm, F.Cu at (271.8, 154.7)
- added U69: 74HC00, Package_SO:SOIC-14_3.9x8.7mm_P1.27mm, F.Cu at (220.7, 160.5)
- added U72: 74AC251, Package_SO:SOIC-16_3.9x9.9mm_P1.27mm, F.Cu at (229.5, 143.5)
- added U81: 74AC251, Package_SO:SOIC-16_3.9x9.9mm_P1.27mm, F.Cu at (187.2, 166.7)
- added U84: 74AC251, Package_SO:SOIC-16_3.9x9.9mm_P1.27mm, F.Cu at (187.2, 131.9)
- added U87: 74HC86, Package_SO:SOIC-14_3.9x8.7mm_P1.27mm, F.Cu at (136.1, 136.8)
- added U90: 74LS283, Package_SO:SOIC-16_3.9x9.9mm_P1.27mm, F.Cu at (136.1, 147.8)
- J3: value Conn_02x06_Odd_Even -> Conn_02x04_Odd_Even; footprint Connector_PinSocket_2.54mm:PinSocket_2x06_P2.54mm_Vertical -> Connector_PinHeader_2.54mm:PinHeader_2x04_P2.54mm_Vertical
- J4: value Conn_02x04_Odd_Even -> Conn_02x16_Odd_Even; footprint Connector_PinHeader_2.54mm:PinHeader_2x04_P2.54mm_Vertical -> Connector_PinHeader_2.54mm:PinHeader_2x16_P2.54mm_Vertical
- J5: value Conn_02x16_Odd_Even -> Conn_02x16_Counter_Clockwise; footprint Connector_PinHeader_2.54mm:PinHeader_2x16_P2.54mm_Vertical -> Connector_PinSocket_2.54mm:PinSocket_2x16_P2.54mm_Vertical
- U17: value 74LS30 -> 74HC86
- U19: value 74LS540 -> 74HC00; footprint Package_SO:SOIC-20W_7.5x12.8mm_P1.27mm -> Package_SO:SOIC-14_3.9x8.7mm_P1.27mm
- U20: value 74LS540 -> 74LS283; footprint Package_SO:SOIC-20W_7.5x12.8mm_P1.27mm -> Package_SO:SOIC-16_3.9x9.9mm_P1.27mm
- U21: value 74AHCT1G08 -> 74AC251; footprint Package_TO_SOT_SMD:SOT-23-5 -> Package_SO:SOIC-16_3.9x9.9mm_P1.27mm
- U22: value 74LS153 -> 74AC251
- U23, U24: value 74LS30 -> 74AC251; footprint Package_SO:SOIC-14_3.9x8.7mm_P1.27mm -> Package_SO:SOIC-16_3.9x9.9mm_P1.27mm
- U27: value 74AHCT1G08 -> 74HC86; footprint Package_TO_SOT_SMD:SOT-23-5 -> Package_SO:SOIC-14_3.9x8.7mm_P1.27mm
- U29: value 74AHC541 -> 74HC00; footprint Package_SO:SOIC-20W_7.5x12.8mm_P1.27mm -> Package_SO:SOIC-14_3.9x8.7mm_P1.27mm
- U30: value 74AHC1G04 -> 74LS283; footprint Package_TO_SOT_SMD:SOT-23-5 -> Package_SO:SOIC-16_3.9x9.9mm_P1.27mm
- U32, U41, U44, U53, U62, U71, U74, U83, U94: value 74HC86 -> 74AC251; footprint Package_SO:SOIC-14_3.9x8.7mm_P1.27mm -> Package_SO:SOIC-16_3.9x9.9mm_P1.27mm
- U37, U67: value 74AC251 -> 74HC86; footprint Package_SO:SOIC-16_3.9x9.9mm_P1.27mm -> Package_SO:SOIC-14_3.9x8.7mm_P1.27mm
- U40, U70: value 74AC251 -> 74LS283
- U49, U79: value 74AC251 -> 74HC00; footprint Package_SO:SOIC-16_3.9x9.9mm_P1.27mm -> Package_SO:SOIC-14_3.9x8.7mm_P1.27mm
- U50, U80: value 74HC86 -> 74LS283; footprint Package_SO:SOIC-14_3.9x8.7mm_P1.27mm -> Package_SO:SOIC-16_3.9x9.9mm_P1.27mm
- U59, U89: value 74HC86 -> 74HC00
- U91, U92: value 74HC00 -> 74AC251; footprint Package_SO:SOIC-14_3.9x8.7mm_P1.27mm -> Package_SO:SOIC-16_3.9x9.9mm_P1.27mm
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Connections:
- C102 pad 1: VCC -> GND
- C102 pad 2: GND -> VCC
- C106 pad 1: VCC -> GND
- C106 pad 2: GND -> VCC
- C110 pad 1: VCC -> GND
- C110 pad 2: GND -> VCC
- C114 pad 1: VCC -> GND
- C114 pad 2: GND -> VCC
- C120 pad 1: VCC -> GND
- C120 pad 2: GND -> VCC
- C126 pad 1: VCC -> GND
- C126 pad 2: GND -> VCC
- C34 pad 1: VCC -> GND
- C34 pad 2: GND -> VCC
- C38 pad 1: VCC -> GND
- C38 pad 2: GND -> VCC
- C42 pad 1: VCC -> GND
- C42 pad 2: GND -> VCC
- C46 pad 1: VCC -> GND
- C46 pad 2: GND -> VCC
- C50 pad 1: VCC -> GND
- C50 pad 2: GND -> VCC
- C54 pad 1: VCC -> GND
- C54 pad 2: GND -> VCC
- C58 pad 1: VCC -> GND
- C58 pad 2: GND -> VCC
- C62 pad 1: VCC -> GND
- C62 pad 2: GND -> VCC
- C66 pad 1: VCC -> GND
- C66 pad 2: GND -> VCC
- C70 pad 1: VCC -> GND
- C70 pad 2: GND -> VCC
- C74 pad 1: VCC -> GND
- C74 pad 2: GND -> VCC
- C78 pad 1: VCC -> GND
- C78 pad 2: GND -> VCC
- C82 pad 1: VCC -> GND
- C82 pad 2: GND -> VCC
- C86 pad 1: VCC -> GND
- C86 pad 2: GND -> VCC
- C90 pad 1: VCC -> GND
- C90 pad 2: GND -> VCC
- C94 pad 1: VCC -> GND
- C94 pad 2: GND -> VCC
- C98 pad 1: VCC -> GND
- C98 pad 2: GND -> VCC
- J3 pad 1: flagZ -> VCC
- J3 pad 2: ~flagZ -> GND
- J3 pad 3: flagN -> VCC
- J3 pad 4: ~flagN -> GND
- J3 pad 5: flagC -> VCC
- J3 pad 6: ~flagC -> GND
- J3 pad 7: flagV -> VCC
- J3 pad 8: ~flagV -> GND
- J4 pad 1: VCC -> C0
- J4 pad 2: GND -> C31
- J4 pad 3: VCC -> C1
- J4 pad 4: GND -> C30
- J4 pad 5: VCC -> C2
- J4 pad 6: GND -> C29
- J4 pad 7: VCC -> C3
- J4 pad 8: GND -> C28
- J5 pad 1: C0 -> OUT0
- J5 pad 10: C27 -> OUT9
- J5 pad 11: C5 -> OUT10
- J5 pad 12: C26 -> OUT11
- J5 pad 13: C6 -> OUT12
- J5 pad 14: C25 -> OUT13
- J5 pad 15: C7 -> OUT14
- J5 pad 16: C24 -> OUT15
- J5 pad 17: C8 -> OUT16
- J5 pad 18: C23 -> OUT17
- J5 pad 19: C9 -> OUT18
- J5 pad 2: C31 -> OUT1
- J5 pad 20: C22 -> OUT19
- J5 pad 21: C10 -> OUT20
- J5 pad 22: C21 -> OUT21
- J5 pad 23: C11 -> OUT22
- J5 pad 24: C20 -> OUT23
- J5 pad 25: C12 -> OUT24
- J5 pad 26: C19 -> OUT25
- J5 pad 27: C13 -> OUT26
- J5 pad 28: C18 -> OUT27
- J5 pad 29: C14 -> OUT28
- J5 pad 3: C1 -> OUT2
- J5 pad 30: C17 -> OUT29
- J5 pad 31: C15 -> OUT30
- J5 pad 32: C16 -> OUT31
- J5 pad 4: C30 -> OUT3
- J5 pad 5: C2 -> OUT4
- J5 pad 6: C29 -> OUT5
- J5 pad 7: C3 -> OUT6
- J5 pad 8: C28 -> OUT7
- J5 pad 9: C4 -> OUT8
- U17 pad 1: Net-(U19-Y0) -> Net-(U17-Pad1)
- U17 pad 10: (no net) -> binv
- U17 pad 11: Net-(U19-Y6) -> /alu-4b-0/sB3
- U17 pad 13: (no net) -> binv
- U17 pad 2: Net-(U19-Y1) -> binv
- U17 pad 3: Net-(U19-Y2) -> /alu-4b-0/sB0
- U17 pad 4: Net-(U19-Y3) -> Net-(U17-Pad4)
- U17 pad 5: Net-(U19-Y4) -> binv
- U17 pad 6: Net-(U19-Y5) -> /alu-4b-0/sB1
- U17 pad 8: Net-(U16-Pad2) -> /alu-4b-0/sB2
- U17 pad 9: (no net) -> Net-(U17-Pad9)
- U19 pad 1: GND -> B0
- U19 pad 10: GND -> bsel
- U19 pad 12: Net-(U19-Y6) -> B3
- U19 pad 13: Net-(U19-Y5) -> bsel
- U19 pad 14: Net-(U19-Y4) -> VCC
- U19 pad 2: OUT0 -> bsel
- U19 pad 3: OUT1 -> Net-(U17-Pad1)
- U19 pad 4: OUT2 -> B1
- U19 pad 5: OUT3 -> bsel
- U19 pad 6: OUT4 -> Net-(U17-Pad4)
- U19 pad 7: OUT5 -> GND
- U19 pad 8: OUT6 -> Net-(U17-Pad9)
- U19 pad 9: OUT7 -> B2
- U20 pad 1: GND -> OUT1
- U20 pad 10: GND -> OUT3
- U20 pad 11: Net-(U20-Y7) -> /alu-4b-0/sB3
- U20 pad 12: Net-(U20-Y6) -> /alu-4b-0/log3
- U20 pad 13: Net-(U20-Y5) -> OUT2
- U20 pad 14: Net-(U20-Y4) -> /alu-4b-0/log2
- U20 pad 15: Net-(U20-Y3) -> /alu-4b-0/sB2
- U20 pad 16: Net-(U20-Y2) -> VCC
- U20 pad 2: OUT16 -> /alu-4b-0/sB1
- U20 pad 3: OUT17 -> /alu-4b-0/log1
- U20 pad 4: OUT18 -> OUT0
- U20 pad 5: OUT19 -> /alu-4b-0/log0
- U20 pad 6: OUT20 -> /alu-4b-0/sB0
- U20 pad 7: OUT21 -> cin-main
- U20 pad 8: OUT22 -> GND
- U20 pad 9: OUT23 -> /cout0
- U21 pad 1: ~ZOUT -> ALU-OPCODE3
- U21 pad 2: LT-SIGN -> ALU-OPCODE2
- U21 pad 3: GND -> ALU-OPCODE1
- U21 pad 4: GT-SIGN -> ALU-OPCODE0
- U21 pad 5: VCC -> /alu-4b-0/log0
- U22 pad 1: unconnected-(U22-Ea-Pad1) -> ALU-OPCODE3
- U22 pad 10: GND -> B1
- U22 pad 11: VCC -> A1
- U22 pad 12: flagC -> ALU-OPCODE7
- U22 pad 13: C0 -> ALU-OPCODE6
- U22 pad 14: csel0 -> ALU-OPCODE5
- U22 pad 15: GND -> ALU-OPCODE4
- U22 pad 2: csel1 -> ALU-OPCODE2
- U22 pad 3: unconnected-(U22-I3a-Pad3) -> ALU-OPCODE1
- U22 pad 4: unconnected-(U22-I2a-Pad4) -> ALU-OPCODE0
- U22 pad 5: unconnected-(U22-I1a-Pad5) -> /alu-4b-0/log1
- U22 pad 7: unconnected-(U22-Za-Pad7) -> GND
- U22 pad 9: Ceff0 -> C1
- U23 pad 1: Net-(U25-Y0) -> ALU-OPCODE3
- U23 pad 10: (no net) -> B2
- U23 pad 11: Net-(U25-Y6) -> A2
- U23 pad 12: Net-(U25-Y7) -> ALU-OPCODE7
- U23 pad 13: (no net) -> ALU-OPCODE6
- U23 pad 14: VCC -> ALU-OPCODE5
- U23 pad 2: Net-(U25-Y1) -> ALU-OPCODE2
- U23 pad 3: Net-(U25-Y2) -> ALU-OPCODE1
- U23 pad 4: Net-(U25-Y3) -> ALU-OPCODE0
- U23 pad 5: Net-(U25-Y4) -> /alu-4b-0/log2
- U23 pad 6: Net-(U25-Y5) -> unconnected-(U23-~{Y}-Pad6)
- U23 pad 8: Net-(U16-Pad4) -> GND
- U23 pad 9: (no net) -> C2
- U24 pad 1: Net-(U26-Y0) -> ALU-OPCODE3
- U24 pad 10: (no net) -> B3
- U24 pad 11: Net-(U26-Y6) -> A3
- U24 pad 12: Net-(U26-Y7) -> ALU-OPCODE7
- U24 pad 13: (no net) -> ALU-OPCODE6
- U24 pad 14: VCC -> ALU-OPCODE5
- U24 pad 2: Net-(U26-Y1) -> ALU-OPCODE2
- U24 pad 3: Net-(U26-Y2) -> ALU-OPCODE1
- U24 pad 4: Net-(U26-Y3) -> ALU-OPCODE0
- U24 pad 5: Net-(U26-Y4) -> /alu-4b-0/log3
- U24 pad 6: Net-(U26-Y5) -> unconnected-(U24-~{Y}-Pad6)
- U24 pad 8: Net-(U16-Pad5) -> GND
- U24 pad 9: (no net) -> C3
- U27 pad 1: csel0 -> Net-(U27-Pad1)
- U27 pad 2: csel1 -> binv
- U27 pad 3: GND -> /alu-4b-1/sB0
- U27 pad 4: CIN-SEL -> Net-(U27-Pad4)
- U27 pad 5: VCC -> binv
- U29 pad 1: Net-(U29-G1) -> B4
- U29 pad 10: GND -> bsel
- U29 pad 11: unconnected-(U29-Y7-Pad11) -> Net-(U27-Pad12)
- U29 pad 12: Ceff7 -> B7
- U29 pad 13: Ceff6 -> bsel
- U29 pad 14: Ceff5 -> VCC
- U29 pad 2: C1 -> bsel
- U29 pad 3: C2 -> Net-(U27-Pad1)
- U29 pad 4: C3 -> B5
- U29 pad 5: C4 -> bsel
- U29 pad 6: C5 -> Net-(U27-Pad4)
- U29 pad 7: C6 -> GND
- U29 pad 8: C7 -> Net-(U27-Pad9)
- U29 pad 9: unconnected-(U29-A7-Pad9) -> B6
- U30 pad 1: unconnected-(U30-NC-Pad1) -> OUT5
- U30 pad 2: CIN-SEL -> /alu-4b-1/sB1
- U30 pad 3: GND -> /alu-4b-1/log1
- U30 pad 4: Net-(U29-G1) -> OUT4
- U30 pad 5: VCC -> /alu-4b-1/log0
- U31 pad 10: /alu-8b-1/alu-1b-1/beff -> B4
- U31 pad 11: /alu-8b-1/alu-1b-1/aeff -> A4
- U31 pad 5: OUT9 -> /alu-4b-1/log0
- U31 pad 9: Ceff9 -> C4
- U32 pad 1: ainv -> ALU-OPCODE3
- U32 pad 10: /alu-8b-1/alu-1b-1/beff -> B6
- U32 pad 11: unconnected-(U32-Pad11) -> A6
- U32 pad 12: unconnected-(U32-Pad12) -> ALU-OPCODE7
- U32 pad 13: unconnected-(U32-Pad13) -> ALU-OPCODE6
- U32 pad 14: VCC -> ALU-OPCODE5
- U32 pad 2: Net-(U32-Pad2) -> ALU-OPCODE2
- U32 pad 3: /alu-8b-1/alu-1b-1/aeff -> ALU-OPCODE1
- U32 pad 4: binv -> ALU-OPCODE0
- U32 pad 5: Net-(U32-Pad5) -> /alu-4b-1/log2
- U32 pad 6: /alu-8b-1/alu-1b-1/beff -> unconnected-(U32-~{Y}-Pad6)
- U32 pad 8: Net-(U32-Pad8) -> GND
- U32 pad 9: /alu-8b-1/alu-1b-1/aeff -> C6
- U34 pad 10: /alu-8b-1/alu-1b-0/beff -> B7
- U34 pad 11: /alu-8b-1/alu-1b-0/aeff -> A7
- U34 pad 5: OUT8 -> /alu-4b-1/log3
- U34 pad 9: Ceff8 -> C7
- U37 pad 1: ALU-OPCODE3 -> Net-(U37-Pad1)
- U37 pad 10: /alu-8b-1/alu-1b-7/beff -> binv
- U37 pad 11: /alu-8b-1/alu-1b-7/aeff -> /alu-4b-2/sB3
- U37 pad 12: ALU-OPCODE7 -> Net-(U37-Pad12)
- U37 pad 13: ALU-OPCODE6 -> binv
- U37 pad 14: ALU-OPCODE5 -> VCC
- U37 pad 2: ALU-OPCODE2 -> binv
- U37 pad 3: ALU-OPCODE1 -> /alu-4b-2/sB0
- U37 pad 4: ALU-OPCODE0 -> Net-(U37-Pad4)
- U37 pad 5: OUT15 -> binv
- U37 pad 6: unconnected-(U37-~{Y}-Pad6) -> /alu-4b-2/sB1
- U37 pad 8: GND -> /alu-4b-2/sB2
- U37 pad 9: Ceff15 -> Net-(U37-Pad9)
- U40 pad 1: ALU-OPCODE3 -> OUT9
- U40 pad 10: /alu-8b-1/alu-1b-6/beff -> OUT11
- U40 pad 11: /alu-8b-1/alu-1b-6/aeff -> /alu-4b-2/sB3
- U40 pad 12: ALU-OPCODE7 -> /alu-4b-2/log3
- U40 pad 13: ALU-OPCODE6 -> OUT10
- U40 pad 14: ALU-OPCODE5 -> /alu-4b-2/log2
- U40 pad 15: ALU-OPCODE4 -> /alu-4b-2/sB2
- U40 pad 2: ALU-OPCODE2 -> /alu-4b-2/sB1
- U40 pad 3: ALU-OPCODE1 -> /alu-4b-2/log1
- U40 pad 4: ALU-OPCODE0 -> OUT8
- U40 pad 5: OUT14 -> /alu-4b-2/log0
- U40 pad 6: unconnected-(U40-~{Y}-Pad6) -> /alu-4b-2/sB0
- U40 pad 7: GND -> /cout1
- U40 pad 9: Ceff14 -> /cout2
- U41 pad 1: ainv -> ALU-OPCODE3
- U41 pad 10: /alu-8b-1/alu-1b-6/beff -> B8
- U41 pad 11: unconnected-(U41-Pad11) -> A8
- U41 pad 12: unconnected-(U41-Pad12) -> ALU-OPCODE7
- U41 pad 13: unconnected-(U41-Pad13) -> ALU-OPCODE6
- U41 pad 14: VCC -> ALU-OPCODE5
- U41 pad 2: Net-(U41-Pad2) -> ALU-OPCODE2
- U41 pad 3: /alu-8b-1/alu-1b-6/aeff -> ALU-OPCODE1
- U41 pad 4: binv -> ALU-OPCODE0
- U41 pad 5: Net-(U41-Pad5) -> /alu-4b-2/log0
- U41 pad 6: /alu-8b-1/alu-1b-6/beff -> unconnected-(U41-~{Y}-Pad6)
- U41 pad 8: Net-(U41-Pad8) -> GND
- U41 pad 9: /alu-8b-1/alu-1b-6/aeff -> C8
- U43 pad 10: /alu-8b-1/alu-1b-5/beff -> B9
- U43 pad 11: /alu-8b-1/alu-1b-5/aeff -> A9
- U43 pad 5: OUT13 -> /alu-4b-2/log1
- U43 pad 9: Ceff13 -> C9
- U44 pad 1: ainv -> ALU-OPCODE3
- U44 pad 10: /alu-8b-1/alu-1b-5/beff -> B11
- U44 pad 11: unconnected-(U44-Pad11) -> A11
- U44 pad 12: unconnected-(U44-Pad12) -> ALU-OPCODE7
- U44 pad 13: unconnected-(U44-Pad13) -> ALU-OPCODE6
- U44 pad 14: VCC -> ALU-OPCODE5
- U44 pad 2: Net-(U44-Pad2) -> ALU-OPCODE2
- U44 pad 3: /alu-8b-1/alu-1b-5/aeff -> ALU-OPCODE1
- U44 pad 4: binv -> ALU-OPCODE0
- U44 pad 5: Net-(U44-Pad5) -> /alu-4b-2/log3
- U44 pad 6: /alu-8b-1/alu-1b-5/beff -> unconnected-(U44-~{Y}-Pad6)
- U44 pad 8: Net-(U44-Pad8) -> GND
- U44 pad 9: /alu-8b-1/alu-1b-5/aeff -> C11
- U47 pad 1: ainv -> Net-(U47-Pad1)
- U47 pad 10: /alu-8b-1/alu-1b-2/beff -> binv
- U47 pad 11: unconnected-(U47-Pad11) -> /alu-4b-3/sB3
- U47 pad 12: unconnected-(U47-Pad12) -> Net-(U47-Pad12)
- U47 pad 13: unconnected-(U47-Pad13) -> binv
- U47 pad 2: Net-(U47-Pad2) -> binv
- U47 pad 3: /alu-8b-1/alu-1b-2/aeff -> /alu-4b-3/sB0
- U47 pad 4: binv -> Net-(U47-Pad4)
- U47 pad 5: Net-(U47-Pad5) -> binv
- U47 pad 6: /alu-8b-1/alu-1b-2/beff -> /alu-4b-3/sB1
- U47 pad 8: Net-(U47-Pad8) -> /alu-4b-3/sB2
- U47 pad 9: /alu-8b-1/alu-1b-2/aeff -> Net-(U47-Pad9)
- U49 pad 1: ALU-OPCODE3 -> B12
- U49 pad 10: /alu-8b-1/alu-1b-4/beff -> bsel
- U49 pad 11: /alu-8b-1/alu-1b-4/aeff -> Net-(U47-Pad12)
- U49 pad 12: ALU-OPCODE7 -> B15
- U49 pad 13: ALU-OPCODE6 -> bsel
- U49 pad 14: ALU-OPCODE5 -> VCC
- U49 pad 2: ALU-OPCODE2 -> bsel
- U49 pad 3: ALU-OPCODE1 -> Net-(U47-Pad1)
- U49 pad 4: ALU-OPCODE0 -> B13
- U49 pad 5: OUT12 -> bsel
- U49 pad 6: unconnected-(U49-~{Y}-Pad6) -> Net-(U47-Pad4)
- U49 pad 8: GND -> Net-(U47-Pad9)
- U49 pad 9: Ceff12 -> B14
- U50 pad 1: ainv -> OUT13
- U50 pad 10: /alu-8b-1/alu-1b-4/beff -> OUT15
- U50 pad 11: unconnected-(U50-Pad11) -> /alu-4b-3/sB3
- U50 pad 12: unconnected-(U50-Pad12) -> /alu-4b-3/log3
- U50 pad 13: unconnected-(U50-Pad13) -> OUT14
- U50 pad 14: VCC -> /alu-4b-3/log2
- U50 pad 2: Net-(U103-Pad3) -> /alu-4b-3/sB1
- U50 pad 3: /alu-8b-1/alu-1b-4/aeff -> /alu-4b-3/log1
- U50 pad 4: binv -> OUT12
- U50 pad 5: Net-(U103-Pad6) -> /alu-4b-3/log0
- U50 pad 6: /alu-8b-1/alu-1b-4/beff -> /alu-4b-3/sB0
- U50 pad 7: GND -> /cout2
- U50 pad 8: Net-(U103-Pad12) -> GND
- U50 pad 9: /alu-8b-1/alu-1b-4/aeff -> /cout3
- U52 pad 10: /alu-8b-1/alu-1b-3/beff -> B14
- U52 pad 11: /alu-8b-1/alu-1b-3/aeff -> A14
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
Commit message: feat: placed data buses; naming to match proposed design layout
Parts:
- moved D13 188.5 mm to (489.7, 89.8)
- moved D14 188.5 mm to (489.7, 92.9)
- moved J5 188.5 mm to (480.0, 205.0)
- moved R13 188.5 mm to (493.9, 89.5)
- moved R14 188.5 mm to (493.9, 92.1)
- moved J3 188.5 mm to (482.6, 84.2)
- moved SW7 188.5 mm to (491.4, 85.4)
- moved C126 179.6 mm to (264.8, 263.4), turned to 180 degrees
- moved RN10 173.3 mm to (120.6, 32.1), turned to 0 degrees
- moved U94 171.6 mm to (259.5, 257.8), turned to -90 degrees
- moved RN11 166.6 mm to (120.6, 43.5), turned to 0 degrees
- moved C124 163.1 mm to (253.1, 263.4), turned to 180 degrees
- moved U87 161.9 mm to (252.9, 249.1), turned to 90 degrees
- moved C70 161.6 mm to (152.3, 116.8), turned to 0 degrees
- moved SW1 161.4 mm to (264.9, 21.0), turned to -90 degrees
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Routing:
- net (no net): track 0.00 -> 6864.0 mm
- net C2: track 0.00 -> 416.0 mm
- net C1: track 0.00 -> 416.0 mm
- net C0: track 0.00 -> 416.0 mm
- net B3: track 0.00 -> 416.0 mm
- net B2: track 0.00 -> 416.0 mm
- net B1: track 0.00 -> 416.0 mm
- net B0: track 0.00 -> 416.0 mm
- net A3: track 0.00 -> 416.0 mm
- net A2: track 0.00 -> 416.0 mm
- net A1: track 0.00 -> 416.0 mm
- net A0: track 0.00 -> 416.0 mm
- net C18: track 0.00 -> 208.0 mm
- net C17: track 0.00 -> 208.0 mm
- net C16: track 0.00 -> 208.0 mm
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
Commit message: feat: routed data buses
Parts:
- moved D13 97.6 mm to (392.2, 94.8)
- moved D14 97.6 mm to (392.2, 97.9)
- moved J3 97.6 mm to (385.1, 89.2)
- moved J5 97.6 mm to (382.5, 210.0)
- moved R13 97.6 mm to (396.4, 94.6)
- moved R14 97.6 mm to (396.4, 97.1)
- moved SW7 97.6 mm to (393.9, 90.4)
- moved U74 20.1 mm to (239.0, 172.6)
- moved U84 20.1 mm to (239.0, 214.9)
- moved C100 20.1 mm to (227.6, 200.7)
- moved C102 20.1 mm to (216.1, 200.7)
- moved C104 20.1 mm to (205.4, 200.7)
- moved C106 20.1 mm to (209.6, 220.4)
- moved C108 20.1 mm to (221.1, 220.4)
- moved C110 20.1 mm to (232.6, 220.4)
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Routing:
- net A0: track 416.0 -> 0.00 mm
- net B0: track 416.0 -> 162.0 mm
- net C0: track 416.0 -> 163.0 mm
- net A1: track 416.0 -> 164.0 mm
- net B1: track 416.0 -> 165.0 mm
- net C1: track 416.0 -> 166.0 mm
- net A2: track 416.0 -> 167.0 mm
- net B2: track 416.0 -> 168.0 mm
- net C2: track 416.0 -> 169.0 mm
- net A3: track 416.0 -> 170.0 mm
- net B3: track 416.0 -> 171.0 mm
- net B19: track 0.00 -> 212.1 mm
- net A19: track 0.00 -> 211.7 mm
- net OUT1: track 0.00 -> 208.2 mm
- net OUT0: track 0.00 -> 208.0 mm
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