File: hardware/kicad/boards/01_alu/alu-32b.kicad_pcb (KiCad board)
At the start: 4 copper layers, 240 x 240 mm, 146 parts, among them J1 Conn_02x16_Odd_Even, J2 Conn_02x16_Odd_Even, J3 Conn_02x04_Odd_Even, J4 Conn_02x16_Odd_Even, J5 Conn_02x16_Counter_Clockwise, SW1 SW_DIP_x08, SW10 SW_DIP_x08, SW11 SW_DIP_x08, SW12 SW_DIP_x08, SW13 SW_DIP_x08, SW2 SW_DIP_x08, SW3 SW_DIP_x08, SW4 SW_DIP_x08, SW5 SW_DIP_x08, SW6 SW_DIP_x08, SW7 SW_SPDT, SW8 SW_DIP_x08, SW9 SW_DIP_x08, U1 74ACT151, U10 74ACT151, U11 74ACT151, U12 74ACT151, U13 74ACT151, U14 74ACT151, U15 74ACT151, U16 74ACT151, U17 74HC86, U18 74ACT151, U19 74HC00, U2 74ACT151, U20 74ACT283, U21 74ACT151, U22 74ACT151, U23 74ACT151, U24 74ACT151, U25 74ACT151, U26 74ACT151, U27 74HC86, U28 74ACT151, U29 74HC00, U3 74ACT151, U30 74ACT283, U31 74ACT151, U32 74ACT151, U33 74ACT151, U34 74ACT151, U35 74ACT151, U36 74ACT151, U37 74HC86, U38 74ACT151, U39 74HC00, U4 74ACT151, U40 74ACT283, U41 74ACT151, U47 74HC86, U49 74HC00, U5 74ACT151, U50 74ACT283, U57 74HC86, U59 74HC00, U6 74ACT151, U60 74ACT283, U67 74HC86, U69 74HC00, U7 74ACT151, U70 74ACT283, U77 74HC86, U79 74HC00, U8 74ACT151, U80 74ACT283, U87 74HC86, U89 74HC00, U9 74ACT151, U90 74ACT283

Commit message: feat: added 8to1 mux for cin variety; routed major bus on RHS cells; updated main.dig with cin mux
Updated alu-control with correct global labels for cin-sel[2..0]
Parts:
- added C25: 100nF, Capacitor_SMD:C_0603_1608Metric, F.Cu at (139.7, 133.6)
- added U42: 74ACT151, Package_SO:SOIC-16_3.9x9.9mm_P1.27mm, F.Cu at (133.5, 138.2)
- moved J1 433.8 mm to (268.1, 470.9)
- moved J2 433.8 mm to (217.7, 470.6)
- moved RN10 433.8 mm to (124.7, 465.9)
- moved RN3 433.8 mm to (225.8, 466.4)
- moved RN4 433.8 mm to (270.9, 466.4)
- moved RN5 433.8 mm to (220.5, 466.1)
- moved RN6 433.8 mm to (175.4, 466.1)
- moved RN7 433.8 mm to (175.4, 477.5)
- moved RN9 433.8 mm to (169.9, 465.9)
- moved SW1 433.8 mm to (269.1, 454.7)
- moved SW2 433.8 mm to (218.7, 454.5)
- moved SW8 433.8 mm to (244.8, 454.7)
- moved SW9 433.8 mm to (194.5, 454.5)
- moved J4 433.8 mm to (167.1, 470.3)
- moved RN1 433.8 mm to (270.9, 477.8)
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Routing:
- net ALU-OPCODE7: track 431.3 -> 653.0 mm, vias 37 -> 40
- net ALU-OPCODE6: track 435.4 -> 649.1 mm, vias 37 -> 40
- net ALU-OPCODE5: track 402.9 -> 611.3 mm, vias 37 -> 40
- net bsel: track 295.4 -> 503.0 mm, vias 19 -> 20
- net ALU-OPCODE0: track 465.2 -> 672.1 mm, vias 37 -> 40
- net ALU-OPCODE4: track 370.9 -> 571.7 mm, vias 37 -> 40
- net ALU-OPCODE1: track 432.4 -> 631.9 mm, vias 37 -> 40
- net binv: track 508.7 -> 702.3 mm
- net ALU-OPCODE2: track 403.9 -> 595.8 mm, vias 37 -> 40
- net ALU-OPCODE3: track 372.1 -> 559.8 mm, vias 39 -> 44
- net OUT18: track 23.2 -> 136.9 mm
- net OUT19: track 18.2 -> 131.5 mm
- net OUT17: track 25.7 -> 135.1 mm, vias 2 -> 1
- net OUT16: track 23.4 -> 132.5 mm, vias 2 -> 1
- net OUT22: track 11.4 -> 105.2 mm, vias 1 -> 2
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
Commit message: feat: laid the main bus; adding control unit and display segments
Parts:
- moved RN4 180.2 mm to (91.1, 478.3), turned to 0 degrees
- moved RN1 180.1 mm to (91.1, 466.9), turned to 0 degrees
- moved SW1 179.6 mm to (93.0, 489.9), turned to 90 degrees
- moved J1 174.2 mm to (93.9, 473.8), turned to 90 degrees
- moved SW11 144.8 mm to (110.7, 455.0), turned to -90 degrees
- moved RN10 140.7 mm to (264.1, 484.9), turned to 180 degrees
- moved SW6 139.6 mm to (262.9, 461.7), turned to -90 degrees
- moved RN11 139.5 mm to (264.1, 473.5), turned to 180 degrees
- moved SW8 132.4 mm to (117.2, 489.9), turned to 90 degrees
- moved SW10 109.8 mm to (245.1, 496.6), turned to 90 degrees
- moved SW4 98.4 mm to (135.0, 455.0), turned to -90 degrees
- moved SW13 92.5 mm to (238.6, 461.7), turned to -90 degrees
- moved RN3 90.3 mm to (136.3, 478.3), turned to 180 degrees
- moved RN2 90.2 mm to (136.3, 466.9), turned to 180 degrees
- moved SW2 68.7 mm to (160.8, 491.4), turned to 90 degrees
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Routing:
- net C0: track 54.3 -> 186.0 mm
- net B0: track 127.1 -> 258.0 mm
- net A0: track 50.5 -> 180.6 mm
- net A31: track 43.0 -> 172.9 mm
- net C1: track 41.4 -> 170.7 mm
- net B31: track 63.1 -> 192.3 mm
- net B1: track 103.8 -> 232.2 mm
- net C31: track 39.9 -> 168.2 mm
- net A1: track 38.5 -> 166.1 mm
- net A30: track 30.8 -> 158.3 mm
- net C2: track 29.6 -> 156.4 mm
- net B30: track 48.5 -> 175.1 mm
- net B2: track 55.7 -> 181.7 mm
- net C30: track 27.5 -> 153.1 mm
- net A2: track 26.1 -> 151.2 mm
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
Commit message: fix: resolved kicad erc tests to 0
Parts:
- removed D13, D14: LED, LED_SMD:LED_0805_2012Metric
- removed J1, J2, J4: Conn_02x16_Odd_Even, Connector_PinHeader_2.54mm:PinHeader_2x16_P2.54mm_Vertical
- removed J3: Conn_02x04_Odd_Even, Connector_PinHeader_2.54mm:PinHeader_2x04_P2.54mm_Vertical
- removed R13: 330, Resistor_SMD:R_0603_1608Metric
- removed R14: 500, Resistor_SMD:R_0603_1608Metric
- removed RN1, RN10, RN11, RN12, RN2, RN3, RN4, RN5, RN6, RN7, RN8, RN9: R_Network08, Resistor_THT:R_Array_SIP9
- removed SW1, SW10, SW11, SW12, SW13, SW2, SW3, SW4, SW5, SW6, SW8, SW9: SW_DIP_x08, Button_Switch_THT:SW_DIP_SPSTx08_Slide_9.78x22.5mm_W7.62mm_P2.54mm
- removed SW7: SW_SPDT, Button_Switch_THT:SW_Slide_SPDT_Straight_CK_OS102011MS2Q
- moved J5 32.1 mm to (179.2, 163.1)
