File: hardware/kicad/boards/01_alu/alu-display.kicad_sch (KiCad schematic)
At the start: 16 parts, among them U173 74LS154, U174 74LS163, U175 74AHC1G04, U176 74LS163, U177 74LS154, U178 KM28C64A, U179 74LS153, U180 74LS153

Commit message: chore: refactored display logic and cleanup alu design
Parts:
- removed C173, C174, C175, C176, C177, C178, C179, C180: 100nF, Capacitor_SMD:C_0805_2012Metric, symbol Device:C
- removed U173, U177: 74LS154, Package_SO:SOIC-24W_7.5x15.4mm_P1.27mm, symbol 74xx:74LS154
- removed U174, U176: 74LS163, Package_SO:SOIC-16_3.9x9.9mm_P1.27mm, symbol 74xx:74LS163
- removed U175: 74AHC1G04, Package_TO_SOT_SMD:SOT-23-5, symbol 74xGxx:74AHC1G04
- removed U178: KM28C64A, Package_DIP:DIP-28_W15.24mm, symbol Memory_EEPROM:KM28C64A
- removed U179, U180: 74LS153, Package_SO:SOIC-16_3.9x9.9mm_P1.27mm, symbol 74xx:74LS153
Connections:
- no-connect marks 68 -> 0
Other:
- removed sheet display-clock
- removed sheet mux4_4to1
- removed sheet mux4_8to1-4
- removed sheet mux4_8to1-5
- removed sheet mux4_8to1-6
- removed sheet mux4_8to1-7
- removed sheet seg-disp32
- added sheet seg-disp13 (1-seg-display.kicad_sch)
- added sheet seg-disp14 (1-seg-display.kicad_sch)
- added sheet seg-disp15 (1-seg-display.kicad_sch)
- added sheet seg-disp16 (1-seg-display.kicad_sch)
- added sheet seg-disp2 (1-seg-display.kicad_sch)
- added sheet seg-disp21 (1-seg-display.kicad_sch)
- added sheet seg-disp22 (1-seg-display.kicad_sch)
- added sheet seg-disp23 (1-seg-display.kicad_sch)
- added sheet seg-disp24 (1-seg-display.kicad_sch)
- added sheet seg-disp5 (1-seg-display.kicad_sch)
- added sheet seg-disp6 (1-seg-display.kicad_sch)
- added sheet seg-disp7 (1-seg-display.kicad_sch)
- added sheet seg-disp8 (1-seg-display.kicad_sch)
- sheet seg-disp0 ports: added d0, d1, d2, d3; removed en
- sheet seg-disp1 ports: added d0, d1, d2, d3; removed en
- sheet seg-disp10 ports: added d0, d1, d2, d3; removed en
- sheet seg-disp11 ports: added d0, d1, d2, d3; removed en
- sheet seg-disp12 ports: added d0, d1, d2, d3; removed en
- sheet seg-disp17 ports: added d0, d1, d2, d3; removed en
- sheet seg-disp18 ports: added d0, d1, d2, d3; removed en
- sheet seg-disp19 ports: added d0, d1, d2, d3; removed en
- sheet seg-disp20 ports: added d0, d1, d2, d3; removed en
- sheet seg-disp25 ports: added d0, d1, d2, d3; removed en
- sheet seg-disp26 ports: added d0, d1, d2, d3; removed en
- sheet seg-disp27 ports: added d0, d1, d2, d3; removed en
- sheet seg-disp28 ports: added d0, d1, d2, d3; removed en
- sheet seg-disp29 ports: added d0, d1, d2, d3; removed en
- sheet seg-disp3 ports: added d0, d1, d2, d3; removed en
- sheet seg-disp30 ports: added d0, d1, d2, d3; removed en
- sheet seg-disp31 ports: added d0, d1, d2, d3; removed en
- sheet seg-disp4 ports: added d0, d1, d2, d3; removed en
- sheet seg-disp9 ports: added d0, d1, d2, d3; removed en
