File: hardware/kicad/boards/01_alu/alu-control.kicad_sch (KiCad schematic)
At the start: 17 parts, among them J7 Conn_02x01, J8 Conn_02x05_Odd_Even, SW14 SW_DIP_x08, SW15 SW_DIP_x08, SW16 SW_Slide_DPDT, U155 KM28C64A, U156 KM28C64A, U157 74AHC541, U158 74AHC541, U159 74AHC541, U160 74AHC541

Commit message: chore: refactored display logic and cleanup alu design
Parts:
- C155: renamed from C158; footprint Capacitor_SMD:C_0805_2012Metric -> Capacitor_SMD:C_0603_1608Metric
- C156: renamed from C155; footprint Capacitor_SMD:C_0805_2012Metric -> Capacitor_SMD:C_0603_1608Metric
- C157: renamed from C159; footprint Capacitor_SMD:C_0805_2012Metric -> Capacitor_SMD:C_0603_1608Metric
- C158: renamed from C160; footprint Capacitor_SMD:C_0805_2012Metric -> Capacitor_SMD:C_0603_1608Metric
- C159: renamed from C157; footprint Capacitor_SMD:C_0805_2012Metric -> Capacitor_SMD:C_0603_1608Metric
- C160: renamed from C156; footprint Capacitor_SMD:C_0805_2012Metric -> Capacitor_SMD:C_0603_1608Metric
- renumbered J8 to J7, J7 to J8, SW16 to SW14, SW14 to SW15, SW15 to SW16, U157 to U155, U155 to U156, U159 to U157, U160 to U158, U158 to U159, U156 to U160

Commit message: feat: updated the kicad schematics with updated correct control fanouts
Parts:
- renumbered C155 to C127, C156 to C128, C157 to C129, C158 to C130, C159 to C131, C160 to C132, U160 to U100, U155 to U95, U156 to U96, U157 to U97, U158 to U98, U159 to U99
Connections:
- net csel0 renamed cin-main
- net csel1 renamed alu-mode

Commit message: chore: modularized the alu into hsheets including flag logic
Parts:
- removed SW16: SW_DIP_x08, Button_Switch_THT:SW_DIP_SPSTx08_Slide_9.78x22.5mm_W7.62mm_P2.54mm, symbol Switch:SW_DIP_x08
- added RN1: R_Network04, Resistor_THT:R_Array_SIP5, symbol Device:R_Network04
- added SW1: SW_DIP_x04, symbol Switch:SW_DIP_x04
Connections:
- net ainv is gone; now on net binv: U99.17 (Y1)
- net asel is gone; now on net bsel: U99.18 (Y0)
- net GND: now also RN1.1 (common)
- net binv: now also RN1.4 (R3), SW1.7; no longer U99.15 (Y3)
- net bsel: now also RN1.5 (R4), SW1.8; no longer U99.16 (Y2)
- net cin-main: now also U99.16 (Y2), RN1.3 (R2), SW1.6; no longer U99.14 (Y4)
- net flagWE: now also U99.15 (Y3), RN1.2 (R1), SW1.5; no longer U99.12 (Y6)
- net alu-mode: no longer names the net of U99.13 (Y5)
- no-connect marks 3 -> 5
