File: hardware/kicad/boards/01_alu/alu-control.kicad_sch (KiCad schematic)
At the start: 18 parts, among them J7 Conn_02x05_Odd_Even, J8 Conn_02x01, SW1 SW_DIP_x04, SW14 SW_Slide_DPDT, SW15 SW_DIP_x08, U100 KM28C64A, U95 74AHC541, U96 KM28C64A, U97 74AHC541, U98 74AHC541, U99 74AHC541

Commit message: feat: added 8to1 mux for cin variety; routed major bus on RHS cells; updated main.dig with cin mux
Updated alu-control with correct global labels for cin-sel[2..0]
Connections:
- net cin-main: no longer U99.16 (Y2)
- net flagWE: now also U99.13 (Y5); no longer U99.15 (Y3)
- net CSEL2: now reaches U99.14 (Y4)
- new net CSEL0: U99.16 (Y2)
- new net CSEL1: U99.15 (Y3)
- no-connect marks 5 -> 3

Commit message: feat: laid the main bus; adding control unit and display segments
Parts:
- renumbered C127 to C1, C128 to C2, C129 to C3, C130 to C4, C131 to C5, C132 to C6, J7 to J6, J8 to J7, RN1 to RN13, SW1 to SW16, U95 to U43, U96 to U44, U97 to U45, U98 to U46, U99 to U48, U100 to U51

Commit message: feat(web): story gallery and live datapath; wire 01_alu display sheet (#27)
* chore(web): add the in-place media optimizer

* media(web): recompress plates, pcb, and gallery WebPs

* media(web): add story gallery stills and responsive WebPs

* test(web): cover story gallery LCP preload

* feat(web): retell the gallery from notebook to 07_alu

* feat(web): embed the Dual-LUT strip on the front page

* feat(web): expand playground with overview, pipe, map, and sliders

* feat(web): let mast burger attach to scroll-rail

* media: compress microcode control log still

* feat(hardware): wire display sheet into 01_alu 32-bit project

* feat(hardware): add display sheet stub for 01_alu
Parts:
- removed C1, C2, C6: 100nF, Capacitor_SMD:C_0603_1608Metric, symbol Device:C
- removed C3, C4, C5: C, Capacitor_SMD:C_0603_1608Metric, symbol Device:C
- removed J6: Conn_02x05_Odd_Even, Connector_PinHeader_2.54mm:PinHeader_2x05_P2.54mm_Vertical, symbol Connector_Generic:Conn_02x05_Odd_Even
- removed J7: Conn_02x01, Connector_PinHeader_2.54mm:PinHeader_2x01_P2.54mm_Horizontal, symbol Connector_Generic:Conn_02x01
- removed RN13: R_Network04, Resistor_THT:R_Array_SIP5, symbol Device:R_Network04
- removed SW14: SW_Slide_DPDT, Button_Switch_SMD:SW_DPDT_CK_JS202011JCQN, symbol Switch:SW_Slide_DPDT
- removed SW15: SW_DIP_x08, Button_Switch_THT:SW_DIP_SPSTx08_Slide_9.78x22.5mm_W7.62mm_P2.54mm, symbol Switch:SW_DIP_x08
- removed SW16: SW_DIP_x04, symbol Switch:SW_DIP_x04
- removed U43, U45, U46, U48: 74AHC541, Package_SO:SOIC-20W_7.5x12.8mm_P1.27mm, symbol 74xx:74AHC541
- removed U44, U51: KM28C64A, Package_DIP:DIP-28_W15.24mm, symbol Memory_EEPROM:KM28C64A
Connections:
- no-connect marks 3 -> 0
