File: hardware/kicad/boards/01_alu/alu-4b.kicad_sch (KiCad schematic)
At the start: 12 parts, among them U15 74LS257, U16 74HC86, U17 74HC86, U18 74HC00, U19 74HC00, U20 74LS283

Commit message: checkpoint: placed components for optimized routing on alu-32b board pcb
Parts:
- removed C15, C17, C19: 100nF, Capacitor_SMD:C_0603_1608Metric, symbol Device:C
- removed U15: 74LS257, Package_SO:SOIC-16_3.9x9.9mm_P1.27mm, symbol 74xx:74LS257
- removed U16: 74HC86, Package_SO:SOIC-14_3.9x8.7mm_P1.27mm, symbol 74xx:74HC86
- removed U18: 74HC00, Package_SO:SOIC-14_3.9x8.7mm_P1.27mm, symbol 74xx:74HC00
Connections:
- net s0 is gone; now on net out-4b0: U20.4 (S1)
- net s1 is gone; now on net out-4b1: U20.1 (S2)
- net s2 is gone; now on net out-4b2: U20.13 (S3)
- net sA0 is gone; now on net log0: U20.5 (A1)
- net sA1 is gone; now on net log1: U20.3 (A2)
- net sA2 is gone; now on net log2: U20.14 (A3)
Other:
- moved on the sheet: C16, U20
