File: hardware/kicad/boards/01_alu/alu-4b.kicad_sch (KiCad schematic)
At the start: 6 parts, among them U17 74HC86, U19 74HC00, U20 74LS283

Commit message: arch(alu): replace 251 tri-state MUX with 151 to prevent High-Z faults
Eliminates dead Tri-State functionality on point-to-point traces, preventing potential logic oscillation and chip damage from floating pins. Drive strength and speed are unaffected.

Closes #4
Parts:
- U20: value 74LS283 -> 74ACT283
Changed lines of the file:
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@@
 			)
 		)
-		(property "Value" "74LS283"
+		(property "Value" "74ACT283"
 			(at 122.7933 41.91 0)
 			(show_name no)
