File: hardware/kicad/boards/06_data_bus/wb_mux.kicad_sch (KiCad schematic)
At the start: 0 parts

Commit message: kicad: checkpoint; designed the alu display logic; clock circuit
Added registers for each display to ensure robustness and less worry about debugging screen, keeping focus on the alu board and other components
Other:
- added sheet drive32_0 (../../modules/mux/drivers-74xx/driver32.kicad_sch)
- added sheet drive32_1 (../../modules/mux/drivers-74xx/driver32.kicad_sch)
- added sheet drive32_2 (../../modules/mux/drivers-74xx/driver32.kicad_sch)
- added sheet drive32_5 (../../modules/mux/drivers-74xx/driver32.kicad_sch)
- added sheet drive32_6 (../../modules/mux/drivers-74xx/driver32.kicad_sch)
- added sheet drive32_7 (../../modules/mux/drivers-74xx/driver32.kicad_sch)
