File: hardware/kicad/modules/mux/mux-74xx/mux_2to1-8b.kicad_sch (KiCad schematic)
At the start: 4 parts, among them U1 74LS157, U2 74LS157

Commit message: schematics: designed mux32_2to1
Parts:
- renumbered C1 to C7, C2 to C8, U1 to U7, U2 to U8

Commit message: module: designed muxes prioritizing drivers for large switching preserving depth of ~1 gate
Parts:
- C1: renamed from C7; footprint (none) -> Capacitor_SMD:C_0201_0603Metric
- C2: renamed from C8; footprint (none) -> Capacitor_SMD:C_0201_0603Metric
- U1: renamed from U7; footprint (none) -> Package_SO:SOIC-16_3.9x9.9mm_P1.27mm
- U2: renamed from U8; footprint (none) -> Package_SO:SOIC-16_3.9x9.9mm_P1.27mm
Changed lines of the file:
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@@
 		(dnp no)
 		(fields_autoplaced yes)
-		(property "Reference" "#PWR020"
+		(property "Reference" "#PWR02"
 			(at 95.25 96.52 0)
 			(hide yes)
@@
 				)
 				(path "/9770a3ff-dcb3-40dd-904f-3792f096cc81/461fdf99-31de-4f28-b803-0ca226183c1b/4bfad7ce-72f4-4d4b-b445-f07a93594dc1"
-					(reference "#PWR020")
+					(reference "#PWR02")
 					(unit 1)
 				)
 				(path "/9770a3ff-dcb3-40dd-904f-3792f096cc81/461fdf99-31de-4f28-b803-0ca226183c1b/9c0f8848-c55e-49fd-9cbe-bfda325c51c8"
-					(reference "#PWR020")
+					(reference "#PWR08")
 					(unit 1)
 				)
 				(path "/9770a3ff-dcb3-40dd-904f-3792f096cc81/461fdf99-31de-4f28-b803-0ca226183c1b/ad6ef6e9-1754-4226-a802-1e45b0c5c28a"
-					(reference "#PWR020")
+					(reference "#PWR014")
 					(unit 1)
 				)
@@
 		(dnp no)
 		(fields_autoplaced yes)
-		(property "Reference" "C8"
+		(property "Reference" "C2"
 			(at 102.87 101.6 90)
 			(show_name no)
@@
 			)
 		)
-		(property "Footprint" ""
+		(property "Footprint" "Capacitor_SMD:C_0201_0603Metric"
 			(at 106.68 108.2548 0)
 			(hide yes)
@@
 				)
 				(path "/9770a3ff-dcb3-40dd-904f-3792f096cc81/461fdf99-31de-4f28-b803-0ca226183c1b/4bfad7ce-72f4-4d4b-b445-f07a93594dc1"
-					(reference "C8")
+					(reference "C2")
 					(unit 1)
 				)
 				(path "/9770a3ff-dcb3-40dd-904f-3792f096cc81/461fdf99-31de-4f28-b803-0ca226183c1b/9c0f8848-c55e-49fd-9cbe-bfda325c51c8"
-					(reference "C8")
+					(reference "C4")
 					(unit 1)
 				)
 				(path "/9770a3ff-dcb3-40dd-904f-3792f096cc81/461fdf99-31de-4f28-b803-0ca226183c1b/ad6ef6e9-1754-4226-a802-1e45b0c5c28a"
-					(reference "C8")
+					(reference "C6")
 					(unit 1)
 				)
@@
 		(dnp no)
 		(fields_autoplaced yes)
-		(property "Reference" "#PWR019"
+		(property "Reference" "#PWR01"
 			(at 95.25 41.91 0)
 			(hide yes)
@@
 				)
 				(path "/9770a3ff-dcb3-40dd-904f-3792f096cc81/461fdf99-31de-4f28-b803-0ca226183c1b/4bfad7ce-72f4-4d4b-b445-f07a93594dc1"
-					(reference "#PWR019")
+					(reference "#PWR01")
 					(unit 1)
 				)
 				(path "/9770a3ff-dcb3-40dd-904f-3792f096cc81/461fdf99-31de-4f28-b803-0ca226183c1b/9c0f8848-c55e-49fd-9cbe-bfda325c51c8"
-					(reference "#PWR019")
+					(reference "#PWR07")
 					(unit 1)
 				)
 				(path "/9770a3ff-dcb3-40dd-904f-3792f096cc81/461fdf99-31de-4f28-b803-0ca226183c1b/ad6ef6e9-1754-4226-a802-1e45b0c5c28a"
-					(reference "#PWR019")
+					(reference "#PWR013")
 					(unit 1)
 				)
@@
 		(dnp no)
 		(fields_autoplaced yes)
-		(property "Reference" "#PWR024"
+		(property "Reference" "#PWR06"
 			(at 113.03 109.22 0)
 			(hide yes)
@@
 				)
 				(path "/9770a3ff-dcb3-40dd-904f-3792f096cc81/461fdf99-31de-4f28-b803-0ca226183c1b/4bfad7ce-72f4-4d4b-b445-f07a93594dc1"
-					(reference "#PWR024")
+					(reference "#PWR06")
 					(unit 1)
 				)
 				(path "/9770a3ff-dcb3-40dd-904f-3792f096cc81/461fdf99-31de-4f28-b803-0ca226183c1b/9c0f8848-c55e-49fd-9cbe-bfda325c51c8"
-					(reference "#PWR024")
+					(reference "#PWR012")
 					(unit 1)
 				)
 				(path "/9770a3ff-dcb3-40dd-904f-3792f096cc81/461fdf99-31de-4f28-b803-0ca226183c1b/ad6ef6e9-1754-4226-a802-1e45b0c5c28a"
-					(reference "#PWR024")
+					(reference "#PWR018")
 					(unit 1)
 				)
@@
 		(dnp no)
 		(fields_autoplaced yes)
-		(property "Reference" "#PWR022"
+		(property "Reference" "#PWR04"
 			(at 96.52 166.37 0)
 			(hide yes)
@@
 				)
 				(path "/9770a3ff-dcb3-40dd-904f-3792f096cc81/461fdf99-31de-4f28-b803-0ca226183c1b/4bfad7ce-72f4-4d4b-b445-f07a93594dc1"
-					(reference "#PWR022")
+					(reference "#PWR04")
 					(unit 1)
 				)
 				(path "/9770a3ff-dcb3-40dd-904f-3792f096cc81/461fdf99-31de-4f28-b803-0ca226183c1b/9c0f8848-c55e-49fd-9cbe-bfda325c51c8"
-					(reference "#PWR022")
+					(reference "#PWR010")
 					(unit 1)
 				)
 				(path "/9770a3ff-dcb3-40dd-904f-3792f096cc81/461fdf99-31de-4f28-b803-0ca226183c1b/ad6ef6e9-1754-4226-a802-1e45b0c5c28a"
-					(reference "#PWR022")
+					(reference "#PWR016")
 					(unit 1)
 				)
@@
 		(dnp no)
 		(fields_autoplaced yes)
-		(property "Reference" "#PWR021"
+		(property "Reference" "#PWR03"
 			(at 96.52 111.76 0)
 			(hide yes)
@@
 				)
 				(path "/9770a3ff-dcb3-40dd-904f-3792f096cc81/461fdf99-31de-4f28-b803-0ca226183c1b/4bfad7ce-72f4-4d4b-b445-f07a93594dc1"
-					(reference "#PWR021")
+					(reference "#PWR03")
 					(unit 1)
 				)
 				(path "/9770a3ff-dcb3-40dd-904f-3792f096cc81/461fdf99-31de-4f28-b803-0ca226183c1b/9c0f8848-c55e-49fd-9cbe-bfda325c51c8"
-					(reference "#PWR021")
+					(reference "#PWR09")
 					(unit 1)
 				)
 				(path "/9770a3ff-dcb3-40dd-904f-3792f096cc81/461fdf99-31de-4f28-b803-0ca226183c1b/ad6ef6e9-1754-4226-a802-1e45b0c5c28a"
-					(reference "#PWR021")
+					(reference "#PWR015")
 					(unit 1)
 				)
@@
 		(dnp no)
 		(fields_autoplaced yes)
-		(property "Reference" "U8"
+		(property "Reference" "U2"
 			(at 98.6633 111.76 0)
 			(show_name no)
@@
 			)
 		)
-		(property "Footprint" ""
+		(property "Footprint" "Package_SO:SOIC-16_3.9x9.9mm_P1.27mm"
 			(at 96.52 134.62 0)
 			(hide yes)
@@
 				)
 				(path "/9770a3ff-dcb3-40dd-904f-3792f096cc81/461fdf99-31de-4f28-b803-0ca226183c1b/4bfad7ce-72f4-4d4b-b445-f07a93594dc1"
-					(reference "U8")
+					(reference "U2")
 					(unit 1)
 				)
 				(path "/9770a3ff-dcb3-40dd-904f-3792f096cc81/461fdf99-31de-4f28-b803-0ca226183c1b/9c0f8848-c55e-49fd-9cbe-bfda325c51c8"
-					(reference "U8")
+					(reference "U4")
 					(unit 1)
 				)
 				(path "/9770a3ff-dcb3-40dd-904f-3792f096cc81/461fdf99-31de-4f28-b803-0ca226183c1b/ad6ef6e9-1754-4226-a802-1e45b0c5c28a"
-					(reference "U8")
+					(reference "U6")
 					(unit 1)
 				)
@@
 		(dnp no)
 		(fields_autoplaced yes)
-		(property "Reference" "C7"
+		(property "Reference" "C1"
 			(at 101.6 31.75 90)
 			(show_name no)
@@
 			)
 		)
-		(property "Footprint" ""
+		(property "Footprint" "Capacitor_SMD:C_0201_0603Metric"
 			(at 105.41 38.4048 0)
 			(hide yes)
@@
 				)
 				(path "/9770a3ff-dcb3-40dd-904f-3792f096cc81/461fdf99-31de-4f28-b803-0ca226183c1b/4bfad7ce-72f4-4d4b-b445-f07a93594dc1"
-					(reference "C7")
+					(reference "C1")
 					(unit 1)
 				)
 				(path "/9770a3ff-dcb3-40dd-904f-3792f096cc81/461fdf99-31de-4f28-b803-0ca226183c1b/9c0f8848-c55e-49fd-9cbe-bfda325c51c8"
-					(reference "C7")
+					(reference "C3")
 					(unit 1)
 				)
 				(path "/9770a3ff-dcb3-40dd-904f-3792f096cc81/461fdf99-31de-4f28-b803-0ca226183c1b/ad6ef6e9-1754-4226-a802-1e45b0c5c28a"
-					(reference "C7")
+					(reference "C5")
 					(unit 1)
 				)
@@
 		(dnp no)
 		(fields_autoplaced yes)
-		(property "Reference" "#PWR023"
+		(property "Reference" "#PWR05"
 			(at 111.76 39.37 0)
 			(hide yes)
@@
 				)
 				(path "/9770a3ff-dcb3-40dd-904f-3792f096cc81/461fdf99-31de-4f28-b803-0ca226183c1b/4bfad7ce-72f4-4d4b-b445-f07a93594dc1"
-					(reference "#PWR023")
+					(reference "#PWR05")
 					(unit 1)
 				)
 				(path "/9770a3ff-dcb3-40dd-904f-3792f096cc81/461fdf99-31de-4f28-b803-0ca226183c1b/9c0f8848-c55e-49fd-9cbe-bfda325c51c8"
-					(reference "#PWR023")
+					(reference "#PWR011")
 					(unit 1)
 				)
 				(path "/9770a3ff-dcb3-40dd-904f-3792f096cc81/461fdf99-31de-4f28-b803-0ca226183c1b/ad6ef6e9-1754-4226-a802-1e45b0c5c28a"
-					(reference "#PWR023")
+					(reference "#PWR017")
 					(unit 1)
 				)
@@
 		(dnp no)
 		(fields_autoplaced yes)
-		(property "Reference" "U7"
+		(property "Reference" "U1"
 			(at 97.3933 41.91 0)
 			(show_name no)
@@
 			)
 		)
-		(property "Footprint" ""
+		(property "Footprint" "Package_SO:SOIC-16_3.9x9.9mm_P1.27mm"
 			(at 95.25 64.77 0)
 			(hide yes)
@@
 				)
 				(path "/9770a3ff-dcb3-40dd-904f-3792f096cc81/461fdf99-31de-4f28-b803-0ca226183c1b/4bfad7ce-72f4-4d4b-b445-f07a93594dc1"
-					(reference "U7")
+					(reference "U1")
 					(unit 1)
 				)
 				(path "/9770a3ff-dcb3-40dd-904f-3792f096cc81/461fdf99-31de-4f28-b803-0ca226183c1b/9c0f8848-c55e-49fd-9cbe-bfda325c51c8"
-					(reference "U7")
+					(reference "U3")
 					(unit 1)
 				)
 				(path "/9770a3ff-dcb3-40dd-904f-3792f096cc81/461fdf99-31de-4f28-b803-0ca226183c1b/ad6ef6e9-1754-4226-a802-1e45b0c5c28a"
-					(reference "U7")
-					(unit 1)
-				)
+					(reference "U5")
+					(unit 1)
+				)
