File: hardware/kicad/modules/mux/drivers-74xx/driver1_8to1.kicad_sch (KiCad schematic)
At the start: 6 parts, among them U1 74AHCT125, U2 74AHCT125, U3 74AHCT138

Commit message: module: designed muxes prioritizing drivers for large switching preserving depth of ~1 gate
Parts:
- renumbered C1 to C35, C2 to C36, C3 to C37, U1 to U39, U2 to U40, U3 to U41

Commit message: refactor: changed hpins to global for asel, ainv, precondition, alu-opcode
Parts:
- renumbered C35 to C111, C36 to C112, C37 to C113, U39 to U131, U40 to U132, U41 to U133

Commit message: refactor: improved driver with data bus for readability
Parts:
- renumbered C111 to C401, C113 to C402, C112 to C403, U131 to U401, U133 to U402, U132 to U403

Commit message: arch: added LEDs, override switches; fixed errors and warnings to 0
ready for routing after logical coherence check
Parts:
- renumbered C401 to C28, C403 to C29, C402 to C30, U401 to U28, U403 to U29, U402 to U30

Commit message: chore: modified muxes that alu depends on
Parts:
- renumbered C28 to C33, C29 to C34, C30 to C35, U28 to U33, U29 to U34, U30 to U35
