File: hardware/kicad/boards/07_alu/alu_1b_X.kicad_sch (KiCad schematic)
At the start: 2 parts, among them U4 74ACT151

Commit message: schematics: implemented adder(lut3, lut3, h(cin)) design
Parts:
- renumbered C6 to C7, U4 to U7

Commit message: chore: renamed and organized 1b cells
Parts:
- renumbered C7 to C54, U7 to U49
