File: hardware/kicad/boards/07_alu/alu_1b_Y.kicad_sch (KiCad schematic)
At the start: 2 parts, among them U10 74ACT151

Commit message: schematics: implemented adder(lut3, lut3, h(cin)) design
Parts:
- removed C42: 100nF, Capacitor_SMD:C_0603_1608Metric, symbol Device:C
- removed U10: 74ACT151, Package_SO:SOIC-16_3.9x9.9mm_P1.27mm, symbol 74xx:74LS151
- added C11: 100nF, Capacitor_SMD:C_0603_1608Metric, symbol Device:C
- added U11: 74ACT151, Package_SO:SOIC-16_3.9x9.9mm_P1.27mm, symbol 74xx:74LS151
Connections:
- net 1b-out: now also U11.5 (Z)
- net ALU_OPCODE_Y0: now also U11.4 (I0)
- net ALU_OPCODE_Y1: now also U11.3 (I1)
- net ALU_OPCODE_Y2: now also U11.2 (I2)
- net ALU_OPCODE_Y3: now also U11.1 (I3)
- net ALU_OPCODE_Y4: now also U11.15 (I4)
- net ALU_OPCODE_Y5: now also U11.14 (I5)
- net ALU_OPCODE_Y6: now also U11.13 (I6)
- net ALU_OPCODE_Y7: now also U11.12 (I7)
- net GND: now also C11.1, U11.7 (~{E}), U11.8 (GND)
- net VCC: now also C11.2, U11.16 (VCC)
- net a: now also U11.11 (S0)
- net b: now also U11.10 (S1)
- net c: now also U11.9 (S2)

Commit message: chore: renamed and organized 1b cells
Parts:
- renumbered C11 to C56, U11 to U56
