File: hardware/kicad/boards/07_alu/flags_logic.kicad_sch (KiCad schematic)
At the start: 14 parts, among them U1 74AHC541, U16 74ACT151, U2 74HC00, U36 74HC86, U4 74HC688, U40 74LS377, U6 74HC00

Commit message: fix: replaced with resistor array/network over individual components
fix #5
Parts:
- U1: value 74AHC541 -> 74ACT541
- U2, U6: value 74HC00 -> 74ACT00
- U36: value 74HC86 -> 74ACT86
- U40: value 74LS377 -> 74ACT377
Other:
- moved on the sheet: C39, U40
